File: hardware/receiver-pro/ByteCollection.sch (KiCad schematic (older format))
At the start: 13 parts, among them U10 74LS273, U21 74LS08, U24 74LS04, U9 74LS164

Commit message: Add part numbers.
Parts:
- gave numbers to parts that had none: 4
Changed lines of the file:
@@
 $EndDescr
 $Comp
-L 74xx:74LS161 U?
+L 74xx:74LS161 U4
 U 1 1 62477F8E
 P 3500 2100
-F 0 "U?" H 3600 2850 50  0000 C CNN
+F 0 "U4" H 3600 2850 50  0000 C CNN
 F 1 "74LS161" H 3700 2750 50  0000 C CNN
 F 2 "" H 3500 2100 50  0001 C CNN
@@
 $EndComp
 $Comp
-L 74xx:74LS10 U?
+L 74xx:74LS10 U5
 U 3 1 62477FA5
 P 4700 1700
-F 0 "U?" H 4700 2025 50  0000 C CNN
+F 0 "U5" H 4700 2025 50  0000 C CNN
 F 1 "74LS10" H 4700 1934 50  0000 C CNN
 F 2 "" H 4700 1700 50  0001 C CNN
@@
 $EndComp
 $Comp
-L 74xx:74LS04 U?
+L 74xx:74LS04 U24
 U 1 1 62477FAC
 P 5050 5700
-F 0 "U?" H 5050 6017 50  0000 C CNN
+F 0 "U24" H 5050 6017 50  0000 C CNN
 F 1 "74LS04" H 5050 5926 50  0000 C CNN
 F 2 "" H 5050 5700 50  0001 C CNN
@@
 $EndComp
 $Comp
-L 74xx:74LS04 U?
+L 74xx:74LS04 U24
 U 2 1 62477FB3
 P 5650 5700
-F 0 "U?" H 5650 6017 50  0000 C CNN
+F 0 "U24" H 5650 6017 50  0000 C CNN
 F 1 "74LS04" H 5650 5926 50  0000 C CNN
 F 2 "" H 5650 5700 50  0001 C CNN
@@
 $EndComp
 $Comp
-L 74xx:74LS04 U?
+L 74xx:74LS04 U24
 U 3 1 62477FBA
 P 6250 5700
-F 0 "U?" H 6250 6017 50  0000 C CNN
+F 0 "U24" H 6250 6017 50  0000 C CNN
 F 1 "74LS04" H 6250 5926 50  0000 C CNN
 F 2 "" H 6250 5700 50  0001 C CNN
@@
 $EndComp
 $Comp
-L 74xx:74LS04 U?
+L 74xx:74LS04 U24
 U 4 1 62477FC1
 P 6850 5700
-F 0 "U?" H 6850 6017 50  0000 C CNN
+F 0 "U24" H 6850 6017 50  0000 C CNN
 F 1 "74LS04" H 6850 5926 50  0000 C CNN
 F 2 "" H 6850 5700 50  0001 C CNN
@@
 $EndComp
 $Comp
-L 74xx:74LS10 U?
+L 74xx:74LS10 U5
 U 2 1 62477FC8
 P 6400 1800
-F 0 "U?" H 6400 2125 50  0000 C CNN
+F 0 "U5" H 6400 2125 50  0000 C CNN
 F 1 "74LS10" H 6400 2034 50  0000 C CNN
 F 2 "" H 6400 1800 50  0001 C CNN
@@
 $EndComp
 $Comp
-L 74xx:74LS32 U?
+L 74xx:74LS32 U22
 U 1 1 62477FCF
 P 7200 2300
-F 0 "U?" H 7200 2625 50  0000 C CNN
+F 0 "U22" H 7200 2625 50  0000 C CNN
 F 1 "74LS32" H 7200 2534 50  0000 C CNN
 F 2 "" H 7200 2300 50  0001 C CNN
@@
 $EndComp
 $Comp
-L 74xx:74LS32 U?
+L 74xx:74LS32 U22
 U 2 1 62477FD6
 P 7800 2400
-F 0 "U?" H 7800 2725 50  0000 C CNN
+F 0 "U22" H 7800 2725 50  0000 C CNN
 F 1 "74LS32" H 7800 2634 50  0000 C CNN
 F 2 "" H 7800 2400 50  0001 C CNN
@@
 Wire Wire Line
 	9500 1100 9650 1100
+Connection ~ 9500 1200
+Wire Wire Line
+	7400 5700 9650 5700
 Wire Bus Line
 	8900 4800 9650 4800
@@
 Wire Bus Line
 	8800 3900 8800 4700
-Connection ~ 9500 1200
-Wire Wire Line
-	7400 5700 9650 5700
 $EndSCHEMATC
