File: hardware/receiver-pro/DimmerMultiplex.sch (KiCad schematic (older format))
At the start: 13 parts

Commit message: Add part numbers.
Parts:
- gave numbers to parts that had none: 10
Connections:
- net labels added: DS4, ~SC_SEL_OUT
- wire segments 159 -> 162
- no-connect marks 13 -> 12
