File: hardware/receiver-pro/d2a.sch (KiCad schematic (older format))
At the start: 29 parts

Commit message: Split RX-Pro into multi-sheet schematic.
Parts:
- removed C?: .01uF, symbol Device:C
- removed R?: 10k, symbol Device:R_US
- removed U? (x2): 74LS32, symbol 74xx:74LS32
- removed U? (x4): 74LS02, symbol 74xx:74LS02
- removed U? (x4): 74LS273, symbol 74xx:74LS273
Connections:
- net labels added: D1_DATA[0..7], D2_DATA[0..7], D3_DATA[0..7], D4_DATA[0..7]
- net labels removed: D0, D1, D1L, D2, D2L, D3, D3L, D4, D4L, D5, D6, D7, DS0, DS1, DS2, DS3, DS[0..3], D[0..7], SB, SM0, SM1
- wire segments 229 -> 116
Other:
- note removed: "Dimmer\nLatches"

Commit message: Add part numbers.
Parts:
- added BAR? (x4): LED, Display:HDSP-4830, symbol LED:HDSP-4830_2
- added RN? (x4): 330, Resistor_THT:R_Array_SIP11, symbol Device:R_Network10_US
Connections:
- net labels added: D1L, D2L, D3L, D4L
- wire segments 116 -> 160
- no-connect marks 0 -> 4
Other:
- moved on the sheet: U?
