File: hardware/receiver-pro/receiver-pro.sch (KiCad schematic (older format))
At the start: 25 parts, among them J1 Input, U1 74LS74, U10 74LS273, U11 74LS161, U12 74LS154, U13 74LS273, U14 74LS85, U15 74LS85, U2 74LS161, U20 74LS10, U21 74LS08, U22 74LS32, U24 74LS04, U3 74LS74, U4 74LS161, U5 74LS10, U6 74LS161, U7 74LS161, U8 74LS32, U9 74LS164

Commit message: Split RX-Pro into multi-sheet schematic.
Parts:
- removed C6: .0056uF, symbol Device:C_Small
- removed DSW1: START_LO, symbol Switch:SW_DIP_x04
- removed DSW2: START_HI, symbol Switch:SW_DIP_x04
- removed J1: Input, symbol Connector_Generic:Conn_01x03
- removed RN1, RN2: 10k, Resistor_THT:R_Array_SIP5, symbol Device:R_Network04
- removed U1, U3: 74LS74, symbol 74xx:74LS74
- removed U10, U13: 74LS273, symbol 74xx:74LS273
- removed U11, U2, U4, U6, U7: 74LS161, symbol 74xx:74LS161
- removed U12: 74LS154, symbol 74xx:74LS154
- removed U14, U15: 74LS85, symbol 74xx:74LS85
- removed U20, U5: 74LS10, symbol 74xx:74LS10
- removed U21: 74LS08, symbol 74xx:74LS08
- removed U22, U8: 74LS32, symbol 74xx:74LS32
- removed U24: 74LS04, symbol 74xx:74LS04
- removed U9: 74LS164, digikey-footprints:DIP-14_W3mm, symbol dk_Logic-Shift-Registers:SN74HC164N
- added J?: Input, symbol Connector_Generic:Conn_01x03
Connections:
- net labels removed: +5V, CLK, D0, D01, D1, D2, D3, D4, D5, D6, D7, DL, DM0, DM1, DM2, DO0, DO2, DO3, DO4, DO5, DO6, DO7, DS0, DS1, DS2, DS3, DS[0..3], D[0..7], SB, SC, SC0, SC1, SC2, SC3, SC4, SC5, SC6, SC7, SCL, SC[0..7], SL0, SL1, SL2, SM0, SM1, SM2, ~FRAME_RST
- wire segments 424 -> 22
- no-connect marks 24 -> 0
Other:
- note added: "Byte\nCollection"
- note added: "Dimmer\nMultiplex"
- note added: "Original\nLogic"
- note added: "Start\nCode"
- note added: "UART"
- note removed: "Break\nDetector"
- note removed: "Byte Sequence\nClock"
- note removed: "Clock Sync\nGenerator"
- note removed: "Clock Sync\nReset"
- note removed: "Clock/2"
- note removed: "Dimmer Counter/\nMultiplexer"
- note removed: "Serial Byte Latch Delay\n"
- note removed: "Serial Shift \nRegister\n"
- note removed: "Serial Transition \nDetector"
- note removed: "Serial\nBit Latch\n"
- note removed: "Serial\nByte Latch\n"
- note removed: "Start Code\nCompare"
- note removed: "Start Code\nLatch"
- note removed: "Stop Bit Delay"
- note removed: "Stop Bit Detector"

Commit message: Add part numbers.
Connections:
- wire segments 22 -> 24
Changed lines of the file:
@@
 $EndDescr
 $Sheet
-S 8750 2150 1450 800
+S 8350 2650 1850 800
 U 5F2B3F8A
 F0 "d2a" 50
 F1 "d2a.sch" 50
+F2 "D1_DATA[0..7]" I L 8350 3000 50
+F3 "D2_DATA[0..7]" I L 8350 3100 50
+F4 "D3_DATA[0..7]" I L 8350 3200 50
+F5 "D4_DATA[0..7]" I L 8350 3300 50
 $EndSheet
 $Sheet
-S 8950 3900 850  600
+S 5000 5450 850  600
 U 5F2B4C18
 F0 "display" 50
@@
 F1 "power.sch" 50
 $EndSheet
-Text Notes 9150 2700 0    100  Italic 20
+Text Notes 8350 2550 0    100  Italic 20
   D to A\nConverters
-Text Notes 9050 4250 0    100  Italic 20
+Text Notes 5100 5800 0    100  Italic 20
 Display
 Text Notes 3000 5550 0    100  Italic 20
 Power
 $Sheet
-S 1450 2150 1450 550
+S 1550 2650 1450 550
 U 615F2306
 F0 "Receiver" 50
 F1 "Receiver.sch" 50
-F2 "RX_DATA_IN" I L 1450 2250 50
-F3 "RX_CLOCK_IN" I L 1450 2350 50
-F4 "BYTE_RESET_OUT" I R 2900 2350 50
-F5 "BIT_CLOCK_OUT" I R 2900 2250 50
-F6 "BYTE_END_IN" I R 2900 2450 50
-F7 "~FRAME_RST_OUT" I R 2900 2600 50
+F2 "RX_DATA_IN" I L 1550 2750 50
+F3 "RX_CLOCK_IN" I L 1550 2950 50
+F4 "BYTE_RESET_OUT" I R 3000 2850 50
+F5 "BIT_CLOCK_OUT" I R 3000 2750 50
+F6 "BYTE_END_IN" I R 3000 2950 50
+F7 "~FRAME_RST_OUT" I R 3000 3100 50
 $EndSheet
 $Sheet
-S 3400 1950 1800 750
+S 3400 2450 1800 750
 U 62477DE1
 F0 "ByteCollection" 50
 F1 "ByteCollection.sch" 50
-F2 "RX_DATA_IN" I L 3400 2050 50
-F3 "BYTE_RESET_IN" I L 3400 2350 50
-F4 "BIT_CLOCK_IN" I L 3400 2250 50
-F5 "DIM_INC_OUT" I R 5200 2450 50
-F6 "DATA[0..7]" I R 5200 2250 50
-F7 "STOP_BIT_OUT" I R 5200 2350 50
-F8 "BYTE_END_OUT" I L 3400 2450 50
+F2 "RX_DATA_IN" I L 3400 2550 50
+F3 "BYTE_RESET_IN" I L 3400 2850 50
+F4 "BIT_CLOCK_IN" I L 3400 2750 50
+F5 "DIM_INC_OUT" I R 5200 3050 50
+F6 "DATA[0..7]" I R 5200 2850 50
+F7 "STOP_BIT_OUT" I R 5200 2950 50
+F8 "BYTE_END_OUT" I L 3400 2950 50
 $EndSheet
 $Sheet
-S 5750 2150 2650 800
+S 5850 2650 2050 800
 U 627E727E
 F0 "DimmerMultiplex" 50
 F1 "DimmerMultiplex.sch" 50
-F2 "~FRAME_RST_IN" I L 5750 2850 50
-F3 "D1_DATA[0..7]" I R 8400 2500 50
-F4 "D2_DATA[0..7]" I R 8400 2600 50
-F5 "D4_DATA[0..7]" I R 8400 2800 50
-F6 "D3_DATA[0..7]" I R 8400 2700 50
-F7 "DIM_INC_IN" I L 5750 2450 50
-F8 "DATA[0..7]" I L 5750 2250 50
-F9 "SC_MATCH_IN" I R 8400 2250 50
-F10 "STOP_BIT_IN" I L 5750 2350 50
+F2 "~FRAME_RST_IN" I L 5850 3350 50
+F3 "D1_DATA[0..7]" I R 7900 3000 50
+F4 "D2_DATA[0..7]" I R 7900 3100 50
+F5 "D4_DATA[0..7]" I R 7900 3300 50
+F6 "D3_DATA[0..7]" I R 7900 3200 50
+F7 "DIM_INC_IN" I L 5850 3050 50
+F8 "DATA[0..7]" I L 5850 2850 50
+F9 "SC_MATCH_IN" I R 7900 2750 50
+F10 "STOP_BIT_IN" I L 5850 2950 50
+F11 "~SC_SEL_OUT" I L 5850 2750 50
 $EndSheet
 $Sheet
-S 5750 1300 2650 600
+S 5850 1800 2050 600
 U 627E73CB
 F0 "StartCode" 50
 F1 "StartCode.sch" 50
-F2 "STOP_BIT_IN" I L 5750 1700 50
-F3 "~FRAME_RST_IN" I L 5750 1600 50
-F4 "SC_MATCH_OUT" I R 8400 1750 50
-F5 "DATA[0..7]" I L 5750 1800 50
+F2 "STOP_BIT_IN" I L 5850 2100 50
+F3 "SC_MATCH_OUT" I R 7900 2250 50
+F4 "DATA[0..7]" I L 5850 2200 50
+F5 "~SC_SEL_IN" I L 5850 2300 50
 $EndSheet
 $Sheet
@@
 F1 "Original-Logic.sch" 50
 $EndSheet
-Text Notes 2050 1950 0    100  Italic 20
+Text Notes 2150 2450 0    100  Italic 20
 UART
-Text Notes 3400 1850 0    100  Italic 20
+Text Notes 3500 2350 0    100  Italic 20
 Byte\nCollection
-Text Notes 6750 2700 0    100  Italic 20
+Text Notes 5850 3850 0    100  Italic 20
 Dimmer\nMultiplex
-Text Notes 6850 1750 0    100  Italic 20
+Text Notes 5850 1700 0    100  Italic 20
 Start\nCode
 Text Notes 5050 7500 0    100  Italic 20
@@
 $EndSheet
 Wire Wire Line
-	1100 2250 1300 2250
-Text Label 1100 2250 0    50   ~ 0
+	1150 2750 1400 2750
+Text Label 1250 2750 0    50   ~ 0
 RX
-Text Label 1100 2350 0    50   ~ 0
+Text Label 1250 2950 0    50   ~ 0
 RXCLK
 $Comp
 L Connector_Generic:Conn_01x03 J?
 U 1 1 6336B4A9
-P 900 2350
+P 950 2850
 AR Path="/615F2306/6336B4A9" Ref="J?"  Part="1"
 AR Path="/6336B4A9" Ref="J?"  Part="1"
-F 0 "J?" H 750 2700 50  0000 L CNN
-F 1 "Input" H 700 2600 50  0000 L CNN
-F 2 "" H 900 2350 50  0001 C CNN
-F 3 "~" H 900 2350 50  0001 C CNN
-	1    900  2350
-	-1   0    0    -1
+F 0 "J?" H 800 2500 50  0000 L CNN
+F 1 "Input" H 750 2600 50  0000 L CNN
+F 2 "" H 950 2850 50  0001 C CNN
+F 3 "~" H 950 2850 50  0001 C CNN
+	1    950  2850
+	-1   0    0    1
 $EndComp
 $Comp
 L power:GND #PWR?
 U 1 1 6336B4B0
-P 1100 2450
+P 1200 3100
 AR Path="/615F2306/6336B4B0" Ref="#PWR?"  Part="1"
 AR Path="/6336B4B0" Ref="#PWR?"  Part="1"
-F 0 "#PWR?" H 1100 2200 50  0001 C CNN
-F 1 "GND" H 1105 2277 50  0000 C CNN
-F 2 "" H 1100 2450 50  0001 C CNN
-F 3 "" H 1100 2450 50  0001 C CNN
-	1    1100 2450
+F 0 "#PWR?" H 1200 2850 50  0001 C CNN
+F 1 "GND" H 1205 2927 50  0000 C CNN
+F 2 "" H 1200 3100 50  0001 C CNN
+F 3 "" H 1200 3100 50  0001 C CNN
+	1    1200 3100
 	-1   0    0    -1
 $EndComp
 Wire Wire Line
-	1450 2350 1100 2350
+	1550 2950 1150 2950
 Wire Wire Line
-	2900 2250 3400 2250
+	3000 2750 3400 2750
 Wire Wire Line
-	1300 2250 1300 2050
+	1400 2750 1400 2550
 Wire Wire Line
-	1300 2050 3400 2050
-Connection ~ 1300 2250
+	1400 2550 3400 2550
+Connection ~ 1400 2750
 Wire Wire Line
-	1300 2250 1450 2250
+	1400 2750 1550 2750
 Wire Wire Line
-	3400 2350 2900 2350
+	3400 2850 3000 2850
 Wire Wire Line
-	2900 2450 3400 2450
+	3000 2950 3400 2950
 Wire Wire Line
-	2900 2600 3150 2600
+	3000 3100 3250 3100
 Wire Wire Line
-	3150 2600 3150 2850
+	3250 3100 3250 3350
 Wire Wire Line
-	5200 2450 5750 2450
+	7900 2250 8050 2250
+Wire Wire Line
+	8050 2250 8050 2750
+Wire Wire Line
+	8050 2750 7900 2750
+Wire Bus Line
+	7900 3000 8350 3000
+Wire Bus Line
+	7900 3100 8350 3100
+Wire Bus Line
+	7900 3200 8350 3200
+Wire Bus Line
+	7900 3300 8350 3300
+Wire Wire Line
+	1150 2850 1200 2850
+Wire Wire Line
+	1200 2850 1200 3100
+Wire Wire Line
+	5200 2950 5400 2950
+Wire Wire Line
+	3250 3350 5850 3350
+Wire Wire Line
+	5400 2100 5850 2100
+Wire Bus Line
+	5850 2200 5600 2200
+Wire Bus Line
+	5600 2200 5600 2750
+Wire Wire Line
+	5400 2100 5400 2950
+Connection ~ 5400 2950
+Wire Wire Line
+	5400 2950 5850 2950
 Entry Bus Bus
-	5500 2250 5600 2150
+	5500 2850 5600 2750
+Wire Wire Line
+	5850 2750 5750 2750
+Wire Wire Line
+	5750 2750 5750 2300
+Wire Wire Line
+	5750 2300 5850 2300
+Wire Wire Line
+	5200 3050 5850 3050
 Wire Bus Line
-	5600 2150 5600 1800
-Wire Bus Line
-	5600 1800 5750 1800
-Wire Wire Line
-	5400 1700 5750 1700
-Wire Wire Line
-	5300 1600 5750 1600
-Wire Wire Line
-	5400 1700 5400 2350
-Wire Wire Line
-	5200 2350 5400 2350
-Connection ~ 5400 2350
-Wire Wire Line
-	5400 2350 5750 2350
-Wire Wire Line
-	3150 2850 5300 2850
-Wire Wire Line
-	5300 1600 5300 2850
-Connection ~ 5300 2850
-Wire Wire Line
-	5300 2850 5750 2850
-Wire Wire Line
-	8400 1750 8500 1750
-Wire Wire Line
-	8500 1750 8500 2250
-Wire Wire Line
-	8500 2250 8400 2250
-Wire Bus Line
-	5200 2250 5750 2250
+	5200 2850 5850 2850
 $EndSCHEMATC
