File: hardware/transmitter-retro/control-dmx/address.sch (KiCad schematic (older format))
At the start: 3 parts

Commit message: Add top level project Update part #s Update power sheets
Parts:
- gave numbers to parts that had none: 3
Connections:
- net labels added: IA[0..11]
- net labels removed: IA[0..7]
Changed lines of the file:
@@
 AR Path="/632F1F43/64A87AD6" Ref="U?"  Part="1"
 AR Path="/63267F40/64A87AD6" Ref="U?"  Part="1"
-AR Path="/649D0DCA/64A87AD6" Ref="U?"  Part="1"
-F 0 "U?" H 4000 4150 50  0000 C CNN
+AR Path="/649D0DCA/64A87AD6" Ref="U4"  Part="1"
+F 0 "U4" H 4000 4150 50  0000 C CNN
 F 1 "74LS161" H 4100 4050 50  0000 C CNN
 F 2 "Package_DIP:DIP-16_W7.62mm" H 3900 3400 50  0001 C CNN
@@
 AR Path="/632F1F43/64A87ADD" Ref="#PWR?"  Part="1"
 AR Path="/63267F40/64A87ADD" Ref="#PWR?"  Part="1"
-AR Path="/649D0DCA/64A87ADD" Ref="#PWR?"  Part="1"
-F 0 "#PWR?" H 3900 3950 50  0001 C CNN
+AR Path="/649D0DCA/64A87ADD" Ref="#PWR0105"  Part="1"
+F 0 "#PWR0105" H 3900 3950 50  0001 C CNN
 F 1 "GND" H 4050 4100 50  0000 C CNN
 F 2 "" H 3900 4200 50  0001 C CNN
@@
 AR Path="/632F1F43/64A87AF0" Ref="#PWR?"  Part="1"
 AR Path="/63267F40/64A87AF0" Ref="#PWR?"  Part="1"
-AR Path="/649D0DCA/64A87AF0" Ref="#PWR?"  Part="1"
-F 0 "#PWR?" H 3250 3000 50  0001 C CNN
+AR Path="/649D0DCA/64A87AF0" Ref="#PWR0106"  Part="1"
+F 0 "#PWR0106" H 3250 3000 50  0001 C CNN
 F 1 "GND" H 3255 3077 50  0000 C CNN
 F 2 "" H 3250 3250 50  0001 C CNN
@@
 AR Path="/632F1F43/64A87AFD" Ref="#PWR?"  Part="1"
 AR Path="/63267F40/64A87AFD" Ref="#PWR?"  Part="1"
-AR Path="/649D0DCA/64A87AFD" Ref="#PWR?"  Part="1"
-F 0 "#PWR?" H 3900 2450 50  0001 C CNN
+AR Path="/649D0DCA/64A87AFD" Ref="#PWR0107"  Part="1"
+F 0 "#PWR0107" H 3900 2450 50  0001 C CNN
 F 1 "+5V" H 3915 2773 50  0000 C CNN
 F 2 "" H 3900 2600 50  0001 C CNN
@@
 AR Path="/632F1F43/64A87B08" Ref="#PWR?"  Part="1"
 AR Path="/63267F40/64A87B08" Ref="#PWR?"  Part="1"
-AR Path="/649D0DCA/64A87B08" Ref="#PWR?"  Part="1"
-F 0 "#PWR?" H 3100 2450 50  0001 C CNN
+AR Path="/649D0DCA/64A87B08" Ref="#PWR0108"  Part="1"
+F 0 "#PWR0108" H 3100 2450 50  0001 C CNN
 F 1 "+5V" H 3115 2773 50  0000 C CNN
 F 2 "" H 3100 2600 50  0001 C CNN
@@
 AR Path="/632F1F43/64A87B10" Ref="U?"  Part="1"
 AR Path="/63267F40/64A87B10" Ref="U?"  Part="1"
-AR Path="/649D0DCA/64A87B10" Ref="U?"  Part="1"
-F 0 "U?" H 5700 4150 50  0000 C CNN
+AR Path="/649D0DCA/64A87B10" Ref="U5"  Part="1"
+F 0 "U5" H 5700 4150 50  0000 C CNN
 F 1 "74LS161" H 5800 4050 50  0000 C CNN
 F 2 "Package_DIP:DIP-16_W7.62mm" H 5600 3400 50  0001 C CNN
@@
 AR Path="/632F1F43/64A87B17" Ref="#PWR?"  Part="1"
 AR Path="/63267F40/64A87B17" Ref="#PWR?"  Part="1"
-AR Path="/649D0DCA/64A87B17" Ref="#PWR?"  Part="1"
-F 0 "#PWR?" H 5600 3950 50  0001 C CNN
+AR Path="/649D0DCA/64A87B17" Ref="#PWR0109"  Part="1"
+F 0 "#PWR0109" H 5600 3950 50  0001 C CNN
 F 1 "GND" H 5750 4100 50  0000 C CNN
 F 2 "" H 5600 4200 50  0001 C CNN
@@
 AR Path="/632F1F43/64A87B29" Ref="#PWR?"  Part="1"
 AR Path="/63267F40/64A87B29" Ref="#PWR?"  Part="1"
-AR Path="/649D0DCA/64A87B29" Ref="#PWR?"  Part="1"
-F 0 "#PWR?" H 4950 3000 50  0001 C CNN
+AR Path="/649D0DCA/64A87B29" Ref="#PWR0110"  Part="1"
+F 0 "#PWR0110" H 4950 3000 50  0001 C CNN
 F 1 "GND" H 4955 3077 50  0000 C CNN
 F 2 "" H 4950 3250 50  0001 C CNN
@@
 AR Path="/632F1F43/64A87B31" Ref="#PWR?"  Part="1"
 AR Path="/63267F40/64A87B31" Ref="#PWR?"  Part="1"
-AR Path="/649D0DCA/64A87B31" Ref="#PWR?"  Part="1"
-F 0 "#PWR?" H 5600 2450 50  0001 C CNN
+AR Path="/649D0DCA/64A87B31" Ref="#PWR0111"  Part="1"
+F 0 "#PWR0111" H 5600 2450 50  0001 C CNN
 F 1 "+5V" H 5615 2773 50  0000 C CNN
 F 2 "" H 5600 2600 50  0001 C CNN
@@
 AR Path="/632F1F43/64A87B3B" Ref="#PWR?"  Part="1"
 AR Path="/63267F40/64A87B3B" Ref="#PWR?"  Part="1"
-AR Path="/649D0DCA/64A87B3B" Ref="#PWR?"  Part="1"
-F 0 "#PWR?" H 4800 2450 50  0001 C CNN
+AR Path="/649D0DCA/64A87B3B" Ref="#PWR0112"  Part="1"
+F 0 "#PWR0112" H 4800 2450 50  0001 C CNN
 F 1 "+5V" H 4815 2773 50  0000 C CNN
 F 2 "" H 4800 2600 50  0001 C CNN
@@
 AR Path="/632F1F43/64A87B65" Ref="U?"  Part="1"
 AR Path="/63267F40/64A87B65" Ref="U?"  Part="1"
-AR Path="/649D0DCA/64A87B65" Ref="U?"  Part="1"
-F 0 "U?" H 7400 4150 50  0000 C CNN
+AR Path="/649D0DCA/64A87B65" Ref="U6"  Part="1"
+F 0 "U6" H 7400 4150 50  0000 C CNN
 F 1 "74LS161" H 7500 4050 50  0000 C CNN
 F 2 "Package_DIP:DIP-16_W7.62mm" H 7300 3400 50  0001 C CNN
@@
 AR Path="/632F1F43/64A87B6C" Ref="#PWR?"  Part="1"
 AR Path="/63267F40/64A87B6C" Ref="#PWR?"  Part="1"
-AR Path="/649D0DCA/64A87B6C" Ref="#PWR?"  Part="1"
-F 0 "#PWR?" H 7300 3950 50  0001 C CNN
+AR Path="/649D0DCA/64A87B6C" Ref="#PWR0113"  Part="1"
+F 0 "#PWR0113" H 7300 3950 50  0001 C CNN
 F 1 "GND" H 7450 4100 50  0000 C CNN
 F 2 "" H 7300 4200 50  0001 C CNN
@@
 AR Path="/632F1F43/64A87B7E" Ref="#PWR?"  Part="1"
 AR Path="/63267F40/64A87B7E" Ref="#PWR?"  Part="1"
-AR Path="/649D0DCA/64A87B7E" Ref="#PWR?"  Part="1"
-F 0 "#PWR?" H 6650 3000 50  0001 C CNN
+AR Path="/649D0DCA/64A87B7E" Ref="#PWR0114"  Part="1"
+F 0 "#PWR0114" H 6650 3000 50  0001 C CNN
 F 1 "GND" H 6655 3077 50  0000 C CNN
 F 2 "" H 6650 3250 50  0001 C CNN
@@
 AR Path="/632F1F43/64A87B86" Ref="#PWR?"  Part="1"
 AR Path="/63267F40/64A87B86" Ref="#PWR?"  Part="1"
-AR Path="/649D0DCA/64A87B86" Ref="#PWR?"  Part="1"
-F 0 "#PWR?" H 7300 2450 50  0001 C CNN
+AR Path="/649D0DCA/64A87B86" Ref="#PWR0115"  Part="1"
+F 0 "#PWR0115" H 7300 2450 50  0001 C CNN
 F 1 "+5V" H 7315 2773 50  0000 C CNN
 F 2 "" H 7300 2600 50  0001 C CNN
@@
 AR Path="/632F1F43/64A87B90" Ref="#PWR?"  Part="1"
 AR Path="/63267F40/64A87B90" Ref="#PWR?"  Part="1"
-AR Path="/649D0DCA/64A87B90" Ref="#PWR?"  Part="1"
-F 0 "#PWR?" H 6500 2450 50  0001 C CNN
+AR Path="/649D0DCA/64A87B90" Ref="#PWR0116"  Part="1"
+F 0 "#PWR0116" H 6500 2450 50  0001 C CNN
 F 1 "+5V" H 6515 2773 50  0000 C CNN
 F 2 "" H 6500 2600 50  0001 C CNN
@@
 ~FRAME_RESET_IN
 Text HLabel 8450 2350 2    50   Input ~ 0
-IA[0..7]
+IA[0..11]
 Wire Bus Line
 	4750 2350 8450 2350
