File: hardware/transmitter-retro/control-dmx/eeprom.sch (KiCad schematic (older format))
At the start: 6 parts

Commit message: Add top level project Update part #s Update power sheets
Parts:
- gave numbers to parts that had none: 3
Connections:
- net labels added: IA[0..11]
- net labels removed: IA[0..7]
Changed lines of the file:
@@
 AR Path="/632F1F43/64A8E383" Ref="U?"  Part="1"
 AR Path="/63267F40/64A8E383" Ref="U?"  Part="1"
-AR Path="/649D105F/64A8E383" Ref="U?"  Part="1"
-F 0 "U?" H 4750 4850 50  0000 C CNN
+AR Path="/649D105F/64A8E383" Ref="U7"  Part="1"
+F 0 "U7" H 4750 4850 50  0000 C CNN
 F 1 "27128" H 4800 4750 50  0000 C CNN
 F 2 "Package_DIP:DIP-28_W15.24mm" H 4600 3700 50  0001 C CNN
@@
 AR Path="/632F1F43/64A8E38A" Ref="#PWR?"  Part="1"
 AR Path="/63267F40/64A8E38A" Ref="#PWR?"  Part="1"
-AR Path="/649D105F/64A8E38A" Ref="#PWR?"  Part="1"
-F 0 "#PWR?" H 4600 4550 50  0001 C CNN
+AR Path="/649D105F/64A8E38A" Ref="#PWR0118"  Part="1"
+F 0 "#PWR0118" H 4600 4550 50  0001 C CNN
 F 1 "GND" H 4605 4627 50  0000 C CNN
 F 2 "" H 4600 4800 50  0001 C CNN
@@
 AR Path="/632F1F43/64A8E390" Ref="#PWR?"  Part="1"
 AR Path="/63267F40/64A8E390" Ref="#PWR?"  Part="1"
-AR Path="/649D105F/64A8E390" Ref="#PWR?"  Part="1"
-F 0 "#PWR?" H 4600 2450 50  0001 C CNN
+AR Path="/649D105F/64A8E390" Ref="#PWR0119"  Part="1"
+F 0 "#PWR0119" H 4600 2450 50  0001 C CNN
 F 1 "+5V" H 4615 2773 50  0000 C CNN
 F 2 "" H 4600 2600 50  0001 C CNN
@@
 AR Path="/632F1F43/64A8E3A2" Ref="#PWR?"  Part="1"
 AR Path="/63267F40/64A8E3A2" Ref="#PWR?"  Part="1"
-AR Path="/649D105F/64A8E3A2" Ref="#PWR?"  Part="1"
-F 0 "#PWR?" H 4100 4550 50  0001 C CNN
+AR Path="/649D105F/64A8E3A2" Ref="#PWR0120"  Part="1"
+F 0 "#PWR0120" H 4100 4550 50  0001 C CNN
 F 1 "GND" H 4105 4627 50  0000 C CNN
 F 2 "" H 4100 4800 50  0001 C CNN
@@
 AR Path="/632F1F43/64A8E3B4" Ref="#PWR?"  Part="1"
 AR Path="/63267F40/64A8E3B4" Ref="#PWR?"  Part="1"
-AR Path="/649D105F/64A8E3B4" Ref="#PWR?"  Part="1"
-F 0 "#PWR?" H 3950 4050 50  0001 C CNN
+AR Path="/649D105F/64A8E3B4" Ref="#PWR0121"  Part="1"
+F 0 "#PWR0121" H 3950 4050 50  0001 C CNN
 F 1 "+5V" H 3965 4373 50  0000 C CNN
 F 2 "" H 3950 4200 50  0001 C CNN
@@
 P 6700 4000
 AR Path="/64A8E3CD" Ref="U?"  Part="3"
-AR Path="/649D105F/64A8E3CD" Ref="U?"  Part="3"
-F 0 "U?" H 6700 4325 50  0000 C CNN
+AR Path="/649D105F/64A8E3CD" Ref="U3"  Part="3"
+F 0 "U3" H 6700 4325 50  0000 C CNN
 F 1 "74LS32" H 6700 4234 50  0000 C CNN
 F 2 "Package_DIP:DIP-14_W7.62mm" H 6700 4000 50  0001 C CNN
@@
 P 7400 4100
 AR Path="/64A8E3D4" Ref="U?"  Part="4"
-AR Path="/649D105F/64A8E3D4" Ref="U?"  Part="4"
-F 0 "U?" H 7400 4425 50  0000 C CNN
+AR Path="/649D105F/64A8E3D4" Ref="U3"  Part="4"
+F 0 "U3" H 7400 4425 50  0000 C CNN
 F 1 "74LS32" H 7400 4334 50  0000 C CNN
 F 2 "Package_DIP:DIP-14_W7.62mm" H 7400 4100 50  0001 C CNN
@@
 AR Path="/632F1F43/64A8E3DC" Ref="U?"  Part="2"
 AR Path="/63267F40/64A8E3DC" Ref="U?"  Part="2"
-AR Path="/649D105F/64A8E3DC" Ref="U?"  Part="2"
-F 0 "U?" H 6000 4733 50  0000 C CNN
+AR Path="/649D105F/64A8E3DC" Ref="U3"  Part="2"
+F 0 "U3" H 6000 4733 50  0000 C CNN
 F 1 "74LS32" H 6000 4824 50  0000 C CNN
 F 2 "Package_DIP:DIP-14_W7.62mm" H 6000 5050 50  0001 C CNN
@@
 P 6000 3900
 AR Path="/64A8E3EF" Ref="U?"  Part="1"
-AR Path="/649D105F/64A8E3EF" Ref="U?"  Part="1"
-F 0 "U?" H 6000 4225 50  0000 C CNN
+AR Path="/649D105F/64A8E3EF" Ref="U1"  Part="1"
+F 0 "U1" H 6000 4225 50  0000 C CNN
 F 1 "74LS00" H 6000 4134 50  0000 C CNN
 F 2 "Package_DIP:DIP-14_W7.62mm" H 6000 3900 50  0001 C CNN
@@
 P 6000 4500
 AR Path="/64A8E3F9" Ref="U?"  Part="1"
-AR Path="/649D105F/64A8E3F9" Ref="U?"  Part="1"
-F 0 "U?" H 6000 4825 50  0000 C CNN
+AR Path="/649D105F/64A8E3F9" Ref="U3"  Part="1"
+F 0 "U3" H 6000 4825 50  0000 C CNN
 F 1 "74LS32" H 6000 4734 50  0000 C CNN
 F 2 "Package_DIP:DIP-14_W7.62mm" H 6000 4500 50  0001 C CNN
@@
 	7700 4100 8300 4100
 Text HLabel 2950 1800 0    50   Input ~ 0
-IA[0..7]
+IA[0..11]
 Wire Bus Line
 	2950 1800 3800 1800
