File: hardware/transmitter-retro/control-logic/sample.sch (KiCad schematic (older format))
At the start: 5 parts, among them U11 74LS08, U14 74LS10, U15 74LS32, U4 74LS163, U5 74LS163

Commit message: Add top level project Update part #s Update power sheets
Parts:
- renumbered U11 to U1, U4 to U13, U5 to U14, U14 to U2, U15 to U6
Changed lines of the file:
@@
 AR Path="/6328016E/634715A6" Ref="U?"  Part="1"
 AR Path="/63397143/634715A6" Ref="U?"  Part="1"
-AR Path="/63268641/634715A6" Ref="U4"  Part="1"
-F 0 "U4" H 4800 4200 50  0000 C CNN
+AR Path="/63268641/634715A6" Ref="U13"  Part="1"
+F 0 "U13" H 4800 4200 50  0000 C CNN
 F 1 "74LS163" H 4900 4100 50  0000 C CNN
 F 2 "Package_DIP:DIP-16_W7.62mm" H 4700 3450 50  0001 C CNN
@@
 P 6000 4300
 AR Path="/63397143/634715DE" Ref="U?"  Part="1"
-AR Path="/63268641/634715DE" Ref="U14"  Part="1"
-F 0 "U14" H 6000 4625 50  0000 C CNN
+AR Path="/63268641/634715DE" Ref="U2"  Part="1"
+F 0 "U2" H 6000 4625 50  0000 C CNN
 F 1 "74LS10" H 6000 4534 50  0000 C CNN
 F 2 "Package_DIP:DIP-14_W7.62mm" H 6000 4300 50  0001 C CNN
@@
 	4300 4850 4150 4850
 $Comp
-L 74xx:74LS08 U11
+L 74xx:74LS08 U1
 U 1 1 634D51C8
 P 6000 2450
-F 0 "U11" H 6000 2775 50  0000 C CNN
+F 0 "U1" H 6000 2775 50  0000 C CNN
 F 1 "74LS08" H 6000 2684 50  0000 C CNN
 F 2 "Package_DIP:DIP-14_W7.62mm" H 6000 2450 50  0001 C CNN
@@
 SA1
 $Comp
-L 74xx:74LS08 U11
+L 74xx:74LS08 U1
 U 3 1 634E4497
 P 4600 4850
-F 0 "U11" H 4600 5175 50  0000 C CNN
+F 0 "U1" H 4600 5175 50  0000 C CNN
 F 1 "74LS08" H 4600 5084 50  0000 C CNN
 F 2 "Package_DIP:DIP-14_W7.62mm" H 4600 4850 50  0001 C CNN
@@
 AR Path="/63397143/634F2D94" Ref="U?"  Part="1"
 AR Path="/6341AE92/634F2D94" Ref="U?"  Part="1"
-AR Path="/63268641/634F2D94" Ref="U5"  Part="1"
-F 0 "U5" H 8100 4300 50  0000 C CNN
+AR Path="/63268641/634F2D94" Ref="U14"  Part="1"
+F 0 "U14" H 8100 4300 50  0000 C CNN
 F 1 "74LS163" H 8200 4200 50  0000 C CNN
 F 2 "Package_DIP:DIP-16_W7.62mm" H 8000 3550 50  0001 C CNN
@@
 	7350 3050 7500 3050
 $Comp
-L 74xx:74LS08 U11
+L 74xx:74LS08 U1
 U 2 1 635C87AA
 P 6800 3750
-F 0 "U11" H 6800 4075 50  0000 C CNN
+F 0 "U1" H 6800 4075 50  0000 C CNN
 F 1 "74LS08" H 6800 3984 50  0000 C CNN
 F 2 "Package_DIP:DIP-14_W7.62mm" H 6800 3750 50  0001 C CNN
@@
 SAMPLE_SEL_MAX_OUT
 $Comp
-L 74xx:74LS32 U15
+L 74xx:74LS32 U6
 U 4 1 637C3685
 P 6000 1850
-F 0 "U15" H 6000 2175 50  0000 C CNN
+F 0 "U6" H 6000 2175 50  0000 C CNN
 F 1 "74LS32" H 6000 2084 50  0000 C CNN
 F 2 "Package_DIP:DIP-14_W7.62mm" H 6000 1850 50  0001 C CNN
@@
 AR Path="/63397143/647C088C" Ref="#PWR?"  Part="1"
 AR Path="/6341AE92/647C088C" Ref="#PWR?"  Part="1"
-AR Path="/63268641/647C088C" Ref="#PWR?"  Part="1"
-F 0 "#PWR?" H 7350 3150 50  0001 C CNN
+AR Path="/63268641/647C088C" Ref="#PWR0117"  Part="1"
+F 0 "#PWR0117" H 7350 3150 50  0001 C CNN
 F 1 "GND" H 7500 3300 50  0000 C CNN
 F 2 "" H 7350 3400 50  0001 C CNN
