File: hardware/transmitter-retro/control-logic/shift.sch (KiCad schematic (older format))
At the start: 5 parts, among them U10 74LS08, U12 74LS00, U14 74LS10, U15 74LS32, U3 74LS162

Commit message: Add top level project Update part #s Update power sheets
Parts:
- U12: renamed from U3; value 74LS162 -> 74LS163
- renumbered U14 to U2, U10 to U4, U12 to U5, U15 to U6
Changed lines of the file:
@@
 P 4550 3450
 AR Path="/63470034" Ref="U?"  Part="1"
-AR Path="/632F1F43/63470034" Ref="U3"  Part="1"
+AR Path="/632F1F43/63470034" Ref="U12"  Part="1"
 AR Path="/63267F40/63470034" Ref="U?"  Part="1"
 AR Path="/6328016E/63470034" Ref="U?"  Part="1"
 AR Path="/63397143/63470034" Ref="U?"  Part="1"
-F 0 "U3" H 4650 4200 50  0000 C CNN
-F 1 "74LS162" H 4750 4100 50  0000 C CNN
+F 0 "U12" H 4650 4200 50  0000 C CNN
+F 1 "74LS163" H 4750 4100 50  0000 C CNN
 F 2 "Package_DIP:DIP-16_W7.62mm" H 4550 3450 50  0001 C CNN
 F 3 "http://www.ti.com/lit/gpn/sn74LS161" H 4550 3450 50  0001 C CNN
@@
 P 5800 3150
 AR Path="/63397143/6347005E" Ref="U?"  Part="1"
-AR Path="/632F1F43/6347005E" Ref="U15"  Part="1"
-F 0 "U15" H 5800 3475 50  0000 C CNN
+AR Path="/632F1F43/6347005E" Ref="U6"  Part="1"
+F 0 "U6" H 5800 3475 50  0000 C CNN
 F 1 "74LS32" H 5800 3384 50  0000 C CNN
 F 2 "Package_DIP:DIP-14_W7.62mm" H 5800 3150 50  0001 C CNN
@@
 P 6750 1950
 AR Path="/63397143/63470077" Ref="U?"  Part="2"
-AR Path="/632F1F43/63470077" Ref="U15"  Part="2"
-F 0 "U15" H 6750 2275 50  0000 C CNN
+AR Path="/632F1F43/63470077" Ref="U6"  Part="2"
+F 0 "U6" H 6750 2275 50  0000 C CNN
 F 1 "74LS32" H 6750 2184 50  0000 C CNN
 F 2 "Package_DIP:DIP-14_W7.62mm" H 6750 1950 50  0001 C CNN
@@
 	7150 1700 7250 1700
 $Comp
-L 74xx:74LS08 U10
+L 74xx:74LS08 U4
 U 2 1 6375104F
 P 4450 5050
-F 0 "U10" H 4450 5375 50  0000 C CNN
+F 0 "U4" H 4450 5375 50  0000 C CNN
 F 1 "74LS08" H 4450 5284 50  0000 C CNN
 F 2 "Package_DIP:DIP-14_W7.62mm" H 4450 5050 50  0001 C CNN
@@
 $EndComp
 $Comp
-L 74xx:74LS32 U15
+L 74xx:74LS32 U6
 U 3 1 6375129D
 P 7550 1600
-F 0 "U15" H 7550 1925 50  0000 C CNN
+F 0 "U6" H 7550 1925 50  0000 C CNN
 F 1 "74LS32" H 7550 1834 50  0000 C CNN
 F 2 "Package_DIP:DIP-14_W7.62mm" H 7550 1600 50  0001 C CNN
@@
 P 7600 4150
 AR Path="/637A582E" Ref="U?"  Part="3"
-AR Path="/632F1F43/637A582E" Ref="U14"  Part="3"
-F 0 "U14" H 7600 4475 50  0000 C CNN
+AR Path="/632F1F43/637A582E" Ref="U2"  Part="3"
+F 0 "U2" H 7600 4475 50  0000 C CNN
 F 1 "74LS10" H 7600 4384 50  0000 C CNN
 F 2 "Package_DIP:DIP-14_W7.62mm" H 7600 4150 50  0001 C CNN
@@
 	5400 3650 5550 3650
 $Comp
-L 74xx:74LS08 U10
+L 74xx:74LS08 U4
 U 4 1 637AB56A
 P 6750 3650
-AR Path="/632F1F43/637AB56A" Ref="U10"  Part="4"
+AR Path="/632F1F43/637AB56A" Ref="U4"  Part="4"
 AR Path="/637AB56A" Ref="U?"  Part="4"
-F 0 "U10" H 6750 3975 50  0000 C CNN
+F 0 "U4" H 6750 3975 50  0000 C CNN
 F 1 "74LS08" H 6750 3884 50  0000 C CNN
 F 2 "Package_DIP:DIP-14_W7.62mm" H 6750 3650 50  0001 C CNN
@@
 	7150 3650 8650 3650
 $Comp
-L 74xx:74LS00 U12
+L 74xx:74LS00 U5
 U 3 1 637C2048
 P 5850 3750
-F 0 "U12" H 5850 4075 50  0000 C CNN
+F 0 "U5" H 5850 4075 50  0000 C CNN
 F 1 "74LS00" H 5850 3984 50  0000 C CNN
 F 2 "Package_DIP:DIP-14_W7.62mm" H 5850 3750 50  0001 C CNN
@@
 $EndComp
 $Comp
-L 74xx:74LS00 U12
+L 74xx:74LS00 U5
 U 4 1 637C2099
 P 6750 4700
-F 0 "U12" H 6750 5025 50  0000 C CNN
+F 0 "U5" H 6750 5025 50  0000 C CNN
 F 1 "74LS00" H 6750 4934 50  0000 C CNN
 F 2 "Package_DIP:DIP-14_W7.62mm" H 6750 4700 50  0001 C CNN
@@
 $EndComp
 $Comp
-L 74xx:74LS08 U10
+L 74xx:74LS08 U4
 U 3 1 637C22D8
 P 5850 2600
-F 0 "U10" H 5850 2925 50  0000 C CNN
+F 0 "U4" H 5850 2925 50  0000 C CNN
 F 1 "74LS08" H 5850 2834 50  0000 C CNN
 F 2 "Package_DIP:DIP-14_W7.62mm" H 5850 2600 50  0001 C CNN
