File: hardware/transmitter-retro/control-logic/control-logic.sch (KiCad schematic (older format))
At the start: 1 part

Commit message: Add top level project Update part #s Update power sheets
Parts:
- gave numbers to parts that had none: 1
Changed lines of the file:
@@
 	4500 1950 4500 4150
 $Comp
-L power:GND #PWR?
+L power:GND #PWR0101
 U 1 1 6475E09B
 P 6150 4750
-AR Path="/6475E09B" Ref="#PWR?"  Part="1"
+AR Path="/6475E09B" Ref="#PWR0101"  Part="1"
 AR Path="/632F1F43/6475E09B" Ref="#PWR?"  Part="1"
 AR Path="/63267F40/6475E09B" Ref="#PWR?"  Part="1"
 AR Path="/64755962/6475E09B" Ref="#PWR?"  Part="1"
-F 0 "#PWR?" H 6150 4500 50  0001 C CNN
+F 0 "#PWR0101" H 6150 4500 50  0001 C CNN
 F 1 "GND" H 6300 4650 50  0000 C CNN
 F 2 "" H 6150 4750 50  0001 C CNN
@@
 	6150 4650 6150 4750
 $Comp
-L power:GND #PWR?
-U 1 1 6475E0A6
-P 5450 4750
-AR Path="/6475E0A6" Ref="#PWR?"  Part="1"
-AR Path="/632F1F43/6475E0A6" Ref="#PWR?"  Part="1"
-AR Path="/63267F40/6475E0A6" Ref="#PWR?"  Part="1"
-AR Path="/64755962/6475E0A6" Ref="#PWR?"  Part="1"
-F 0 "#PWR?" H 5450 4500 50  0001 C CNN
-F 1 "GND" H 5600 4650 50  0000 C CNN
-F 2 "" H 5450 4750 50  0001 C CNN
-F 3 "" H 5450 4750 50  0001 C CNN
-	1    5450 4750
-	1    0    0    -1
-$EndComp
-Wire Wire Line
-	5450 4750 5450 4650
-Wire Wire Line
-	5450 4550 5550 4550
-Wire Wire Line
-	5550 4650 5450 4650
-Connection ~ 5450 4650
-Wire Wire Line
-	5450 4650 5450 4550
-$Comp
-L power:+5V #PWR?
+L power:+5V #PWR0102
 U 1 1 6475E0B1
 P 6150 2650
-AR Path="/6475E0B1" Ref="#PWR?"  Part="1"
+AR Path="/6475E0B1" Ref="#PWR0102"  Part="1"
 AR Path="/632F1F43/6475E0B1" Ref="#PWR?"  Part="1"
 AR Path="/63267F40/6475E0B1" Ref="#PWR?"  Part="1"
 AR Path="/64755962/6475E0B1" Ref="#PWR?"  Part="1"
-F 0 "#PWR?" H 6150 2500 50  0001 C CNN
+F 0 "#PWR0102" H 6150 2500 50  0001 C CNN
 F 1 "+5V" H 6165 2823 50  0000 C CNN
 F 2 "" H 6150 2650 50  0001 C CNN
@@
 	6150 2750 6150 2650
 $Comp
-L power:+5V #PWR?
+L power:+5V #PWR0103
 U 1 1 6475E0BC
 P 5450 2650
-AR Path="/6475E0BC" Ref="#PWR?"  Part="1"
+AR Path="/6475E0BC" Ref="#PWR0103"  Part="1"
 AR Path="/632F1F43/6475E0BC" Ref="#PWR?"  Part="1"
 AR Path="/63267F40/6475E0BC" Ref="#PWR?"  Part="1"
 AR Path="/64755962/6475E0BC" Ref="#PWR?"  Part="1"
-F 0 "#PWR?" H 5450 2500 50  0001 C CNN
+F 0 "#PWR0103" H 5450 2500 50  0001 C CNN
 F 1 "+5V" H 5465 2823 50  0000 C CNN
 F 2 "" H 5450 2650 50  0001 C CNN
@@
 ~FRAME_RESET
 NoConn ~ 6050 3850
-NoConn ~ 6050 4350
-NoConn ~ 6050 4450
 NoConn ~ 5550 2950
 NoConn ~ 5550 3050
@@
 P 5750 3650
 AR Path="/63267F40/6475E0DF" Ref="J?"  Part="1"
-AR Path="/6475E0DF" Ref="J?"  Part="1"
+AR Path="/6475E0DF" Ref="J1"  Part="1"
 AR Path="/64755962/6475E0DF" Ref="J?"  Part="1"
-F 0 "J?" H 5800 4767 50  0000 C CNN
+F 0 "J1" H 5800 4767 50  0000 C CNN
 F 1 "Expansion" H 5800 4676 50  0000 C CNN
 F 2 "Connector_PinHeader_2.54mm:PinHeader_2x20_P2.54mm_Vertical" H 5750 3650 50  0001 C CNN
@@
 NoConn ~ 6050 2950
 NoConn ~ 6050 3050
+Wire Wire Line
+	6050 4350 6150 4350
+Wire Wire Line
+	6150 4350 6150 4450
+Connection ~ 6150 4550
+Wire Wire Line
+	6050 4450 6150 4450
+Connection ~ 6150 4450
+Wire Wire Line
+	6150 4450 6150 4550
+NoConn ~ 5550 4550
+NoConn ~ 5550 4650
 $EndSCHEMATC

Commit message: Prototype and PCB layout for core Prototype and PCB layout for demo Prototype and PCB layout for control-eprom Move display design forward Refactor control-dmx to dmx Update expansion connector on all boards Add test suites Add tx-retro readme Cleanup
Parts:
- removed J1: Expansion, Connector_PinHeader_2.54mm:PinHeader_2x20_P2.54mm_Vertical, symbol Connector_Generic:Conn_02x20_Odd_Even
- added J?: Expansion, Connector_PinHeader_2.54mm:PinHeader_2x20_P2.54mm_Vertical, symbol Connector_Generic:Conn_02x20_Odd_Even
Connections:
- net labels added: CLK_RX, CLK_SAMPLE, D0, D1, D2, D3, D4, D5, D6, D7, DATA_RX, DATA_SHIFT, SAMPLE_COUNT, SPD_HI, SPD_LO, SPD_MID, ~BUS_ACK, ~BUS_REQ, ~CLK_FST, ~CLK_SLO, ~CLK_STEP, ~SAMPLE_OVERRIDE
- net labels removed: CLK_FAST, CLK_SLOW
- wire segments 74 -> 70
- no-connect marks 20 -> 0
