File: hardware/transmitter-retro/control-logic/reset.sch (KiCad schematic (older format))
At the start: 4 parts, among them U11 74LS08, U14 74LS10, U6 74LS74, U7 74LS161

Commit message: Add top level project Update part #s Update power sheets
Parts:
- U7: value 74LS161 -> 74LS163
- U8: renamed from U6; footprint (none) -> Package_DIP:DIP-14_W7.62mm
- renumbered U11 to U1, U14 to U2
Changed lines of the file:
@@
 AR Path="/6341AE92/635901C0" Ref="U7"  Part="1"
 F 0 "U7" H 6050 4400 50  0000 C CNN
-F 1 "74LS161" H 6150 4300 50  0000 C CNN
+F 1 "74LS163" H 6150 4300 50  0000 C CNN
 F 2 "Package_DIP:DIP-16_W7.62mm" H 5950 3650 50  0001 C CNN
 F 3 "http://www.ti.com/lit/gpn/sn74LS161" H 5950 3650 50  0001 C CNN
@@
 AR Path="/63268641/637970D0" Ref="U?"  Part="2"
 AR Path="/637970D0" Ref="U?"  Part="2"
-AR Path="/6341AE92/637970D0" Ref="U14"  Part="2"
-F 0 "U14" H 6950 3975 50  0000 C CNN
+AR Path="/6341AE92/637970D0" Ref="U2"  Part="2"
+F 0 "U2" H 6950 3975 50  0000 C CNN
 F 1 "74LS10" H 6950 3884 50  0000 C CNN
 F 2 "Package_DIP:DIP-14_W7.62mm" H 6950 3650 50  0001 C CNN
@@
 AR Path="/6328016E/647B1D12" Ref="#PWR?"  Part="1"
 AR Path="/63397143/647B1D12" Ref="#PWR?"  Part="1"
-AR Path="/6341AE92/647B1D12" Ref="#PWR?"  Part="1"
-F 0 "#PWR?" H 5300 3250 50  0001 C CNN
+AR Path="/6341AE92/647B1D12" Ref="#PWR0118"  Part="1"
+F 0 "#PWR0118" H 5300 3250 50  0001 C CNN
 F 1 "GND" H 5450 3400 50  0000 C CNN
 F 2 "" H 5300 3500 50  0001 C CNN
@@
 $EndComp
 $Comp
-L 74xx:74LS74 U6
+L 74xx:74LS74 U8
 U 1 1 647B5D21
 P 4150 3950
-F 0 "U6" H 4300 4300 50  0000 C CNN
+F 0 "U8" H 4300 4300 50  0000 C CNN
 F 1 "74LS74" H 4300 4200 50  0000 C CNN
-F 2 "" H 4150 3950 50  0001 C CNN
+F 2 "Package_DIP:DIP-14_W7.62mm" H 4150 3950 50  0001 C CNN
 F 3 "74xx/74hc_hct74.pdf" H 4150 3950 50  0001 C CNN
 	1    4150 3950
@@
 AR Path="/6328016E/647B99E7" Ref="#PWR?"  Part="1"
 AR Path="/63397143/647B99E7" Ref="#PWR?"  Part="1"
-AR Path="/6341AE92/647B99E7" Ref="#PWR?"  Part="1"
-F 0 "#PWR?" H 4150 3400 50  0001 C CNN
+AR Path="/6341AE92/647B99E7" Ref="#PWR0123"  Part="1"
+F 0 "#PWR0123" H 4150 3400 50  0001 C CNN
 F 1 "+5V" H 4165 3723 50  0000 C CNN
 F 2 "" H 4150 3550 50  0001 C CNN
@@
 AR Path="/63422E72" Ref="U?"  Part="4"
 AR Path="/6BB77A68/63422E72" Ref="U?"  Part="4"
-AR Path="/6341AE92/63422E72" Ref="U11"  Part="4"
-F 0 "U11" H 3450 4275 50  0000 C CNN
+AR Path="/6341AE92/63422E72" Ref="U1"  Part="4"
+F 0 "U1" H 3450 4275 50  0000 C CNN
 F 1 "74LS08" H 3450 4184 50  0000 C CNN
 F 2 "Package_DIP:DIP-14_W7.62mm" H 3450 3950 50  0001 C CNN

Commit message: Prototype and PCB layout for core Prototype and PCB layout for demo Prototype and PCB layout for control-eprom Move display design forward Refactor control-dmx to dmx Update expansion connector on all boards Add test suites Add tx-retro readme Cleanup
Parts:
- added JP? (x4): SolderJumper_2_Open, symbol Jumper:SolderJumper_2_Open
Other:
- note added: "JP5-8"
Changed lines of the file:
@@
 Wire Wire Line
 	2800 3850 3150 3850
+$Comp
+L Jumper:SolderJumper_2_Open JP?
+U 1 1 64593377
+P 3950 2400
+AR Path="/634170D9/64593377" Ref="JP?"  Part="1"
+AR Path="/6341AE92/64593377" Ref="JP?"  Part="1"
+F 0 "JP?" H 3950 2605 50  0001 C CNN
+F 1 "SolderJumper_2_Open" H 3950 2513 50  0001 C CNN
+F 2 "" H 3950 2400 50  0001 C CNN
+F 3 "~" H 3950 2400 50  0001 C CNN
+	1    3950 2400
+	1    0    0    -1
+$EndComp
+$Comp
+L Jumper:SolderJumper_2_Open JP?
+U 1 1 6459337D
+P 3950 2500
+AR Path="/634170D9/6459337D" Ref="JP?"  Part="1"
+AR Path="/6341AE92/6459337D" Ref="JP?"  Part="1"
+F 0 "JP?" H 3950 2705 50  0001 C CNN
+F 1 "SolderJumper_2_Open" H 3950 2613 50  0001 C CNN
+F 2 "" H 3950 2500 50  0001 C CNN
+F 3 "~" H 3950 2500 50  0001 C CNN
+	1    3950 2500
+	1    0    0    -1
+$EndComp
+$Comp
+L Jumper:SolderJumper_2_Open JP?
+U 1 1 64593383
+P 3950 2600
+AR Path="/634170D9/64593383" Ref="JP?"  Part="1"
+AR Path="/6341AE92/64593383" Ref="JP?"  Part="1"
+F 0 "JP?" H 3950 2805 50  0001 C CNN
+F 1 "SolderJumper_2_Open" H 3950 2713 50  0001 C CNN
+F 2 "" H 3950 2600 50  0001 C CNN
+F 3 "~" H 3950 2600 50  0001 C CNN
+	1    3950 2600
+	1    0    0    -1
+$EndComp
+$Comp
+L Jumper:SolderJumper_2_Open JP?
+U 1 1 64593389
+P 3950 2700
+AR Path="/634170D9/64593389" Ref="JP?"  Part="1"
+AR Path="/6341AE92/64593389" Ref="JP?"  Part="1"
+F 0 "JP?" H 3950 2905 50  0001 C CNN
+F 1 "SolderJumper_2_Open" H 3950 2813 50  0001 C CNN
+F 2 "" H 3950 2700 50  0001 C CNN
+F 3 "~" H 3950 2700 50  0001 C CNN
+	1    3950 2700
+	1    0    0    -1
+$EndComp
+Text Notes 3850 2300 0    50   ~ 0
+JP5-8
 $EndSCHEMATC
