File: hardware/transmitter-retro/core/clock.sch (KiCad schematic (older format))
At the start: 23 parts, among them U1 556, U14 74LS04, U15 74LS74, U16 74LS74, U18 74LS32, U19 74LS08, U2 74LS163

Commit message: Add top level project Update part #s Update power sheets
Parts:
- U2: renamed from U?; footprint (none) -> Package_DIP:DIP-16_W7.62mm
- gave numbers to parts that had none: 1
- renumbered R11 to R10, R8 to R11, R9 to R7, R10 to R8, R11 to R9, U2 to U3, U16 to U4, U15 to U5, U19 to U6, U18 to U7, U14 to U8
Changed lines of the file:
@@
 	7000 1650 7150 1650
 $Comp
-L 74xx:74LS04 U14
+L 74xx:74LS04 U8
 U 3 1 63357AA3
 P 4650 7400
-F 0 "U14" H 4650 7717 50  0000 C CNN
+F 0 "U8" H 4650 7717 50  0000 C CNN
 F 1 "74LS04" H 4650 7626 50  0000 C CNN
 F 2 "Package_DIP:DIP-14_W7.62mm" H 4650 7400 50  0001 C CNN
@@
 	1700 6850 1700 6800
 $Comp
-L 74xx:74LS04 U14
+L 74xx:74LS04 U8
 U 4 1 6329DA61
 P 9600 2350
-F 0 "U14" H 9600 2667 50  0000 C CNN
+F 0 "U8" H 9600 2667 50  0000 C CNN
 F 1 "74LS04" H 9600 2576 50  0000 C CNN
 F 2 "Package_DIP:DIP-14_W7.62mm" H 9600 2350 50  0001 C CNN
@@
 Slow/Adj Clock
 $Comp
-L 74xx:74LS74 U15
+L 74xx:74LS74 U5
 U 2 1 63588395
 P 5450 6350
-F 0 "U15" H 5600 6700 50  0000 C CNN
+F 0 "U5" H 5600 6700 50  0000 C CNN
 F 1 "74LS74" H 5650 6600 50  0000 C CNN
 F 2 "Package_DIP:DIP-14_W7.62mm" H 5450 6350 50  0001 C CNN
@@
 $EndComp
 $Comp
-L 74xx:74LS74 U15
+L 74xx:74LS74 U5
 U 1 1 63588326
 P 3200 6700
-F 0 "U15" H 3350 7050 50  0000 C CNN
+F 0 "U5" H 3350 7050 50  0000 C CNN
 F 1 "74LS74" H 3400 6950 50  0000 C CNN
 F 2 "Package_DIP:DIP-14_W7.62mm" H 3200 6700 50  0001 C CNN
@@
 	3200 6300 3200 6150
 $Comp
-L 74xx:74LS32 U18
+L 74xx:74LS32 U7
 U 3 1 63653D6B
 P 3900 6900
-F 0 "U18" H 3900 7225 50  0000 C CNN
+F 0 "U7" H 3900 7225 50  0000 C CNN
 F 1 "74LS32" H 3900 7134 50  0000 C CNN
 F 2 "Package_DIP:DIP-14_W7.62mm" H 3900 6900 50  0001 C CNN
@@
 	3550 7000 3550 7150
 $Comp
-L 74xx:74LS32 U18
+L 74xx:74LS32 U7
 U 4 1 63665A56
 P 6250 6350
-F 0 "U18" H 6250 6675 50  0000 C CNN
+F 0 "U7" H 6250 6675 50  0000 C CNN
 F 1 "74LS32" H 6250 6584 50  0000 C CNN
 F 2 "Package_DIP:DIP-14_W7.62mm" H 6250 6350 50  0001 C CNN
@@
 	8700 2350 8700 4650
 $Comp
-L 74xx:74LS08 U19
+L 74xx:74LS08 U6
 U 2 1 6376957E
 P 4650 6350
-F 0 "U19" H 4650 6675 50  0000 C CNN
+F 0 "U6" H 4650 6675 50  0000 C CNN
 F 1 "74LS08" H 4650 6584 50  0000 C CNN
 F 2 "Package_DIP:DIP-14_W7.62mm" H 4650 6350 50  0001 C CNN
@@
 	5450 5900 6700 5900
 $Comp
-L 74xx:74LS08 U19
+L 74xx:74LS08 U6
 U 3 1 63A6E069
 P 5350 7300
-F 0 "U19" H 5350 7625 50  0000 C CNN
+F 0 "U6" H 5350 7625 50  0000 C CNN
 F 1 "74LS08" H 5350 7534 50  0000 C CNN
 F 2 "Package_DIP:DIP-14_W7.62mm" H 5350 7300 50  0001 C CNN
@@
 $EndComp
 $Comp
-L 74xx:74LS04 U14
+L 74xx:74LS04 U8
 U 6 1 63A6E114
 P 6050 7300
-F 0 "U14" H 6050 7617 50  0000 C CNN
+F 0 "U8" H 6050 7617 50  0000 C CNN
 F 1 "74LS04" H 6050 7526 50  0000 C CNN
 F 2 "Package_DIP:DIP-14_W7.62mm" H 6050 7300 50  0001 C CNN
@@
 AR Path="/63399130" Ref="U?"  Part="1"
 AR Path="/63268641/63399130" Ref="U?"  Part="1"
-AR Path="/63268613/63399130" Ref="U2"  Part="1"
-F 0 "U2" H 8150 2900 50  0000 C CNN
+AR Path="/63268613/63399130" Ref="U3"  Part="1"
+F 0 "U3" H 8150 2900 50  0000 C CNN
 F 1 "74LS163" H 8250 2800 50  0000 C CNN
 F 2 "Package_DIP:DIP-16_W7.62mm" H 8050 2150 50  0001 C CNN
@@
 P 1700 7000
 AR Path="/6347633F" Ref="R?"  Part="1"
-AR Path="/63268613/6347633F" Ref="R8"  Part="1"
-F 0 "R8" H 1550 7050 50  0000 L CNN
+AR Path="/63268613/6347633F" Ref="R11"  Part="1"
+F 0 "R11" H 1550 7050 50  0000 L CNN
 F 1 "10k" H 1500 6950 50  0000 L CNN
 F 2 "Resistor_THT:R_Axial_DIN0207_L6.3mm_D2.5mm_P10.16mm_Horizontal" V 1740 6990 50  0001 C CNN
@@
 	1700 7150 1700 7250
 $Comp
-L 74xx:74LS08 U19
+L 74xx:74LS08 U6
 U 4 1 63500ED3
 P 2200 7150
-F 0 "U19" H 2200 7475 50  0000 C CNN
+F 0 "U6" H 2200 7475 50  0000 C CNN
 F 1 "74LS08" H 2200 7384 50  0000 C CNN
 F 2 "Package_DIP:DIP-14_W7.62mm" H 2200 7150 50  0001 C CNN
@@
 P 1850 6250
 AR Path="/6352ADE7" Ref="R?"  Part="1"
-AR Path="/63268613/6352ADE7" Ref="R11"  Part="1"
-F 0 "R11" H 1650 6300 50  0000 L CNN
+AR Path="/63268613/6352ADE7" Ref="R10"  Part="1"
+F 0 "R10" H 1650 6300 50  0000 L CNN
 F 1 "10k" H 1650 6200 50  0000 L CNN
 F 2 "Resistor_THT:R_Axial_DIN0207_L6.3mm_D2.5mm_P10.16mm_Horizontal" V 1890 6240 50  0001 C CNN
@@
 ~CLK_FAST_OUT
 $Comp
-L 74xx:74LS74 U16
+L 74xx:74LS74 U4
 U 1 1 6394DF68
 P 3500 4100
-F 0 "U16" H 3650 4450 50  0000 C CNN
+F 0 "U4" H 3650 4450 50  0000 C CNN
 F 1 "74LS74" H 3700 4350 50  0000 C CNN
 F 2 "Package_DIP:DIP-14_W7.62mm" H 3500 4100 50  0001 C CNN
@@
 $EndComp
 $Comp
-L 74xx:74LS74 U16
+L 74xx:74LS74 U4
 U 2 1 6394E00D
 P 4650 4100
-F 0 "U16" H 4850 4450 50  0000 C CNN
+F 0 "U4" H 4850 4450 50  0000 C CNN
 F 1 "74LS74" H 4850 4350 50  0000 C CNN
 F 2 "Package_DIP:DIP-14_W7.62mm" H 4650 4100 50  0001 C CNN
@@
 P 5550 1450
 AR Path="/63A0E79F" Ref="R?"  Part="1"
-AR Path="/63268613/63A0E79F" Ref="R?"  Part="1"
-F 0 "R?" H 5350 1500 50  0000 L CNN
+AR Path="/63268613/63A0E79F" Ref="R6"  Part="1"
+F 0 "R6" H 5350 1500 50  0000 L CNN
 F 1 "10k" H 5350 1400 50  0000 L CNN
 F 2 "Resistor_THT:R_Axial_DIN0207_L6.3mm_D2.5mm_P10.16mm_Horizontal" V 5590 1440 50  0001 C CNN
 F 3 "~" H 5550 1450 50  0001 C CNN
 	1    5550 1450
-	-1   0    0    1
-$EndComp
-$Comp
-L 74xx:74LS151 U?
+	-1   0    0    -1
+$EndComp
+$Comp
+L 74xx:74LS151 U2
 U 1 1 64301AD7
 P 6500 2250
-F 0 "U?" H 6650 3100 50  0000 C CNN
+F 0 "U2" H 6650 3100 50  0000 C CNN
 F 1 "74LS151" H 6700 3000 50  0000 C CNN
-F 2 "" H 6500 2250 50  0001 C CNN
+F 2 "Package_DIP:DIP-16_W7.62mm" H 6500 2250 50  0001 C CNN
 F 3 "http://www.ti.com/lit/gpn/sn74LS151" H 6500 2250 50  0001 C CNN
 	1    6500 2250
@@
 P 2150 3650
 AR Path="/63536C51" Ref="R?"  Part="1"
-AR Path="/63268613/63536C51" Ref="R10"  Part="1"
-F 0 "R10" H 1950 3700 50  0000 L CNN
+AR Path="/63268613/63536C51" Ref="R8"  Part="1"
+F 0 "R8" H 1950 3700 50  0000 L CNN
 F 1 "10k" H 1950 3600 50  0000 L CNN
 F 2 "Resistor_THT:R_Axial_DIN0207_L6.3mm_D2.5mm_P10.16mm_Horizontal" V 2190 3640 50  0001 C CNN
@@
 P 1750 3650
 AR Path="/63540EEA" Ref="R?"  Part="1"
-AR Path="/63268613/63540EEA" Ref="R9"  Part="1"
-F 0 "R9" H 1550 3700 50  0000 L CNN
+AR Path="/63268613/63540EEA" Ref="R7"  Part="1"
+F 0 "R7" H 1550 3700 50  0000 L CNN
 F 1 "10k" H 1550 3600 50  0000 L CNN
 F 2 "Resistor_THT:R_Axial_DIN0207_L6.3mm_D2.5mm_P10.16mm_Horizontal" V 1790 3640 50  0001 C CNN
@@
 AR Path="/6359368B" Ref="#PWR?"  Part="1"
 AR Path="/64132440/6359368B" Ref="#PWR?"  Part="1"
-AR Path="/63268613/6359368B" Ref="#PWR?"  Part="1"
-F 0 "#PWR?" H 4000 1100 50  0001 C CNN
+AR Path="/63268613/6359368B" Ref="#PWR0104"  Part="1"
+F 0 "#PWR0104" H 4000 1100 50  0001 C CNN
 F 1 "+5V" H 4015 1423 50  0000 C CNN
 F 2 "" H 4000 1250 50  0001 C CNN
@@
 AR Path="/635936D0" Ref="#PWR?"  Part="1"
 AR Path="/64132440/635936D0" Ref="#PWR?"  Part="1"
-AR Path="/63268613/635936D0" Ref="#PWR?"  Part="1"
-F 0 "#PWR?" H 2150 3250 50  0001 C CNN
+AR Path="/63268613/635936D0" Ref="#PWR0107"  Part="1"
+F 0 "#PWR0107" H 2150 3250 50  0001 C CNN
 F 1 "+5V" H 2165 3573 50  0000 C CNN
 F 2 "" H 2150 3400 50  0001 C CNN
@@
 AR Path="/63593715" Ref="#PWR?"  Part="1"
 AR Path="/64132440/63593715" Ref="#PWR?"  Part="1"
-AR Path="/63268613/63593715" Ref="#PWR?"  Part="1"
-F 0 "#PWR?" H 3500 3650 50  0001 C CNN
+AR Path="/63268613/63593715" Ref="#PWR0109"  Part="1"
+F 0 "#PWR0109" H 3500 3650 50  0001 C CNN
 F 1 "+5V" H 3515 3973 50  0000 C CNN
 F 2 "" H 3500 3800 50  0001 C CNN
@@
 AR Path="/6359DDFE" Ref="#PWR?"  Part="1"
 AR Path="/64132440/6359DDFE" Ref="#PWR?"  Part="1"
-AR Path="/63268613/6359DDFE" Ref="#PWR?"  Part="1"
-F 0 "#PWR?" H 4650 3650 50  0001 C CNN
+AR Path="/63268613/6359DDFE" Ref="#PWR0110"  Part="1"
+F 0 "#PWR0110" H 4650 3650 50  0001 C CNN
 F 1 "+5V" H 4665 3973 50  0000 C CNN
 F 2 "" H 4650 3800 50  0001 C CNN
@@
 AR Path="/63762EEC" Ref="#PWR?"  Part="1"
 AR Path="/64132440/63762EEC" Ref="#PWR?"  Part="1"
-AR Path="/63268613/63762EEC" Ref="#PWR?"  Part="1"
-F 0 "#PWR?" H 1850 5950 50  0001 C CNN
+AR Path="/63268613/63762EEC" Ref="#PWR0112"  Part="1"
+F 0 "#PWR0112" H 1850 5950 50  0001 C CNN
 F 1 "+5V" H 1865 6273 50  0000 C CNN
 F 2 "" H 1850 6100 50  0001 C CNN
@@
 AR Path="/6376307D" Ref="#PWR?"  Part="1"
 AR Path="/64132440/6376307D" Ref="#PWR?"  Part="1"
-AR Path="/63268613/6376307D" Ref="#PWR?"  Part="1"
-F 0 "#PWR?" H 1700 6650 50  0001 C CNN
+AR Path="/63268613/6376307D" Ref="#PWR0117"  Part="1"
+F 0 "#PWR0117" H 1700 6650 50  0001 C CNN
 F 1 "+5V" H 1715 6973 50  0000 C CNN
 F 2 "" H 1700 6800 50  0001 C CNN
@@
 AR Path="/637630C2" Ref="#PWR?"  Part="1"
 AR Path="/64132440/637630C2" Ref="#PWR?"  Part="1"
-AR Path="/63268613/637630C2" Ref="#PWR?"  Part="1"
-F 0 "#PWR?" H 3200 6000 50  0001 C CNN
+AR Path="/63268613/637630C2" Ref="#PWR0125"  Part="1"
+F 0 "#PWR0125" H 3200 6000 50  0001 C CNN
 F 1 "+5V" H 3215 6323 50  0000 C CNN
 F 2 "" H 3200 6150 50  0001 C CNN
@@
 P 6500 3350
 AR Path="/63268641/637631D3" Ref="#PWR?"  Part="1"
-AR Path="/63268613/637631D3" Ref="#PWR?"  Part="1"
-F 0 "#PWR?" H 6500 3100 50  0001 C CNN
+AR Path="/63268613/637631D3" Ref="#PWR0126"  Part="1"
+F 0 "#PWR0126" H 6500 3100 50  0001 C CNN
 F 1 "GND" H 6505 3177 50  0000 C CNN
 F 2 "" H 6500 3350 50  0001 C CNN
@@
 P 2500 3650
 AR Path="/639E1B8D" Ref="R?"  Part="1"
-AR Path="/63268613/639E1B8D" Ref="R11"  Part="1"
-F 0 "R11" H 2300 3700 50  0000 L CNN
+AR Path="/63268613/639E1B8D" Ref="R9"  Part="1"
+F 0 "R9" H 2300 3700 50  0000 L CNN
 F 1 "10k" H 2300 3600 50  0000 L CNN
 F 2 "Resistor_THT:R_Axial_DIN0207_L6.3mm_D2.5mm_P10.16mm_Horizontal" V 2540 3640 50  0001 C CNN

Commit message: Prototype and PCB layout for core Prototype and PCB layout for demo Prototype and PCB layout for control-eprom Move display design forward Refactor control-dmx to dmx Update expansion connector on all boards Add test suites Add tx-retro readme Cleanup
Parts:
- removed C31: 1uF, Capacitor_THT:C_Rect_L4.6mm_W2.0mm_P2.50mm_MKS02_FKP02, symbol Device:C_Small
- removed C32: .001uF, Capacitor_THT:C_Rect_L4.6mm_W2.0mm_P2.50mm_MKS02_FKP02, symbol Device:C_Small
- removed C33, C34: .01uF, Capacitor_THT:C_Rect_L4.6mm_W2.0mm_P2.50mm_MKS02_FKP02, symbol Device:C_Small
- removed R10, R11, R6, R7, R8, R9: 10k, Resistor_THT:R_Axial_DIN0207_L6.3mm_D2.5mm_P10.16mm_Horizontal, symbol Device:R_US
- removed R2: 100, Resistor_THT:R_Axial_DIN0207_L6.3mm_D2.5mm_P10.16mm_Horizontal, symbol Device:R_US
- removed R3: 1M, Resistor_THT:R_Axial_DIN0207_L6.3mm_D2.5mm_P10.16mm_Horizontal, symbol Device:R_US
- removed R4: 1k, Resistor_THT:R_Axial_DIN0207_L6.3mm_D2.5mm_P10.16mm_Horizontal, symbol Device:R_US
- removed R5: 3.3k, Resistor_THT:R_Axial_DIN0207_L6.3mm_D2.5mm_P10.16mm_Horizontal, symbol Device:R_US
- removed U1: 556, Silicon-Standard:DIP14, symbol transmitter-pro:556
- removed U2: 74LS151, Package_DIP:DIP-16_W7.62mm, symbol 74xx:74LS151
- removed U4, U5: 74LS74, Package_DIP:DIP-14_W7.62mm, symbol 74xx:74LS74
- removed U6: 74LS08, Package_DIP:DIP-14_W7.62mm, symbol 74xx:74LS08
- removed U7: 74LS32, Package_DIP:DIP-14_W7.62mm, symbol 74xx:74LS32
- removed U8: 74LS04, Package_DIP:DIP-14_W7.62mm, symbol 74xx:74LS04
- added U10: 74LS04, Package_DIP:DIP-14_W7.62mm, symbol 74xx:74LS04
- R1: value 2.2k -> 10k
- renumbered U3 to U1
Connections:
- net labels added: CLK_SAMPLE_IN
- net labels removed: CLK_EXT, CLK_EXT_IN, CLK_FAST, CLK_SAMPLE_OUT, CLK_SLOW, CLK_STEP, CLK_TX, S0, S1, SPD_LO, SPD_WIPER, ~CLK_EXT_SEL_IN, ~CLK_FAST_IN, ~CLK_FAST_OUT, ~CLK_SLOW_IN, ~CLK_SLOW_OUT, ~CLK_STEP_INA, ~CLK_STEP_INB
- wire segments 199 -> 27
- no-connect marks 13 -> 4
Other:
- note added: "CLK_TX\n\nCLK_RX"
- note added: "CLK_TX\n\nCLK_SAMPLE"
- note added: "Clock Divide"
- note removed: "CLK_EXT_SEL sets S0=S1=0, selecting\nthe CLK_EXT input to feed the clock."
- note removed: "Clock Multiplexer:\nS0=0,S1=0: External\nS0=1,S1=0: Fast\nS0=0,S1=1: Slow/Adj\nS0=1,S1=1: Step"
- note removed: "Create a reset\npulse from the\nCLK_STEP inputs"
- note removed: "Enable CLK_STEP while\nCLK_TX is high, then low."
- note removed: "Fast Clock"
- note removed: "S0 and S1 are set on the rising edge\nof the fast clock."
- note removed: "Send CLK_FAST\nto CLK_STEP"
- note removed: "Slow/Adj Clock"
- note removed: "Step Clock\nStarts a cycle of CLK_TX from hi to lo to hi."
- note removed: "To external\npotentiometer"
