File: hardware/transmitter-retro/core/shift.sch (KiCad schematic (older format))
At the start: 3 parts, among them U18 74LS32, U19 74LS08, U8 74LS165

Commit message: Add top level project Update part #s Update power sheets
Parts:
- renumbered U8 to U10, U19 to U6, U18 to U7
Changed lines of the file:
@@
 P 6350 4450
 AR Path="/633286AB" Ref="U?"  Part="1"
-AR Path="/632F1F43/633286AB" Ref="U19"  Part="1"
-F 0 "U19" H 6350 4775 50  0000 C CNN
+AR Path="/632F1F43/633286AB" Ref="U6"  Part="1"
+F 0 "U6" H 6350 4775 50  0000 C CNN
 F 1 "74LS08" H 6350 4684 50  0000 C CNN
 F 2 "Package_DIP:DIP-14_W7.62mm" H 6350 4450 50  0001 C CNN
@@
 P 7150 4650
 AR Path="/633286B2" Ref="U?"  Part="1"
-AR Path="/632F1F43/633286B2" Ref="U18"  Part="1"
-F 0 "U18" H 7150 4975 50  0000 C CNN
+AR Path="/632F1F43/633286B2" Ref="U7"  Part="1"
+F 0 "U7" H 7150 4975 50  0000 C CNN
 F 1 "74LS32" H 7150 4884 50  0000 C CNN
 F 2 "Package_DIP:DIP-14_W7.62mm" H 7150 4650 50  0001 C CNN
@@
 P 5450 3350
 AR Path="/633286A4" Ref="U?"  Part="1"
-AR Path="/632F1F43/633286A4" Ref="U8"  Part="1"
-F 0 "U8" H 5550 4200 50  0000 C CNN
+AR Path="/632F1F43/633286A4" Ref="U10"  Part="1"
+F 0 "U10" H 5550 4200 50  0000 C CNN
 F 1 "74LS165" H 5650 4100 50  0000 C CNN
 F 2 "Package_DIP:DIP-16_W7.62mm" H 5450 3350 50  0001 C CNN
@@
 Wire Wire Line
 	7550 4000 6050 4000
+Connection ~ 6050 4000
+Wire Wire Line
+	6050 4000 6050 2750
 Wire Bus Line
 	4750 2100 4750 3450
-Connection ~ 6050 4000
-Wire Wire Line
-	6050 4000 6050 2750
 $EndSCHEMATC

Commit message: Update part numbers Swap out input connector footprint Placement tweaks
Parts:
- added U17: ULN2003A, Package_DIP:DIP-16_W7.62mm, symbol Transistor_Array:ULN2003A
Connections:
- net labels added: ~CLK_OUT, ~DATA_OUT
- net labels removed: CLK_OUT, DATA_OUT
- wire segments 34 -> 36
- no-connect marks 1 -> 12
Changed lines of the file:
@@
 	6050 4350 6050 4000
 Wire Bus Line
-	4850 2000 7650 2000
-Text HLabel 7650 2000 2    50   Input ~ 0
+	4850 2000 8550 2000
+Text HLabel 8550 2000 2    50   Input ~ 0
 D[0..7]
 Text HLabel 7650 4650 2    50   Input ~ 0
@@
 Text HLabel 3700 1250 0    50   Input ~ 0
 ~CLK_SLOW_IN
-Text HLabel 7650 1050 2    50   Input ~ 0
+Text HLabel 8550 1050 2    50   Input ~ 0
 ~CLK_STEP_OUT
 Text HLabel 3700 1050 0    50   Input ~ 0
@@
 Text HLabel 3700 1150 0    50   Input ~ 0
 ~CLK_FAST_IN
-Text HLabel 7650 1250 2    50   Input ~ 0
+Text HLabel 8550 1250 2    50   Input ~ 0
 ~CLK_SLOW_OUT
-Text HLabel 7650 1150 2    50   Input ~ 0
+Text HLabel 8550 1150 2    50   Input ~ 0
 ~CLK_FAST_OUT
-Text HLabel 7650 1400 2    50   Input ~ 0
+Text HLabel 8550 1400 2    50   Input ~ 0
 CLK_RX_OUT
 Text HLabel 3700 1400 0    50   Input ~ 0
 CLK_RX_IN
 Wire Wire Line
-	7650 1400 7550 1400
+	8550 1400 7550 1400
 Wire Wire Line
-	3700 1150 7650 1150
+	3700 1150 8550 1150
 Wire Wire Line
-	3700 1250 7650 1250
+	3700 1250 8550 1250
 Wire Wire Line
-	7650 1050 3700 1050
-Text HLabel 7650 4750 2    50   Input ~ 0
-DATA_OUT
-Text HLabel 7650 1500 2    50   Input ~ 0
-CLK_OUT
-Wire Wire Line
-	7650 4750 7550 4750
-Wire Wire Line
-	7550 4750 7550 4650
+	8550 1050 3700 1050
+Text HLabel 8550 2900 2    50   Input ~ 0
+~DATA_OUT
+Text HLabel 8550 2800 2    50   Input ~ 0
+~CLK_OUT
 Connection ~ 7550 4650
 Wire Wire Line
 	7550 4650 7650 4650
-Wire Wire Line
-	7650 1500 7550 1500
-Wire Wire Line
-	7550 1500 7550 1400
 Connection ~ 7550 1400
 Wire Wire Line
@@
 Wire Wire Line
 	3700 3950 4950 3950
-Text HLabel 7550 4000 2    50   Input ~ 0
+Text HLabel 8600 4000 2    50   Input ~ 0
 DATA_SHIFT_OUT
 Wire Wire Line
-	7550 4000 6050 4000
+	8600 4000 6050 4000
 Connection ~ 6050 4000
 Wire Wire Line
 	6050 4000 6050 2750
+Wire Wire Line
+	7550 4650 7550 2900
+Wire Wire Line
+	7550 2900 7650 2900
+Wire Wire Line
+	7550 2800 7650 2800
+Wire Wire Line
+	7550 1400 7550 2800
+$Comp
+L Transistor_Array:ULN2003A U17
+U 1 1 63EEB811
+P 8050 3000
+F 0 "U17" H 8050 3667 50  0000 C CNN
+F 1 "ULN2003A" H 8050 3576 50  0000 C CNN
+F 2 "Package_DIP:DIP-16_W7.62mm" H 8100 2450 50  0001 L CNN
+F 3 "http://www.ti.com/lit/ds/symlink/uln2003a.pdf" H 8150 2800 50  0001 C CNN
+	1    8050 3000
+	1    0    0    -1
+$EndComp
+NoConn ~ 7650 3000
+NoConn ~ 7650 3100
+NoConn ~ 7650 3200
+NoConn ~ 7650 3300
+NoConn ~ 7650 3400
+NoConn ~ 8450 2600
+NoConn ~ 8450 3000
+NoConn ~ 8450 3100
+NoConn ~ 8450 3200
+NoConn ~ 8450 3300
+NoConn ~ 8450 3400
+Wire Wire Line
+	8450 2800 8550 2800
+Wire Wire Line
+	8450 2900 8550 2900
+$Comp
+L power:GND #PWR?
+U 1 1 63EF339F
+P 8050 3600
+AR Path="/6841E790/63EF339F" Ref="#PWR?"  Part="1"
+AR Path="/63EF339F" Ref="#PWR?"  Part="1"
+AR Path="/632F1F43/63EF339F" Ref="#PWR0146"  Part="1"
+F 0 "#PWR0146" H 8050 3350 50  0001 C CNN
+F 1 "GND" H 8200 3500 50  0000 C CNN
+F 2 "" H 8050 3600 50  0001 C CNN
+F 3 "" H 8050 3600 50  0001 C CNN
+	1    8050 3600
+	1    0    0    -1
+$EndComp
 Wire Bus Line
 	4750 2100 4750 3450

Commit message: Prototype and PCB layout for core Prototype and PCB layout for demo Prototype and PCB layout for control-eprom Move display design forward Refactor control-dmx to dmx Update expansion connector on all boards Add test suites Add tx-retro readme Cleanup
Parts:
- removed U17: ULN2003A, Package_DIP:DIP-16_W7.62mm, symbol Transistor_Array:ULN2003A
- removed U6: 74LS08, Package_DIP:DIP-14_W7.62mm, symbol 74xx:74LS08
- removed U7: 74LS32, Package_DIP:DIP-14_W7.62mm, symbol 74xx:74LS32
- added U11: 74LS32, Package_DIP:DIP-14_W7.62mm, symbol 74xx:74LS32
- added U12: 74LS08, Package_DIP:DIP-14_W7.62mm, symbol 74xx:74LS08
- renumbered U10 to U2
Connections:
- net labels removed: ~CLK_FAST_IN, ~CLK_FAST_OUT, ~CLK_OUT, ~CLK_SLOW_IN, ~CLK_SLOW_OUT, ~CLK_STEP_IN, ~CLK_STEP_OUT, ~DATA_OUT
- wire segments 36 -> 26
- no-connect marks 12 -> 1
Other:
- note added: ""The ’LS165A is a 8-bit serial shift registers that shift the data\nin the direction of (D0) toward (D7) when clocked."\n\nWhen shifting, the Q7 output first see the data from D7, then D6, then D5,\netc... Q7 output will see the data from D0 on the eighth clock pulse on CP.\n\nIn DMX, the least significant bit (LSB) is sent first, which equates to D0.\nTherefore, the D0 but from the bus is connec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"
- note added: "Data Shift"
- note added: "The data sent to DATA_RX_OUT is a combination of the shoft register output\nand the data from DATA_FIXED_IN. DATA_FIXED_IN is always feed to DATA_RX_OUT,\nso any value is has is seen at DATA_RX_OUT. For the portions of the packet that need\nto be 1, DATA_FIXED_IN is 1; for all other portions it is 0. \n\nSHIFT_TRANSMIT_IN combines with the shift register output using an AND gate so the\nshift reg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"
- note removed: "Shift\nRegister"
