File: hardware/transmitter-retro/core/core.sch (KiCad schematic (older format))
At the start: 3 parts, among them J1 Input, J2 Output, J4 Expansion

Commit message: Add top level project Update part #s Update power sheets
Connections:
- net labels added: CLK_RX_OUT, ~CLK_EXT_SEL
- wire segments 161 -> 162
Changed lines of the file:
@@
 F12 "~CLK_FAST_OUT" I R 4200 4300 50
 F13 "CLK_EXT_IN" I R 4200 4000 50
-F14 "~CLK_EXT_SEL_IN" I R 4200 3900 50
+F14 "~CLK_EXT_SEL_IN" I R 4200 4600 50
 $EndSheet
 $Sheet
@@
 AR Path="/6BB77683/645E6BD8" Ref="J?"  Part="1"
 AR Path="/645E6BD8" Ref="J2"  Part="1"
-F 0 "J2" H 9080 5842 50  0000 L CNN
-F 1 "Output" H 9080 5751 50  0000 L CNN
+F 0 "J2" H 9100 5750 50  0000 L CNN
+F 1 "Output" H 9100 5850 50  0000 L CNN
 F 2 "Connector_PinHeader_2.54mm:PinHeader_1x03_P2.54mm_Horizontal" H 9000 5800 50  0001 C CNN
 F 3 "~" H 9000 5800 50  0001 C CNN
@@
 Wire Wire Line
 	6200 4600 6200 4700
-$Comp
-L power:GND #PWR0147
-U 1 1 635885B3
-P 5500 4700
-AR Path="/635885B3" Ref="#PWR0147"  Part="1"
-AR Path="/632F1F43/635885B3" Ref="#PWR?"  Part="1"
-AR Path="/63267F40/635885B3" Ref="#PWR?"  Part="1"
-F 0 "#PWR0147" H 5500 4450 50  0001 C CNN
-F 1 "GND" H 5650 4600 50  0000 C CNN
-F 2 "" H 5500 4700 50  0001 C CNN
-F 3 "" H 5500 4700 50  0001 C CNN
-	1    5500 4700
-	1    0    0    -1
-$EndComp
-Wire Wire Line
-	5500 4700 5500 4600
-Wire Wire Line
-	5500 4500 5600 4500
-Wire Wire Line
-	5600 4600 5500 4600
-Connection ~ 5500 4600
-Wire Wire Line
-	5500 4600 5500 4500
 $Comp
 L power:+5V #PWR0148
@@
 	6800 5900 7750 5900
 NoConn ~ 6100 3800
-NoConn ~ 6100 4300
-NoConn ~ 6100 4400
 Wire Wire Line
 	6100 4200 7050 4200
@@
 	8050 3000 7350 3000
 Connection ~ 7350 3000
+Text Label 8000 5700 0    50   ~ 0
+DATA_RX
+Text Label 8000 5900 0    50   ~ 0
+CLK_RX_OUT
+Wire Wire Line
+	6100 4300 6200 4300
+Wire Wire Line
+	6200 4300 6200 4400
+Connection ~ 6200 4500
+Wire Wire Line
+	6100 4400 6200 4400
+Connection ~ 6200 4400
+Wire Wire Line
+	6200 4400 6200 4500
+Text Label 5100 4600 0    50   ~ 0
+~CLK_EXT_SEL
+Wire Wire Line
+	4200 4600 5600 4600
+NoConn ~ 5600 4500
+NoConn ~ 10800 1300
 Wire Bus Line
 	6950 2150 6950 5100

Commit message: Update part numbers Swap out input connector footprint Placement tweaks
Parts:
- J1: footprint Connector_PinHeader_2.54mm:PinHeader_2x08_P2.54mm_Vertical -> Connector_IDC:IDC-Header_2x08_P2.54mm_Horizontal
Changed lines of the file:
@@
 F 0 "J1" H 3250 1967 50  0000 C CNN
 F 1 "Input" H 3250 1876 50  0000 C CNN
-F 2 "Connector_PinHeader_2.54mm:PinHeader_2x08_P2.54mm_Vertical" H 3200 1450 50  0001 C CNN
+F 2 "Connector_IDC:IDC-Header_2x08_P2.54mm_Horizontal" H 3200 1450 50  0001 C CNN
 F 3 "~" H 3200 1450 50  0001 C CNN
 	1    3200 1450
@@
 F15 "~CLK_STEP_IN" I R 6800 5700 50
 F16 "~SHIFT_ENABLE_IN" I R 6800 5500 50
-F17 "DATA_OUT" I L 4850 6000 50
-F18 "CLK_OUT" I L 4850 6100 50
-F19 "DATA_SHIFT_OUT" I R 6800 6000 50
+F17 "DATA_SHIFT_OUT" I R 6800 6000 50
+F18 "~DATA_OUT" I L 4850 6100 50
+F19 "~CLK_OUT" I L 4850 6000 50
 $EndSheet
 Wire Wire Line

Commit message: Prototype and PCB layout for core Prototype and PCB layout for demo Prototype and PCB layout for control-eprom Move display design forward Refactor control-dmx to dmx Update expansion connector on all boards Add test suites Add tx-retro readme Cleanup
Parts:
- added U13: ULN2003A, Package_DIP:DIP-16_W7.62mm, symbol Transistor_Array:ULN2003A
- renumbered J4 to J1, J1 to J3
Connections:
- net labels added: CLK_SAMPLE, DIM1, DIM2, DIM3, DIM4, D[0..7], SPD_HI, SPD_LO, SPD_MID, SPD_WIPER, ~CLK_FST, ~CLK_SLO, ~CLK_STEP, ~CLOCK, ~DATA, ~HWD_DT
- net labels removed: CLK_EXT, CLK_FAST, CLK_RX_OUT, CLK_SLOW, SAMPLE_REF, ~CLK_EXT_SEL
- wire segments 162 -> 154
- no-connect marks 4 -> 8

Commit message: Rev 1.1 - Value labels - 74LS06 led driver
Parts:
- removed U13: ULN2003A, Package_DIP:DIP-16_W7.62mm, symbol Transistor_Array:ULN2003A
- added U13: 74LS06, Package_DIP:DIP-14_W7.62mm, symbol 74xx:74LS06
Connections:
- wire segments 154 -> 144
- no-connect marks 8 -> 1
Changed lines of the file:
@@
 Text Label 8800 4200 0    50   ~ 0
 CLK_RX
-NoConn ~ 10800 1300
-NoConn ~ 9050 3300
-NoConn ~ 9050 3200
-NoConn ~ 9050 3100
-NoConn ~ 9050 3000
-NoConn ~ 9050 2900
-NoConn ~ 9050 2500
-$Comp
-L Transistor_Array:ULN2003A U?
-U 1 1 6431D1B4
-P 8650 2900
-AR Path="/632F1F43/6431D1B4" Ref="U?"  Part="1"
-AR Path="/6431D1B4" Ref="U13"  Part="1"
-F 0 "U13" H 8650 3567 50  0000 C CNN
-F 1 "ULN2003A" H 8650 3476 50  0000 C CNN
-F 2 "Package_DIP:DIP-16_W7.62mm" H 8700 2350 50  0001 L CNN
-F 3 "http://www.ti.com/lit/ds/symlink/uln2003a.pdf" H 8750 2700 50  0001 C CNN
-	1    8650 2900
-	1    0    0    -1
-$EndComp
 Wire Wire Line
 	7650 4000 7650 5000
@@
 	7250 3300 6100 3300
 Connection ~ 7650 4000
-Wire Wire Line
-	7650 4000 7650 2800
 Connection ~ 7750 4200
 Wire Wire Line
 	2900 1600 1600 1600
 Wire Wire Line
-	3950 750  9550 750
+	3950 750  9000 750
 Wire Wire Line
 	3950 750  3950 1700
 Wire Wire Line
-	3850 650  9650 650
-Wire Wire Line
-	9650 650  9650 2700
+	3850 650  9100 650
 Wire Wire Line
 	3850 650  3850 1600
@@
 $Comp
 L power:GND #PWR?
-U 1 1 648DFAC9
-P 8650 3500
-AR Path="/6841E790/648DFAC9" Ref="#PWR?"  Part="1"
-AR Path="/648DFAC9" Ref="#PWR0104"  Part="1"
-F 0 "#PWR0104" H 8650 3250 50  0001 C CNN
-F 1 "GND" H 8655 3327 50  0000 C CNN
-F 2 "" H 8650 3500 50  0001 C CNN
-F 3 "" H 8650 3500 50  0001 C CNN
-	1    8650 3500
-	1    0    0    -1
-$EndComp
-$Comp
-L power:GND #PWR?
 U 1 1 648DFADC
 P 10050 5900
@@
 	1    0    0    -1
 $EndComp
-$Comp
-L power:GND #PWR?
-U 1 1 648DFAEF
-P 8150 3500
-AR Path="/6841E790/648DFAEF" Ref="#PWR?"  Part="1"
-AR Path="/648DFAEF" Ref="#PWR0110"  Part="1"
-F 0 "#PWR0110" H 8150 3250 50  0001 C CNN
-F 1 "GND" H 8155 3327 50  0000 C CNN
-F 2 "" H 8150 3500 50  0001 C CNN
-F 3 "" H 8150 3500 50  0001 C CNN
-	1    8150 3500
-	1    0    0    -1
-$EndComp
-Wire Wire Line
-	8150 3500 8150 3300
-Wire Wire Line
-	8150 2900 8250 2900
-Wire Wire Line
-	8250 3000 8150 3000
-Connection ~ 8150 3000
-Wire Wire Line
-	8150 3000 8150 2900
-Wire Wire Line
-	8250 3100 8150 3100
-Connection ~ 8150 3100
-Wire Wire Line
-	8150 3100 8150 3000
-Wire Wire Line
-	8250 3200 8150 3200
-Connection ~ 8150 3200
-Wire Wire Line
-	8150 3200 8150 3100
-Wire Wire Line
-	8250 3300 8150 3300
-Connection ~ 8150 3300
-Wire Wire Line
-	8150 3300 8150 3200
 Entry Bus Bus
 	4300 2400 4400 2300
 Text Label 6650 2300 0    50   ~ 0
 D[0..7]
-Wire Wire Line
-	9550 2800 9050 2800
-Wire Wire Line
-	9550 750  9550 2800
-Wire Wire Line
-	7750 2700 8250 2700
-Wire Wire Line
-	7750 2700 7750 4200
-Wire Wire Line
-	8250 2800 7650 2800
-Wire Wire Line
-	9050 2700 9650 2700
 Wire Wire Line
 	5600 2900 2100 2900
@@
 	7500 2050 7500 2300
 Connection ~ 7500 2300
+Wire Wire Line
+	8050 1750 7650 1750
+Wire Wire Line
+	7650 1750 7650 4000
+Wire Wire Line
+	8650 1750 9000 1750
+Wire Wire Line
+	8050 2300 7750 2300
+Wire Wire Line
+	8650 2300 9100 2300
+$Comp
+L 74xx:74LS06 U13
+U 1 1 652D4C06
+P 8350 2300
+F 0 "U13" H 8350 2617 50  0000 C CNN
+F 1 "74LS06" H 8350 2526 50  0000 C CNN
+F 2 "Package_DIP:DIP-14_W7.62mm" H 8350 2300 50  0001 C CNN
+F 3 "http://www.ti.com/lit/gpn/sn74LS06" H 8350 2300 50  0001 C CNN
+	1    8350 2300
+	1    0    0    -1
+$EndComp
+$Comp
+L 74xx:74LS06 U13
+U 2 1 652D4C67
+P 8350 1750
+F 0 "U13" H 8350 2067 50  0000 C CNN
+F 1 "74LS06" H 8350 1976 50  0000 C CNN
+F 2 "Package_DIP:DIP-14_W7.62mm" H 8350 1750 50  0001 C CNN
+F 3 "http://www.ti.com/lit/gpn/sn74LS06" H 8350 1750 50  0001 C CNN
+	2    8350 1750
+	1    0    0    -1
+$EndComp
+Wire Wire Line
+	9000 750  9000 1750
+Wire Wire Line
+	7750 2300 7750 4200
+Wire Wire Line
+	9100 2300 9100 650
 Wire Bus Line
 	7500 2300 7500 5900
