File: hardware/transmitter-retro/core/power.sch (KiCad schematic (older format))
At the start: 41 parts, among them J3 Power, U14 74LS04, U15 74LS74, U16 74LS74, U18 74LS32, U19 74LS08, U21 LM339

Commit message: Add top level project Update part #s Update power sheets
Parts:
- removed U? (x3): 74LS32, symbol 74xx:74LS32
- U7, U9: renamed from U?; footprint (none) -> Package_DIP:DIP-14_W7.62mm
- gave numbers to parts that had none: 1
- renumbered C21 to C20, C29 to C21, C30 to C22, U21 to U17, U15 to U4, U16 to U5, U19 to U6, U18 to U7, U14 to U8
Connections:
- wire segments 125 -> 119
- no-connect marks 0 -> 3
Other:
- moved on the sheet: U17E

Commit message: Update part numbers Swap out input connector footprint Placement tweaks
Parts:
- removed C19, C20: .01uF, Capacitor_THT:C_Rect_L4.6mm_W2.0mm_P2.50mm_MKS02_FKP02, symbol Device:C
- U16: renamed from U17; footprint Package_DIP:DIP-14_W7.62mm -> Package_DIP:DIP-16_W7.62mm
Connections:
- wire segments 119 -> 109
Changed lines of the file:
@@
 L Device:C C?
 U 1 1 714E82A9
-P 8050 4950
+P 2950 6800
 AR Path="/5F2B3F8A/714E82A9" Ref="C?"  Part="1"
 AR Path="/5F2B505F/714E82A9" Ref="C?"  Part="1"
 AR Path="/6BB77A68/714E82A9" Ref="C17"  Part="1"
 AR Path="/64132440/6413313E/714E82A9" Ref="C?"  Part="1"
-F 0 "C17" H 8165 4996 50  0000 L CNN
-F 1 ".01uF" H 8165 4905 50  0000 L CNN
-F 2 "Capacitor_THT:C_Rect_L4.6mm_W2.0mm_P2.50mm_MKS02_FKP02" H 8088 4800 50  0001 C CNN
-F 3 "~" H 8050 4950 50  0001 C CNN
-	1    8050 4950
+F 0 "C17" H 3065 6846 50  0000 L CNN
+F 1 ".01uF" H 3065 6755 50  0000 L CNN
+F 2 "Capacitor_THT:C_Rect_L4.6mm_W2.0mm_P2.50mm_MKS02_FKP02" H 2988 6650 50  0001 C CNN
+F 3 "~" H 2950 6800 50  0001 C CNN
+	1    2950 6800
 	1    0    0    -1
 $EndComp
@@
 L Device:C C?
 U 1 1 681CF588
-P 8500 4950
+P 3400 6800
 AR Path="/5F2B3F8A/681CF588" Ref="C?"  Part="1"
 AR Path="/5F2B505F/681CF588" Ref="C?"  Part="1"
 AR Path="/6BB77A68/681CF588" Ref="C18"  Part="1"
 AR Path="/64132440/6413313E/681CF588" Ref="C?"  Part="1"
-F 0 "C18" H 8615 4996 50  0000 L CNN
-F 1 ".01uF" H 8615 4905 50  0000 L CNN
-F 2 "Capacitor_THT:C_Rect_L4.6mm_W2.0mm_P2.50mm_MKS02_FKP02" H 8538 4800 50  0001 C CNN
-F 3 "~" H 8500 4950 50  0001 C CNN
-	1    8500 4950
-	1    0    0    -1
-$EndComp
-$Comp
-L Device:C C?
-U 1 1 681CF58E
-P 9000 4950
-AR Path="/5F2B3F8A/681CF58E" Ref="C?"  Part="1"
-AR Path="/5F2B505F/681CF58E" Ref="C?"  Part="1"
-AR Path="/6BB77A68/681CF58E" Ref="C19"  Part="1"
-AR Path="/64132440/6413313E/681CF58E" Ref="C?"  Part="1"
-F 0 "C19" H 9115 4996 50  0000 L CNN
-F 1 ".01uF" H 9115 4905 50  0000 L CNN
-F 2 "Capacitor_THT:C_Rect_L4.6mm_W2.0mm_P2.50mm_MKS02_FKP02" H 9038 4800 50  0001 C CNN
-F 3 "~" H 9000 4950 50  0001 C CNN
-	1    9000 4950
-	1    0    0    -1
-$EndComp
-$Comp
-L Device:C C?
-U 1 1 714E82AD
-P 9450 4950
-AR Path="/5F2B3F8A/714E82AD" Ref="C?"  Part="1"
-AR Path="/5F2B505F/714E82AD" Ref="C?"  Part="1"
-AR Path="/6BB77A68/714E82AD" Ref="C20"  Part="1"
-AR Path="/64132440/6413313E/714E82AD" Ref="C?"  Part="1"
-F 0 "C20" H 9565 4996 50  0000 L CNN
-F 1 ".01uF" H 9565 4905 50  0000 L CNN
-F 2 "Capacitor_THT:C_Rect_L4.6mm_W2.0mm_P2.50mm_MKS02_FKP02" H 9488 4800 50  0001 C CNN
-F 3 "~" H 9450 4950 50  0001 C CNN
-	1    9450 4950
-	1    0    0    -1
-$EndComp
-Wire Wire Line
-	9450 4800 9450 4700
-Wire Wire Line
-	9000 4800 9000 4700
-Connection ~ 9000 4700
-Wire Wire Line
-	9000 4700 9450 4700
-Wire Wire Line
-	8500 4800 8500 4700
-Wire Wire Line
-	8500 4700 8750 4700
-Wire Wire Line
-	8050 4800 8050 4700
-Wire Wire Line
-	8050 4700 8500 4700
-Wire Wire Line
-	9450 5100 9450 5200
-Wire Wire Line
-	9000 5100 9000 5200
-Connection ~ 9000 5200
-Wire Wire Line
-	9000 5200 9450 5200
-Wire Wire Line
-	8500 5100 8500 5200
-Wire Wire Line
-	8500 5200 8750 5200
-Wire Wire Line
-	8050 5100 8050 5200
-Wire Wire Line
-	8050 5200 8500 5200
-$Comp
-L power:GND #PWR0217
-U 1 1 714E82B1
-P 8750 5300
-AR Path="/6BB77A68/714E82B1" Ref="#PWR0217"  Part="1"
-AR Path="/64132440/6413313E/714E82B1" Ref="#PWR0217"  Part="1"
-F 0 "#PWR0217" H 8750 5050 50  0001 C CNN
-F 1 "GND" H 8755 5127 50  0000 C CNN
-F 2 "" H 8750 5300 50  0001 C CNN
-F 3 "" H 8750 5300 50  0001 C CNN
-	1    8750 5300
-	1    0    0    -1
-$EndComp
-Connection ~ 8500 5200
-Connection ~ 8500 4700
-Wire Wire Line
-	8750 4700 8750 4600
-Connection ~ 8750 4700
-Wire Wire Line
-	8750 4700 9000 4700
-$Comp
-L power:+5V #PWR0218
-U 1 1 681CF5E5
-P 8750 4600
-AR Path="/6BB77A68/681CF5E5" Ref="#PWR0218"  Part="1"
-AR Path="/64132440/6413313E/681CF5E5" Ref="#PWR0218"  Part="1"
-F 0 "#PWR0218" H 8750 4450 50  0001 C CNN
-F 1 "+5V" H 8765 4773 50  0000 C CNN
-F 2 "" H 8750 4600 50  0001 C CNN
-F 3 "" H 8750 4600 50  0001 C CNN
-	1    8750 4600
-	1    0    0    -1
-$EndComp
-Wire Wire Line
-	8750 5300 8750 5200
-Connection ~ 8750 5200
-Wire Wire Line
-	8750 5200 9000 5200
+F 0 "C18" H 3515 6846 50  0000 L CNN
+F 1 ".01uF" H 3515 6755 50  0000 L CNN
+F 2 "Capacitor_THT:C_Rect_L4.6mm_W2.0mm_P2.50mm_MKS02_FKP02" H 3438 6650 50  0001 C CNN
+F 3 "~" H 3400 6800 50  0001 C CNN
+	1    3400 6800
+	1    0    0    -1
+$EndComp
+Wire Wire Line
+	3400 6650 3400 6550
+Wire Wire Line
+	2950 6650 2950 6550
+Wire Wire Line
+	2950 6550 3400 6550
+Wire Wire Line
+	3400 6950 3400 7050
+Wire Wire Line
+	2950 6950 2950 7050
+Wire Wire Line
+	2950 7050 3400 7050
+Connection ~ 3400 7050
 $Comp
 L Device:CP1 C22
@@
 P 3950 4350
 AR Path="/63268641/63467635" Ref="U?"  Part="5"
-AR Path="/6BB77A68/63467635" Ref="U17"  Part="5"
-F 0 "U17" H 3908 4396 50  0000 L CNN
+AR Path="/6BB77A68/63467635" Ref="U16"  Part="5"
+F 0 "U16" H 3908 4396 50  0000 L CNN
 F 1 "LM339" H 3908 4305 50  0000 L CNN
-F 2 "Package_DIP:DIP-14_W7.62mm" H 3900 4450 50  0001 C CNN
+F 2 "Package_DIP:DIP-16_W7.62mm" H 3900 4450 50  0001 C CNN
 F 3 "http://www.ti.com/lit/ds/symlink/lm339.pdf" H 4000 4550 50  0001 C CNN
 	5    3950 4350
@@
 	1    0    0    -1
 $EndComp
-Text HLabel 2950 6550 2    50   Input ~ 0
+Text HLabel 3900 6550 2    50   Input ~ 0
 +5V_OUT
-Text HLabel 2950 7050 2    50   Input ~ 0
+Text HLabel 3900 7050 2    50   Input ~ 0
 GND_OUT
 Wire Wire Line
@@
 Wire Wire Line
 	4800 2450 4800 2650
+Wire Wire Line
+	3400 7050 3900 7050
+Connection ~ 3400 6550
+Wire Wire Line
+	3400 6550 3900 6550
+Connection ~ 2950 6550
+Connection ~ 2950 7050
 $EndSCHEMATC

Commit message: Prototype and PCB layout for core Prototype and PCB layout for demo Prototype and PCB layout for control-eprom Move display design forward Refactor control-dmx to dmx Update expansion connector on all boards Add test suites Add tx-retro readme Cleanup
Parts:
- removed C13, C14, C15, C16: .01uF, Capacitor_THT:C_Rect_L4.6mm_W2.0mm_P2.50mm_MKS02_FKP02, symbol Device:C
- removed U4, U5: 74LS74, Package_DIP:DIP-14_W7.62mm, symbol 74xx:74LS74
- removed unit 2 of U7
- removed unit 5 of U8
- removed U9: 74LS02, Package_DIP:DIP-14_W7.62mm, symbol 74xx:74LS02
- added J5: Power, Connectors:POWER_JACK_PTH_BREAD, symbol CrazyGiraffe_DMXDemonstrator:POWER_JACKPTH_BREAD
- added unit 2 of U11
- added unit 4 of U11
- added unit 1 of U11
- added unit 4 of U12
- added U9: TLV2772CP, Package_DIP:DIP-8_W7.62mm, symbol CrazyGiraffe_DMXDemonstrator:TLV2772CP
- C13: renamed from C21; value CP1 -> 10uF
- C14: renamed from C22; value CP1 -> 10uF
- U8: renamed from U16; footprint Package_DIP:DIP-16_W7.62mm -> Package_DIP:DIP-14_W7.62mm
- renumbered C17 to C15, C18 to C16, J3 to J4, U8 to U10, U7 to U11, U6 to U12
Connections:
- wire segments 109 -> 110
- no-connect marks 3 -> 5
Other:
- moved on the sheet: U8E

Commit message: Rev 1.1 - Value labels - 74LS06 led driver
Parts:
- added U13: 74LS06, Package_DIP:DIP-14_W7.62mm, symbol 74xx:74LS06
- C1, C10, C11, C12, C15, C16, C2, C3, C4, C5, C6, C7, C8, C9: value .01uF -> 0.1uF
Connections:
- wire segments 110 -> 117
- no-connect marks 5 -> 9
