File: hardware/transmitter-retro/core/sample.sch (KiCad schematic (older format))
At the start: 14 parts, among them U10 74LS163, U11 TLC7524CN, U14 74LS04, U21 LM339, U7 74LS373, U9 74LS163

Commit message: Add top level project Update part #s Update power sheets
Parts:
- U11: renamed from U?; footprint (none) -> Package_DIP:DIP-16_W7.62mm
- U15: renamed from U7; footprint (none) -> Package_DIP:DIP-20_W7.62mm
- U9: renamed from U?; footprint (none) -> Package_DIP:DIP-14_W7.62mm
- gave numbers to parts that had none: 4
- renumbered U9 to U12, U10 to U13, U11 to U16, U21 to U17, U14 to U8
Changed lines of the file:
@@
 $Descr A4 11693 8268
 encoding utf-8
-Sheet 7 6
+Sheet 6 6
 Title "DMX Demonstrator - Transmitter-Pro (DMX-TX3)"
 Date "2022-09-30"
@@
 P 2200 2050
 AR Path="/63304670" Ref="U?"  Part="1"
-AR Path="/63268641/63304670" Ref="U21"  Part="1"
-F 0 "U21" H 2200 1750 50  0000 C CNN
+AR Path="/63268641/63304670" Ref="U17"  Part="1"
+F 0 "U17" H 2200 1750 50  0000 C CNN
 F 1 "LM339" H 2200 1850 50  0000 C CNN
 F 2 "Package_DIP:DIP-14_W7.62mm" H 2150 2150 50  0001 C CNN
@@
 P 2200 4050
 AR Path="/63304677" Ref="U?"  Part="4"
-AR Path="/63268641/63304677" Ref="U21"  Part="4"
-F 0 "U21" H 2200 3750 50  0000 C CNN
+AR Path="/63268641/63304677" Ref="U17"  Part="4"
+F 0 "U17" H 2200 3750 50  0000 C CNN
 F 1 "LM339" H 2200 3850 50  0000 C CNN
 F 2 "Package_DIP:DIP-14_W7.62mm" H 2150 4150 50  0001 C CNN
@@
 P 2200 2700
 AR Path="/6330467E" Ref="U?"  Part="2"
-AR Path="/63268641/6330467E" Ref="U21"  Part="2"
-F 0 "U21" H 2200 2400 50  0000 C CNN
+AR Path="/63268641/6330467E" Ref="U17"  Part="2"
+F 0 "U17" H 2200 2400 50  0000 C CNN
 F 1 "LM339" H 2200 2500 50  0000 C CNN
 F 2 "Package_DIP:DIP-14_W7.62mm" H 2150 2800 50  0001 C CNN
@@
 P 2200 3400
 AR Path="/63304685" Ref="U?"  Part="3"
-AR Path="/63268641/63304685" Ref="U21"  Part="3"
-F 0 "U21" H 2200 3100 50  0000 C CNN
+AR Path="/63268641/63304685" Ref="U17"  Part="3"
+F 0 "U17" H 2200 3100 50  0000 C CNN
 F 1 "LM339" H 2200 3200 50  0000 C CNN
 F 2 "Package_DIP:DIP-14_W7.62mm" H 2150 3500 50  0001 C CNN
@@
 P 8000 3750
 AR Path="/633046D2" Ref="U?"  Part="1"
-AR Path="/63268641/633046D2" Ref="U10"  Part="1"
-F 0 "U10" H 8100 4500 50  0000 C CNN
+AR Path="/63268641/633046D2" Ref="U13"  Part="1"
+F 0 "U13" H 8100 4500 50  0000 C CNN
 F 1 "74LS163" H 8200 4400 50  0000 C CNN
 F 2 "Package_DIP:DIP-16_W7.62mm" H 8000 3750 50  0001 C CNN
@@
 P 6300 3750
 AR Path="/6330471C" Ref="U?"  Part="1"
-AR Path="/63268641/6330471C" Ref="U9"  Part="1"
-F 0 "U9" H 6400 4500 50  0000 C CNN
+AR Path="/63268641/6330471C" Ref="U12"  Part="1"
+F 0 "U12" H 6400 4500 50  0000 C CNN
 F 1 "74LS163" H 6500 4400 50  0000 C CNN
 F 2 "Package_DIP:DIP-16_W7.62mm" H 6300 3750 50  0001 C CNN
@@
 	6700 1100 6950 1100
 $Comp
-L transmitter-retro:TLC7524CN U11
+L transmitter-retro:TLC7524CN U16
 U 1 1 634200B5
 P 6300 1500
-F 0 "U11" H 6100 2150 50  0000 C CNN
+F 0 "U16" H 6100 2150 50  0000 C CNN
 F 1 "TLC7524CN" H 6000 2050 50  0000 C CNN
 F 2 "Package_DIP:DIP-16_W7.62mm" H 6300 1500 50  0001 C CNN
@@
 	5750 3950 5800 3950
 $Comp
-L 74xx:74LS373 U7
+L 74xx:74LS373 U15
 U 1 1 638DE1BD
 P 9550 3750
-F 0 "U7" H 9700 4500 50  0000 C CNN
+F 0 "U15" H 9700 4500 50  0000 C CNN
 F 1 "74LS373" H 9800 4400 50  0000 C CNN
-F 2 "" H 9550 3750 50  0001 C CNN
+F 2 "Package_DIP:DIP-20_W7.62mm" H 9550 3750 50  0001 C CNN
 F 3 "http://www.ti.com/lit/gpn/sn74LS373" H 9550 3750 50  0001 C CNN
 	1    9550 3750
@@
 AR Path="/63268613/63A2F4D2" Ref="U?"  Part="1"
 AR Path="/639E280B/63A2F4D2" Ref="U?"  Part="1"
-AR Path="/63268641/63A2F4D2" Ref="U14"  Part="1"
-F 0 "U14" H 3050 6967 50  0000 C CNN
+AR Path="/63268641/63A2F4D2" Ref="U8"  Part="1"
+F 0 "U8" H 3050 6967 50  0000 C CNN
 F 1 "74LS04" H 3050 6876 50  0000 C CNN
 F 2 "Package_DIP:DIP-14_W7.62mm" H 3050 6650 50  0001 C CNN
@@
 AR Path="/63268613/63A2F4D9" Ref="U?"  Part="2"
 AR Path="/639E280B/63A2F4D9" Ref="U?"  Part="2"
-AR Path="/63268641/63A2F4D9" Ref="U14"  Part="2"
-F 0 "U14" H 3950 6967 50  0000 C CNN
+AR Path="/63268641/63A2F4D9" Ref="U8"  Part="2"
+F 0 "U8" H 3950 6967 50  0000 C CNN
 F 1 "74LS04" H 3950 6876 50  0000 C CNN
 F 2 "Package_DIP:DIP-14_W7.62mm" H 3950 6650 50  0001 C CNN
@@
 Connection ~ 8550 5100
 $Comp
-L 74xx:74LS02 U?
+L 74xx:74LS02 U9
 U 1 1 63C57B8A
 P 3200 4650
-F 0 "U?" H 3200 4975 50  0000 C CNN
+F 0 "U9" H 3200 4975 50  0000 C CNN
 F 1 "74LS02" H 3200 4884 50  0000 C CNN
-F 2 "" H 3200 4650 50  0001 C CNN
+F 2 "Package_DIP:DIP-14_W7.62mm" H 3200 4650 50  0001 C CNN
 F 3 "http://www.ti.com/lit/gpn/sn74ls02" H 3200 4650 50  0001 C CNN
 	1    3200 4650
@@
 $EndComp
 $Comp
-L 74xx:74LS02 U?
+L 74xx:74LS02 U9
 U 2 1 63C57C0D
 P 3200 5200
-F 0 "U?" H 3200 5525 50  0000 C CNN
+F 0 "U9" H 3200 5525 50  0000 C CNN
 F 1 "74LS02" H 3200 5434 50  0000 C CNN
-F 2 "" H 3200 5200 50  0001 C CNN
+F 2 "Package_DIP:DIP-14_W7.62mm" H 3200 5200 50  0001 C CNN
 F 3 "http://www.ti.com/lit/gpn/sn74ls02" H 3200 5200 50  0001 C CNN
 	2    3200 5200
@@
 $EndComp
 $Comp
-L 74xx:74LS02 U?
+L 74xx:74LS02 U9
 U 3 1 63C57C78
 P 8000 5200
-F 0 "U?" H 8000 5525 50  0000 C CNN
+F 0 "U9" H 8000 5525 50  0000 C CNN
 F 1 "74LS02" H 8000 5434 50  0000 C CNN
-F 2 "" H 8000 5200 50  0001 C CNN
+F 2 "Package_DIP:DIP-14_W7.62mm" H 8000 5200 50  0001 C CNN
 F 3 "http://www.ti.com/lit/gpn/sn74ls02" H 8000 5200 50  0001 C CNN
 	3    8000 5200
@@
 AR Path="/63D680DF" Ref="R?"  Part="1"
 AR Path="/63268613/63D680DF" Ref="R?"  Part="1"
-AR Path="/63268641/63D680DF" Ref="R?"  Part="1"
-F 0 "R?" H 1850 6450 50  0000 L CNN
+AR Path="/63268641/63D680DF" Ref="R15"  Part="1"
+F 0 "R15" H 1850 6450 50  0000 L CNN
 F 1 "10k" H 1850 6350 50  0000 L CNN
 F 2 "Resistor_THT:R_Axial_DIN0207_L6.3mm_D2.5mm_P10.16mm_Horizontal" V 2090 6390 50  0001 C CNN
@@
 AR Path="/63D680E7" Ref="#PWR?"  Part="1"
 AR Path="/63268613/63D680E7" Ref="#PWR?"  Part="1"
-AR Path="/63268641/63D680E7" Ref="#PWR?"  Part="1"
-F 0 "#PWR?" H 2050 6100 50  0001 C CNN
+AR Path="/63268641/63D680E7" Ref="#PWR0133"  Part="1"
+F 0 "#PWR0133" H 2050 6100 50  0001 C CNN
 F 1 "+5V" H 2150 6350 50  0000 C CNN
 F 2 "" H 2050 6250 50  0001 C CNN
@@
 AR Path="/63E9F755" Ref="R?"  Part="1"
 AR Path="/63268613/63E9F755" Ref="R?"  Part="1"
-AR Path="/63268641/63E9F755" Ref="R?"  Part="1"
-F 0 "R?" H 2150 5000 50  0000 L CNN
+AR Path="/63268641/63E9F755" Ref="R14"  Part="1"
+F 0 "R14" H 2150 5000 50  0000 L CNN
 F 1 "10k" H 2150 4900 50  0000 L CNN
 F 2 "Resistor_THT:R_Axial_DIN0207_L6.3mm_D2.5mm_P10.16mm_Horizontal" V 2390 4940 50  0001 C CNN
@@
 AR Path="/63F58472" Ref="#PWR?"  Part="1"
 AR Path="/63268613/63F58472" Ref="#PWR?"  Part="1"
-AR Path="/63268641/63F58472" Ref="#PWR?"  Part="1"
-F 0 "#PWR?" H 2050 4550 50  0001 C CNN
+AR Path="/63268641/63F58472" Ref="#PWR0137"  Part="1"
+F 0 "#PWR0137" H 2050 4550 50  0001 C CNN
 F 1 "+5V" H 2150 4800 50  0000 C CNN
 F 2 "" H 2050 4700 50  0001 C CNN
@@
 AR Path="/63F584D4" Ref="R?"  Part="1"
 AR Path="/63268613/63F584D4" Ref="R?"  Part="1"
-AR Path="/63268641/63F584D4" Ref="R?"  Part="1"
-F 0 "R?" H 1550 5000 50  0000 L CNN
+AR Path="/63268641/63F584D4" Ref="R12"  Part="1"
+F 0 "R12" H 1550 5000 50  0000 L CNN
 F 1 "10k" H 1550 4900 50  0000 L CNN
 F 2 "Resistor_THT:R_Axial_DIN0207_L6.3mm_D2.5mm_P10.16mm_Horizontal" V 1790 4940 50  0001 C CNN
@@
 	1650 6650 2050 6650
 $Comp
-L 74xx:74LS151 U?
+L 74xx:74LS151 U11
 U 1 1 640AA7BE
 P 4400 3800
-F 0 "U?" H 4550 4650 50  0000 C CNN
+F 0 "U11" H 4550 4650 50  0000 C CNN
 F 1 "74LS151" H 4600 4550 50  0000 C CNN
-F 2 "" H 4400 3800 50  0001 C CNN
+F 2 "Package_DIP:DIP-16_W7.62mm" H 4400 3800 50  0001 C CNN
 F 3 "http://www.ti.com/lit/gpn/sn74LS151" H 4400 3800 50  0001 C CNN
 	1    4400 3800
@@
 AR Path="/642529A8" Ref="R?"  Part="1"
 AR Path="/63268613/642529A8" Ref="R?"  Part="1"
-AR Path="/63268641/642529A8" Ref="R?"  Part="1"
-F 0 "R?" H 1850 5000 50  0000 L CNN
+AR Path="/63268641/642529A8" Ref="R13"  Part="1"
+F 0 "R13" H 1850 5000 50  0000 L CNN
 F 1 "10k" H 1850 4900 50  0000 L CNN
 F 2 "Resistor_THT:R_Axial_DIN0207_L6.3mm_D2.5mm_P10.16mm_Horizontal" V 2090 4940 50  0001 C CNN
@@
 Wire Wire Line
 	3450 6650 3650 6650
+Wire Wire Line
+	2050 6650 2750 6650
 Wire Bus Line
 	8750 2800 8750 3850
@@
 Wire Bus Line
 	7050 1200 7050 3450
-Wire Wire Line
-	2050 6650 2750 6650
 $EndSCHEMATC

Commit message: Update part numbers Swap out input connector footprint Placement tweaks
Parts:
- U15: renamed from U16; footprint Package_DIP:DIP-16_W7.62mm -> Package_DIP:DIP-20_W7.62mm
- U16: renamed from U17; footprint Package_DIP:DIP-14_W7.62mm -> Package_DIP:DIP-16_W7.62mm
- renumbered U15 to U14
Changed lines of the file:
@@
 P 2200 2050
 AR Path="/63304670" Ref="U?"  Part="1"
-AR Path="/63268641/63304670" Ref="U17"  Part="1"
-F 0 "U17" H 2200 1750 50  0000 C CNN
+AR Path="/63268641/63304670" Ref="U16"  Part="1"
+F 0 "U16" H 2200 1750 50  0000 C CNN
 F 1 "LM339" H 2200 1850 50  0000 C CNN
-F 2 "Package_DIP:DIP-14_W7.62mm" H 2150 2150 50  0001 C CNN
+F 2 "Package_DIP:DIP-16_W7.62mm" H 2150 2150 50  0001 C CNN
 F 3 "http://www.ti.com/lit/ds/symlink/lm339.pdf" H 2250 2250 50  0001 C CNN
 	1    2200 2050
@@
 P 2200 4050
 AR Path="/63304677" Ref="U?"  Part="4"
-AR Path="/63268641/63304677" Ref="U17"  Part="4"
-F 0 "U17" H 2200 3750 50  0000 C CNN
+AR Path="/63268641/63304677" Ref="U16"  Part="4"
+F 0 "U16" H 2200 3750 50  0000 C CNN
 F 1 "LM339" H 2200 3850 50  0000 C CNN
-F 2 "Package_DIP:DIP-14_W7.62mm" H 2150 4150 50  0001 C CNN
+F 2 "Package_DIP:DIP-16_W7.62mm" H 2150 4150 50  0001 C CNN
 F 3 "http://www.ti.com/lit/ds/symlink/lm339.pdf" H 2250 4250 50  0001 C CNN
 	4    2200 4050
@@
 P 2200 2700
 AR Path="/6330467E" Ref="U?"  Part="2"
-AR Path="/63268641/6330467E" Ref="U17"  Part="2"
-F 0 "U17" H 2200 2400 50  0000 C CNN
+AR Path="/63268641/6330467E" Ref="U16"  Part="2"
+F 0 "U16" H 2200 2400 50  0000 C CNN
 F 1 "LM339" H 2200 2500 50  0000 C CNN
-F 2 "Package_DIP:DIP-14_W7.62mm" H 2150 2800 50  0001 C CNN
+F 2 "Package_DIP:DIP-16_W7.62mm" H 2150 2800 50  0001 C CNN
 F 3 "http://www.ti.com/lit/ds/symlink/lm339.pdf" H 2250 2900 50  0001 C CNN
 	2    2200 2700
@@
 P 2200 3400
 AR Path="/63304685" Ref="U?"  Part="3"
-AR Path="/63268641/63304685" Ref="U17"  Part="3"
-F 0 "U17" H 2200 3100 50  0000 C CNN
+AR Path="/63268641/63304685" Ref="U16"  Part="3"
+F 0 "U16" H 2200 3100 50  0000 C CNN
 F 1 "LM339" H 2200 3200 50  0000 C CNN
-F 2 "Package_DIP:DIP-14_W7.62mm" H 2150 3500 50  0001 C CNN
+F 2 "Package_DIP:DIP-16_W7.62mm" H 2150 3500 50  0001 C CNN
 F 3 "http://www.ti.com/lit/ds/symlink/lm339.pdf" H 2250 3600 50  0001 C CNN
 	3    2200 3400
@@
 	6700 1100 6950 1100
 $Comp
-L transmitter-retro:TLC7524CN U16
+L transmitter-retro:TLC7524CN U15
 U 1 1 634200B5
 P 6300 1500
-F 0 "U16" H 6100 2150 50  0000 C CNN
+F 0 "U15" H 6100 2150 50  0000 C CNN
 F 1 "TLC7524CN" H 6000 2050 50  0000 C CNN
-F 2 "Package_DIP:DIP-16_W7.62mm" H 6300 1500 50  0001 C CNN
+F 2 "Package_DIP:DIP-20_W7.62mm" H 6300 1500 50  0001 C CNN
 F 3 "http://www.pinballpcb.com/datasheets/OnMC1408-dac.pdf" H 6300 1500 50  0001 C CNN
 	1    6300 1500
@@
 	5750 3950 5800 3950
 $Comp
-L 74xx:74LS373 U15
+L 74xx:74LS373 U14
 U 1 1 638DE1BD
 P 9550 3750
-F 0 "U15" H 9700 4500 50  0000 C CNN
+F 0 "U14" H 9700 4500 50  0000 C CNN
 F 1 "74LS373" H 9800 4400 50  0000 C CNN
 F 2 "Package_DIP:DIP-20_W7.62mm" H 9550 3750 50  0001 C CNN

Commit message: Prototype and PCB layout for core Prototype and PCB layout for demo Prototype and PCB layout for control-eprom Move display design forward Refactor control-dmx to dmx Update expansion connector on all boards Add test suites Add tx-retro readme Cleanup
Parts:
- removed R12, R13: 10k, Resistor_THT:R_Axial_DIN0207_L6.3mm_D2.5mm_P10.16mm_Horizontal, symbol Device:R_US
- removed U9: 74LS02, Package_DIP:DIP-14_W7.62mm, symbol 74xx:74LS02
- added R4: 1.6k, Resistor_THT:R_Axial_DIN0207_L6.3mm_D2.5mm_P10.16mm_Horizontal, symbol Device:R_US
- added R5, R6: 10k, Resistor_THT:R_Axial_DIN0207_L6.3mm_D2.5mm_P10.16mm_Horizontal, symbol Device:R_US
- added unit 6 of U10
- added unit 4 of U10
- added unit 5 of U10
- added U12: 74LS08, Package_DIP:DIP-14_W7.62mm, symbol 74xx:74LS08
- added U9: TLV2772CP, Package_DIP:DIP-8_W7.62mm, symbol CrazyGiraffe_DMXDemonstrator:TLV2772CP
- added VR1: TL1431, Package_TO_SOT_THT:TO-92L_HandSolder, symbol CrazyGiraffe_DMXDemonstrator:TL1431
- U7: renamed from U15; footprint Package_DIP:DIP-20_W7.62mm -> Package_DIP:DIP-16_W7.62mm; symbol transmitter-retro:TLC7524CN -> CrazyGiraffe_DMXDemonstrator:TLC7524CN
- U8: renamed from U16; footprint Package_DIP:DIP-16_W7.62mm -> Package_DIP:DIP-14_W7.62mm
- renumbered R15 to R2, R14 to R3, U8 to U10, U11 to U3, U12 to U4, U13 to U5, U14 to U6
Connections:
- net labels added: CLK_SAMPLE_IN
- net labels removed: D01, SAMPLE_CLOCK_IN, SAMPLE_REF_OUT
- wire segments 170 -> 181
Other:
- note added: "0-5V D-to-A Converter\n\nSee: \nhttps://www.ti.com/lit/an/sloa039a/sloa039a.pdf\nFigure 18"
- note added: "2 * VREF * (D/256)"
- note added: "2.5V=VREF"
- note added: "Analog Section"
- note added: "Data Latch\n"
- note added: "Dimmer\nCompare"
- note added: "Dimmer\nSelect"
- note added: "Sample Counter"
- note added: "U4 and U5 count from 0-255 at the rate of CLK_SAMPLE_IN. This value is sent to U7\nwhich converts this value into an analog voltage from 0-5v. This value is also sent to U6,\nwhich is can be captured and held for the shift register to send the value to DATA_RX_OUT.\nU4 and U5 are reset by ~SAMPLE_RESET_IN~ at the start of the sampling period.\n\nCLK_SAMPLE_IN is 32x faster than CLK_TX_OUT so that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"
- note added: "VREF * (D/256)"
- note removed: "Dimmer Level\nCounter"
- note removed: "Dimmer\nLevel Latch\n"
- note removed: "Dimmer\nMultiplexer"
- note removed: "voltage-mode operation,\nsee datasheet"
- moved on the sheet: U8A, U8B, U8C, U8D
