File: hardware/dimmer-dmx/dimmer-dmx.kicad_pcb (KiCad board)
At the start: 2 copper layers, 60 x 60 mm, 22 parts, among them J1 IO EXTENSION, J2 DIMMER_B, J5 12V_A, J6 12V_B, U1 LM317T, U2 74LS164, U3 TLC7226A, U4 LM324A

Commit message: Add analog, pwm, dmx, and io boards. Still needs work.
Parts:
- removed C1: .01uF, Capacitors:CAP-PTH-2.54
- removed D8: 1N5819, Diode_THT:D_DO-41_SOD81_P10.16mm_Horizontal
- removed J5: 12V_A, Connector_BarrelJack:BarrelJack_CUI_PJ-063AH_Horizontal
- removed J6: 12V_B, Connector_Phoenix_MSTB:PhoenixContact_MSTBA_2,5_2-G-5,08_1x02_P5.08mm_Horizontal
- added ?: , footprints:OSHW-LOGO-S, B.Cu at (154.8, 117.1)
- added J3: NC3MAH/NC5MAH, footprints:NEUTRIK-NC3MAH-NC5MAH, F.Cu at (156.1, 66.1)
- added R1: 330, Resistor_THT:R_Axial_DIN0207_L6.3mm_D2.5mm_P10.16mm_Horizontal, F.Cu at (125.6, 104.3)
- added R10: 680, Resistor_THT:R_Axial_DIN0207_L6.3mm_D2.5mm_P10.16mm_Horizontal, F.Cu at (167.3, 71.9)
- added R2: 470, Resistor_THT:R_Axial_DIN0207_L6.3mm_D2.5mm_P10.16mm_Horizontal, F.Cu at (129.2, 104.3)
- added R3: 470, Resistor_THT:R_Axial_DIN0207_L6.3mm_D2.5mm_P10.16mm_Horizontal, F.Cu at (156.7, 87.8)
- added R4: 470, Resistor_THT:R_Axial_DIN0207_L6.3mm_D2.5mm_P10.16mm_Horizontal, F.Cu at (164.5, 104.3)
- added R5: 470, Resistor_THT:R_Axial_DIN0207_L6.3mm_D2.5mm_P10.16mm_Horizontal, F.Cu at (153.8, 87.8)
- added R6: 470, Resistor_THT:R_Axial_DIN0207_L6.3mm_D2.5mm_P10.16mm_Horizontal, F.Cu at (161.0, 104.3)
- added R9: 120, Resistor_THT:R_Axial_DIN0207_L6.3mm_D2.5mm_P10.16mm_Horizontal, F.Cu at (117.7, 71.9)
- added U5: MAX3485CPA+, Package_DIP:DIP-8_W7.62mm_Socket, F.Cu at (133.1, 99.1)
- C5: value 10uF -> .01uF; footprint Capacitor_THT:CP_Radial_D5.0mm_P2.50mm -> Capacitors:CAP-PTH-2.54
- J2: value DIMMER_B -> NC3FAH/NC5FAH; footprint Connector_Phoenix_MSTB:PhoenixContact_MSTBA_2,5_5-G-5,08_1x05_P5.08mm_Horizontal -> footprints:NEUTRIK-NC3FAH-NC5FAH
- R7: value 390 -> 470
- R8: value 2.7k -> 680
- U1: value LM317T -> NMA0505SC; footprint Package_TO_SOT_THT:TO-220-3_Horizontal_TabDown -> footprints:Converter_DCDC_muRata_NMAxxxxSC_THT_Bypass
- U2: value 74LS164 -> 6N137; footprint Package_DIP:DIP-14_W7.62mm -> Package_DIP:DIP-8_W7.62mm_Socket
- U3: value TLC7226A -> 6N137; footprint Package_DIP:DIP-20_W7.62mm -> Package_DIP:DIP-8_W7.62mm_Socket
- U4: value LM324A -> 6N137; footprint Package_DIP:DIP-14_W7.62mm -> Package_DIP:DIP-8_W7.62mm_Socket
- moved R8 57.6 mm to (171.2, 71.9), turned to 270 degrees
- moved C4 38.1 mm to (135.9, 97.8), turned to 90 degrees
- moved J2 31.1 mm to (132.7, 66.1), turned to 0 degrees
- moved U4 25.5 mm to (146.2, 99.1), turned to 180 degrees
- moved U1 22.2 mm to (116.6, 106.6)
- moved U2 21.5 mm to (172.1, 99.1), turned to 180 degrees
- moved R7 21.2 mm to (128.4, 87.9), turned to 0 degrees
- moved U3 17.9 mm to (159.1, 99.1), turned to 180 degrees
- moved C5 16.8 mm to (122.8, 97.8), turned to 90 degrees
- moved C3 9.40 mm to (148.8, 97.8), turned to 90 degrees
- moved C2 8.01 mm to (161.8, 95.2)
- moved MH4 0.25 mm to (170.1, 116.6)
- moved MH2 0.13 mm to (170.1, 64.8)
Connections:
- C3 pad 1: +5V -> VDD
- C3 pad 2: GND -> GNDD
- C4 pad 1: +10V -> VDD
- C4 pad 2: GND -> GNDD
- C5 pad 1: +10V -> VDD
- C5 pad 2: GND -> GNDD
- J1 pad 3: /~WR -> Net-(J1-Pad3)
- J1 pad 5: /A0 -> Net-(J1-Pad5)
- J1 pad 7: /A1 -> Net-(J1-Pad7)
- R7 pad 2: +10V -> VDD
- R8 pad 1: GND -> Net-(J2-Pad3)
- R8 pad 2: Net-(R7-Pad1) -> VDD
- U1 pad 1: Net-(R7-Pad1) -> +5V
- U1 pad 2: +10V -> GND
- U2 pad 1: +5V -> Net-(U2-Pad1)
- U2 pad 2: Net-(J1-Pad4) -> VDD
- U2 pad 3: Net-(U2-Pad3) -> Net-(R3-Pad2)
- U2 pad 5: Net-(U2-Pad5) -> GND
- U2 pad 6: Net-(U2-Pad6) -> Net-(J1-Pad9)
- U2 pad 7: GND -> Net-(U2-Pad7)
- U2 pad 8: Net-(J1-Pad6) -> +5V
- U3 pad 1: /AO1 -> Net-(U3-Pad1)
- U3 pad 2: /AO0 -> +5V
- U3 pad 3: GND -> Net-(R4-Pad1)
- U3 pad 4: +10V -> Net-(U3-Pad4)
- U3 pad 5: GND -> GNDD
- U3 pad 6: GND -> Net-(R5-Pad1)
- U3 pad 7: Net-(U2-Pad13) -> Net-(U3-Pad7)
- U3 pad 8: Net-(U2-Pad12) -> VDD
- U4 pad 1: Net-(J2-Pad3) -> Net-(U4-Pad1)
- U4 pad 2: Net-(J2-Pad3) -> +5V
- U4 pad 3: /AO1 -> Net-(R6-Pad1)
- U4 pad 4: +10V -> Net-(U4-Pad4)
- U4 pad 5: /AO2 -> GNDD
- U4 pad 6: Net-(J2-Pad4) -> Net-(R7-Pad1)
- U4 pad 7: Net-(J2-Pad4) -> Net-(U4-Pad7)
- U4 pad 8: Net-(J2-Pad5) -> VDD
Routing:
- net Net-(J2-Pad3): track 0.00 -> 102.5 mm, vias 0 -> 1
- net Net-(J2-Pad2A): track 0.00 -> 98.7 mm, vias 0 -> 3
- net Net-(J1-Pad9): track 0.00 -> 62.1 mm, vias 0 -> 3
- net Net-(R5-Pad1): track 0.00 -> 41.3 mm, vias 0 -> 1
- net Net-(R6-Pad1): track 0.00 -> 41.1 mm, vias 0 -> 1
- net Net-(R3-Pad1): track 0.00 -> 40.9 mm, vias 0 -> 2
- net Net-(J1-Pad11): track 0.00 -> 30.8 mm, vias 0 -> 1
- net Net-(J1-Pad10): track 0.00 -> 29.5 mm, vias 0 -> 1
- net Net-(J1-Pad12): track 0.00 -> 20.7 mm, vias 0 -> 1
- net Net-(R7-Pad1): track 0.00 -> 16.3 mm, vias 0 -> 1
- net Net-(R4-Pad1): track 0.00 -> 14.5 mm, vias 0 -> 1
- net Net-(R3-Pad2): track 0.00 -> 13.3 mm
- net VDD: track 0.00 -> 10.7 mm
- net +5V: track 0.00 -> 2.67 mm
- added copper zone on B.Cu, net GNDD
- added copper zone on F.Cu, net VDD
- removed copper zone on F.Cu, net +10V
Other:
- outline, holes or cut-outs redrawn
- net class Power added: clearance 0.1524, trace_width 0.3048, via_dia 1.27, via_drill 0.635
- board text added: "Bridge to bypass Iso"
- board text added: "DMX Termination: 120 ohms"
- board text added: "DMX-DD1"
- board text added: "DMX-DD1, Rev 1.1 Crazy Giraffe Software"
- board text added: "RDM Termination: 680 ohms"
- board text removed: "- +"
- board text removed: "12v In"
- board text removed: "DMX-DA1"
- board text removed: "DMX-DA1, Rev 1.1 Crazy Giraffe Software"
- board text removed: "G 1 2 3 4 0-10v Dimmer Out"
- board text removed: "J5/6"
