File: hardware/transmitter-retro/control-eprom/control-eprom.sch (KiCad schematic (older format))
At the start: 15 parts, among them U18 74LS32, U20 74LS00, U3 74LS161, U4 74LS161, U5 27128

Commit message: Add top level project Update part #s Update power sheets
Parts:
- gave numbers to parts that had none: 1
- renumbered U18 to U1, U20 to U2
Changed lines of the file:
@@
 	5800 3500 6450 3500
 $Comp
-L 74xx:74LS32 U18
+L 74xx:74LS32 U1
 U 3 1 63E3B12B
 P 7500 4000
-F 0 "U18" H 7500 4325 50  0000 C CNN
+F 0 "U1" H 7500 4325 50  0000 C CNN
 F 1 "74LS32" H 7500 4234 50  0000 C CNN
 F 2 "Package_DIP:DIP-14_W7.62mm" H 7500 4000 50  0001 C CNN
@@
 $EndComp
 $Comp
-L 74xx:74LS32 U18
+L 74xx:74LS32 U1
 U 4 1 63E3B1AE
 P 8200 4100
-F 0 "U18" H 8200 4425 50  0000 C CNN
+F 0 "U1" H 8200 4425 50  0000 C CNN
 F 1 "74LS32" H 8200 4334 50  0000 C CNN
 F 2 "Package_DIP:DIP-14_W7.62mm" H 8200 4100 50  0001 C CNN
@@
 $EndComp
 $Comp
-L 74xx:74LS32 U18
+L 74xx:74LS32 U1
 U 5 1 63E3B20B
 P 2150 6900
-F 0 "U18" H 2380 6946 50  0000 L CNN
+F 0 "U1" H 2380 6946 50  0000 L CNN
 F 1 "74LS32" H 2380 6855 50  0000 L CNN
 F 2 "Package_DIP:DIP-14_W7.62mm" H 2150 6900 50  0001 C CNN
@@
 AR Path="/6BB77A68/681C43A0" Ref="C1"  Part="1"
 AR Path="/64132440/6413313E/681C43A0" Ref="C?"  Part="1"
-AR Path="/681C43A0" Ref="C3"  Part="1"
-F 0 "C3" H 3715 6946 50  0000 L CNN
+AR Path="/681C43A0" Ref="C1"  Part="1"
+F 0 "C1" H 3715 6946 50  0000 L CNN
 F 1 ".01uF" H 3715 6855 50  0000 L CNN
 F 2 "Capacitor_THT:C_Rect_L4.6mm_W2.0mm_P2.50mm_MKS02_FKP02" H 3638 6750 50  0001 C CNN
@@
 AR Path="/6BB77A68/681C4400" Ref="C2"  Part="1"
 AR Path="/64132440/6413313E/681C4400" Ref="C?"  Part="1"
-AR Path="/681C4400" Ref="C4"  Part="1"
-F 0 "C4" H 4215 6946 50  0000 L CNN
+AR Path="/681C4400" Ref="C2"  Part="1"
+F 0 "C2" H 4215 6946 50  0000 L CNN
 F 1 ".01uF" H 4215 6855 50  0000 L CNN
 F 2 "Capacitor_THT:C_Rect_L4.6mm_W2.0mm_P2.50mm_MKS02_FKP02" H 4138 6750 50  0001 C CNN
@@
 AR Path="/6BB77A68/681C443E" Ref="C3"  Part="1"
 AR Path="/64132440/6413313E/681C443E" Ref="C?"  Part="1"
-AR Path="/681C443E" Ref="C5"  Part="1"
-F 0 "C5" H 4665 6946 50  0000 L CNN
+AR Path="/681C443E" Ref="C3"  Part="1"
+F 0 "C3" H 4665 6946 50  0000 L CNN
 F 1 ".01uF" H 4665 6855 50  0000 L CNN
 F 2 "Capacitor_THT:C_Rect_L4.6mm_W2.0mm_P2.50mm_MKS02_FKP02" H 4588 6750 50  0001 C CNN
@@
 AR Path="/6BB77A68/714E8297" Ref="C4"  Part="1"
 AR Path="/64132440/6413313E/714E8297" Ref="C?"  Part="1"
-AR Path="/714E8297" Ref="C18"  Part="1"
-F 0 "C18" H 5115 6946 50  0000 L CNN
+AR Path="/714E8297" Ref="C4"  Part="1"
+F 0 "C4" H 5115 6946 50  0000 L CNN
 F 1 ".01uF" H 5115 6855 50  0000 L CNN
 F 2 "Capacitor_THT:C_Rect_L4.6mm_W2.0mm_P2.50mm_MKS02_FKP02" H 5038 6750 50  0001 C CNN
@@
 AR Path="/6BB77A68/714E8299" Ref="C5"  Part="1"
 AR Path="/64132440/6413313E/714E8299" Ref="C?"  Part="1"
-AR Path="/714E8299" Ref="C20"  Part="1"
-F 0 "C20" H 5565 6946 50  0000 L CNN
+AR Path="/714E8299" Ref="C5"  Part="1"
+F 0 "C5" H 5565 6946 50  0000 L CNN
 F 1 ".01uF" H 5565 6855 50  0000 L CNN
 F 2 "Capacitor_THT:C_Rect_L4.6mm_W2.0mm_P2.50mm_MKS02_FKP02" H 5488 6750 50  0001 C CNN
@@
 Reset: 10001101b (0x4d, 141d)\nThis is the final value in a packet. At this point,\nthe counter will reset and start the break again.\n\nIts' chosen because it's a value which is unlikely\nto be used in a packet, i.e. sample reset and latch \nany dimmer and shift load while enabled while \ntransmitting a break.\n
 $Comp
-L 74xx:74LS32 U18
+L 74xx:74LS32 U1
 U 2 1 63871246
 P 6800 5050
-AR Path="/63871246" Ref="U18"  Part="2"
+AR Path="/63871246" Ref="U1"  Part="2"
 AR Path="/632F1F43/63871246" Ref="U?"  Part="2"
 AR Path="/63267F40/63871246" Ref="U?"  Part="2"
-F 0 "U18" H 6800 4733 50  0000 C CNN
+F 0 "U1" H 6800 4733 50  0000 C CNN
 F 1 "74LS32" H 6800 4824 50  0000 C CNN
 F 2 "Package_DIP:DIP-14_W7.62mm" H 6800 5050 50  0001 C CNN
@@
 	6450 3800 6450 3500
 $Comp
-L 74xx:74LS00 U20
+L 74xx:74LS00 U2
 U 1 1 639D9D08
 P 6800 3900
-F 0 "U20" H 6800 4225 50  0000 C CNN
+F 0 "U2" H 6800 4225 50  0000 C CNN
 F 1 "74LS00" H 6800 4134 50  0000 C CNN
 F 2 "Package_DIP:DIP-14_W7.62mm" H 6800 3900 50  0001 C CNN
@@
 $EndComp
 $Comp
-L 74xx:74LS00 U20
+L 74xx:74LS00 U2
 U 3 1 639D9E78
 P 1250 6900
-F 0 "U20" H 1250 7225 50  0000 C CNN
+F 0 "U2" H 1250 7225 50  0000 C CNN
 F 1 "74LS00" H 1250 7134 50  0000 C CNN
 F 2 "Package_DIP:DIP-14_W7.62mm" H 1250 6900 50  0001 C CNN
@@
 	6150 4600 6500 4600
 $Comp
-L 74xx:74LS32 U18
+L 74xx:74LS32 U1
 U 1 1 639F9CBD
 P 6800 4500
-F 0 "U18" H 6800 4825 50  0000 C CNN
+F 0 "U1" H 6800 4825 50  0000 C CNN
 F 1 "74LS32" H 6800 4734 50  0000 C CNN
 F 2 "Package_DIP:DIP-14_W7.62mm" H 6800 4500 50  0001 C CNN
@@
 	6250 3400 9400 3400
 $Comp
-L 74xx:74LS00 U20
+L 74xx:74LS00 U2
 U 2 1 63AF0D80
 P 1250 6350
-F 0 "U20" H 1250 6675 50  0000 C CNN
+F 0 "U2" H 1250 6675 50  0000 C CNN
 F 1 "74LS00" H 1250 6584 50  0000 C CNN
 F 2 "Package_DIP:DIP-14_W7.62mm" H 1250 6350 50  0001 C CNN
@@
 $EndComp
 $Comp
-L 74xx:74LS00 U20
+L 74xx:74LS00 U2
 U 4 1 639D9EE1
 P 1250 7450
-F 0 "U20" H 1250 7775 50  0000 C CNN
+F 0 "U2" H 1250 7775 50  0000 C CNN
 F 1 "74LS00" H 1250 7684 50  0000 C CNN
 F 2 "Package_DIP:DIP-14_W7.62mm" H 1250 7450 50  0001 C CNN
@@
 	850  6150 850  6250
 $Comp
-L 74xx:74LS00 U20
+L 74xx:74LS00 U2
 U 5 1 63AF9174
 P 2950 6900
-F 0 "U20" H 3180 6946 50  0000 L CNN
+F 0 "U2" H 3180 6946 50  0000 L CNN
 F 1 "74LS00" H 3180 6855 50  0000 L CNN
 F 2 "Package_DIP:DIP-14_W7.62mm" H 2950 6900 50  0001 C CNN
@@
 $EndComp
 $Comp
-L power:GND #PWR?
-U 1 1 64610829
-P 9300 4400
-AR Path="/64610829" Ref="#PWR?"  Part="1"
-AR Path="/632F1F43/64610829" Ref="#PWR?"  Part="1"
-AR Path="/63267F40/64610829" Ref="#PWR?"  Part="1"
-AR Path="/646018E8/64610829" Ref="#PWR?"  Part="1"
-F 0 "#PWR?" H 9300 4150 50  0001 C CNN
-F 1 "GND" H 9450 4300 50  0000 C CNN
-F 2 "" H 9300 4400 50  0001 C CNN
-F 3 "" H 9300 4400 50  0001 C CNN
-	1    9300 4400
-	-1   0    0    -1
-$EndComp
-Wire Wire Line
-	9400 4200 9300 4200
-Wire Wire Line
-	9300 4200 9300 4300
-Wire Wire Line
-	9400 4300 9300 4300
-Connection ~ 9300 4300
-Wire Wire Line
-	9300 4300 9300 4400
-$Comp
-L power:GND #PWR?
+L power:GND #PWR0113
 U 1 1 64610834
 P 10000 4400
-AR Path="/64610834" Ref="#PWR?"  Part="1"
+AR Path="/64610834" Ref="#PWR0113"  Part="1"
 AR Path="/632F1F43/64610834" Ref="#PWR?"  Part="1"
 AR Path="/63267F40/64610834" Ref="#PWR?"  Part="1"
 AR Path="/646018E8/64610834" Ref="#PWR?"  Part="1"
-F 0 "#PWR?" H 10000 4150 50  0001 C CNN
+F 0 "#PWR0113" H 10000 4150 50  0001 C CNN
 F 1 "GND" H 10150 4300 50  0000 C CNN
 F 2 "" H 10000 4400 50  0001 C CNN
@@
 	10000 4300 10000 4200
 $Comp
-L power:+5V #PWR?
+L power:+5V #PWR0114
 U 1 1 6461083F
 P 9300 2300
-AR Path="/6461083F" Ref="#PWR?"  Part="1"
+AR Path="/6461083F" Ref="#PWR0114"  Part="1"
 AR Path="/632F1F43/6461083F" Ref="#PWR?"  Part="1"
 AR Path="/63267F40/6461083F" Ref="#PWR?"  Part="1"
 AR Path="/646018E8/6461083F" Ref="#PWR?"  Part="1"
-F 0 "#PWR?" H 9300 2150 50  0001 C CNN
+F 0 "#PWR0114" H 9300 2150 50  0001 C CNN
 F 1 "+5V" H 9315 2473 50  0000 C CNN
 F 2 "" H 9300 2300 50  0001 C CNN
@@
 	9300 2400 9300 2300
 $Comp
-L power:+5V #PWR?
+L power:+5V #PWR0115
 U 1 1 6461084A
 P 10000 2300
-AR Path="/6461084A" Ref="#PWR?"  Part="1"
+AR Path="/6461084A" Ref="#PWR0115"  Part="1"
 AR Path="/632F1F43/6461084A" Ref="#PWR?"  Part="1"
 AR Path="/63267F40/6461084A" Ref="#PWR?"  Part="1"
 AR Path="/646018E8/6461084A" Ref="#PWR?"  Part="1"
-F 0 "#PWR?" H 10000 2150 50  0001 C CNN
+F 0 "#PWR0115" H 10000 2150 50  0001 C CNN
 F 1 "+5V" H 10015 2473 50  0000 C CNN
 F 2 "" H 10000 2300 50  0001 C CNN
@@
 P 9700 3300
 AR Path="/63267F40/6461086D" Ref="J?"  Part="1"
-AR Path="/6461086D" Ref="J?"  Part="1"
+AR Path="/6461086D" Ref="J1"  Part="1"
 AR Path="/646018E8/6461086D" Ref="J?"  Part="1"
-F 0 "J?" H 9750 4417 50  0000 C CNN
+F 0 "J1" H 9750 4417 50  0000 C CNN
 F 1 "Expansion" H 9750 4326 50  0000 C CNN
 F 2 "Connector_PinHeader_2.54mm:PinHeader_2x20_P2.54mm_Vertical" H 9700 3300 50  0001 C CNN
@@
 NoConn ~ 9900 3600
 NoConn ~ 9900 3700
-NoConn ~ 9900 4100
-NoConn ~ 9900 4000
 NoConn ~ 9900 3900
 NoConn ~ 9400 3700
@@
 Wire Wire Line
 	2950 7400 2950 7450
+Connection ~ 2950 7450
+Wire Wire Line
+	2950 7450 3600 7450
+Wire Wire Line
+	9900 4000 10000 4000
+Wire Wire Line
+	10000 4000 10000 4100
+Connection ~ 10000 4200
+Wire Wire Line
+	9900 4100 10000 4100
+Connection ~ 10000 4100
+Wire Wire Line
+	10000 4100 10000 4200
+NoConn ~ 9400 4200
+NoConn ~ 9400 4300
 Wire Bus Line
 	2750 1800 4650 1800
@@
 Wire Bus Line
 	4750 1900 4750 3400
-Connection ~ 2950 7450
-Wire Wire Line
-	2950 7450 3600 7450
 $EndSCHEMATC

Commit message: Prototype and PCB layout for core Prototype and PCB layout for demo Prototype and PCB layout for control-eprom Move display design forward Refactor control-dmx to dmx Update expansion connector on all boards Add test suites Add tx-retro readme Cleanup
Parts:
- removed U1: 74LS32, Package_DIP:DIP-14_W7.62mm, symbol 74xx:74LS32
- removed U2: 74LS00, Package_DIP:DIP-14_W7.62mm, symbol 74xx:74LS00
- added C10: 0.1uF, Capacitor_THT:C_Rect_L4.6mm_W2.0mm_P2.50mm_MKS02_FKP02, symbol Device:C_Small
- added C6, C7, C8: 0.1uF, Capacitor_THT:C_Rect_L4.6mm_W2.0mm_P2.50mm_MKS02_FKP02, symbol Device:C
- added C9: 10uF, Capacitor_THT:CP_Radial_D4.0mm_P1.50mm, symbol Device:CP1
- added R1: 10k, Resistor_THT:R_Axial_DIN0207_L6.3mm_D2.5mm_P10.16mm_Horizontal, symbol Device:R_US
- added U1, U2: 74LS161, Package_DIP:DIP-16_W7.62mm, symbol 74xx:74LS161
- added U6: 74LS273, Package_DIP:DIP-20_W7.62mm, symbol 74xx:74LS273
- added U7: 74LS32, Package_DIP:DIP-14_W7.62mm, symbol 74xx:74LS32
- C1, C2, C3, C4, C5: value .01uF -> 0.1uF
Connections:
- net labels added: CARRY_0, CARRY_1, CARRY_2, IA10, IA11, IA12, IA13, IA8, IA9
- wire segments 179 -> 238
- no-connect marks 26 -> 25
Other:
- note added: "Data\nLatch"
- note added: "Decoupling Capacitors"
- note added: "Frame Reset Value: 00000001b (0x01, 1d). This is the final instruction value in a packet;\nthe counter will reset and start the break again. This allows the data in U5 to determine when\nthe reset occurs, i.e., the timing of the reset can be programmed as part of the control instructions.\n\nIt's chosen because it's a value which is not used at any point in a real packet, i.e.,\n\nDATA_FIXED = Do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"
- note added: "Logic Ic Power"
- note added: "The address counters U1-U4 count from 0-16383 and that value is sent to U5, which uses that value\nto "lookup" the value to be sent to the control lines. U5 is programmed such that the value at address 0 \nis the instructions for the 1st bit in the packet, address 1 contains the instructions for the 2nd bit,...\n\n0-8191 is required since a DMX-512 packet needs 5670 bits minimum to form a complet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"
- note added: "This RC circuit will initialize the counters which presents the\ndata at address 0 to the latch. It also initializes the control \nlines to all 0's, which generates a ~FRAME_RESET~. The next\nclock pulse will reset the address counters (again) and load the\ndata at address 0 into the latch to start the frame."
- note removed: "Reset"
- note removed: "Reset: 10001101b (0x4d, 141d)\nThis is the final value in a packet. At this point,\nthe counter will reset and start the break again.\n\nIts' chosen because it's a value which is unlikely\nto be used in a packet, i.e. sample reset and latch \nany dimmer and shift load while enabled while \ntransmitting a break.\n"
