File: hardware/transmitter-retro/display/data.sch (KiCad schematic (older format))
At the start: 23 parts

Commit message: Prototype and PCB layout for core Prototype and PCB layout for demo Prototype and PCB layout for control-eprom Move display design forward Refactor control-dmx to dmx Update expansion connector on all boards Add test suites Add tx-retro readme Cleanup
Parts:
- removed BAR?: LED, Display:HDSP-4830, symbol LED:HDSP-4830_2
- removed RN?: 330, Resistor_THT:R_Array_SIP11, symbol Device:R_Network10_US
- removed RN? (x5): 330x8, Package_DIP:DIP-16_W7.62mm, symbol Device:R_Pack08
- removed U? (x5): MAN71A, Display_7Segment:MAN71A, symbol Display_Character:MAN71A
- removed U? (x5): 74LS47, Package_DIP:DIP-16_W7.62mm, symbol 74xx:74LS47
- removed U?: ULN2803A, symbol Transistor_Array:ULN2803A
- removed U?: 74LS161, Package_DIP:DIP-16_W7.62mm, symbol 74xx:74LS161
- removed U? (x2): 74LS162, Package_DIP:DIP-16_W7.62mm, symbol 74xx:74LS161
- removed U? (x2): 74LS373, symbol 74xx:74LS373
- added D?: D0, symbol Device:LED
- added D?: D2, symbol Device:LED
- added D?: D1, symbol Device:LED
- added D?: D4, symbol Device:LED
- added D?: D6, symbol Device:LED
- added D?: D5, symbol Device:LED
- added D?: D3, symbol Device:LED
- added D?: D7, symbol Device:LED
- added R? (x8): 330, symbol Device:R_US
- added U?: 74LS240, symbol 74xx:74LS240
Connections:
- net labels removed: CLK_TX_IN, IA0, IA1, IA2, IA3, IA4, IA5, IA6, IA7, LT, TA0, TA1, TA2, TA3, TA4, TA5, TA6, TA7, ~FRAME_RESET
- wire segments 259 -> 52
- no-connect marks 8 -> 0
Other:
- note removed: "Can we do this as 0-255?"
- note removed: "Can we show sampled and latched data?"
- note removed: "Data Value Display"
- note removed: "Do this for sure."
- note removed: "Step Value Display"
