File: hardware/transmitter-retro/display/display.sch (KiCad schematic (older format))
At the start: 1 part, among them J4 Expansion

Commit message: Prototype and PCB layout for core Prototype and PCB layout for demo Prototype and PCB layout for control-eprom Move display design forward Refactor control-dmx to dmx Update expansion connector on all boards Add test suites Add tx-retro readme Cleanup
Parts:
- removed J4: Expansion, Connector_PinHeader_2.54mm:PinHeader_2x20_P2.54mm_Vertical, symbol Connector_Generic:Conn_02x20_Odd_Even
- added J?: Expansion, Connector_PinHeader_2.54mm:PinHeader_2x20_P2.54mm_Vertical, symbol Connector_Generic:Conn_02x20_Odd_Even
Connections:
- net labels added: CLK_SAMPLE, DATA_SHIFT, SAMPLE_COUNT, ~CLK_FST, ~CLK_SLO, ~CLK_STEP, ~SAMPLE_OVERRIDE, ~SHIFT_ENABLE
- net labels removed: CLK_FAST, CLK_SLOW, SHIFT_DISABLE, ~SAMPLE_ASSERT
- wire segments 39 -> 87
- no-connect marks 9 -> 8
Other:
- note added: "Orig\nAddress - 8 bit\nClock\nData\nShift Register Output\nLatched Data - 8 bit\nSample Sel - 1-4\nFrame - 18 parts of the frame\nForce 0\nForce 1\n\n\nCurrent\nClock\nData\nFrame - 18 parts of the frame\nShift Register Output\nLatched Data - 8 bit\nSampel Latch\nSample Reset\nShift Load\n"
