File: hardware/transmitter-retro/display/power.sch (KiCad schematic (older format))
At the start: 23 parts

Commit message: Prototype and PCB layout for core Prototype and PCB layout for demo Prototype and PCB layout for control-eprom Move display design forward Refactor control-dmx to dmx Update expansion connector on all boards Add test suites Add tx-retro readme Cleanup
Parts:
- added U1: 74LS139, symbol 74xx:74LS139
- added U3, U4, U5: 74LS04, symbol 74xx:74LS04
