File: hardware/display-pro/display-pro.sch (KiCad schematic (older format))
At the start: 17 parts, among them J1 POWER_A, J2 POWER_B, J3 Input, J4 Output, J5 Clock, J6 Data, Q1 FQP30N06L, Q2 FQP30N06L

Commit message: Remove coax power jack from display-pro; the Sparkfun footprint does not nest inside the 2 pin connector so only providing that option.
Parts:
- removed J1: POWER_A, Connector_BarrelJack:BarrelJack_CUI_PJ-063AH_Horizontal, symbol Connector:Barrel_Jack
- J2: value POWER_B -> POWER
- Q1: footprint TO220V -> Package_TO_SOT_THT:TO-220-3_Horizontal_TabDown
Connections:
- wire segments 58 -> 53
Other:
- moved on the sheet: J2
Changed lines of the file:
@@
 Sheet 1 1
 Title "DMX Demonstrator - Display-Pro (DMX-DSP)"
-Date "2020-09-14"
-Rev "1.0"
+Date "2020-11-08"
+Rev "1.2"
 Comp "Crazy Giraffe Software"
 Comment1 ""
@@
 L Connector:Screw_Terminal_01x02 J2
 U 1 1 5F4DF77C
-P 4650 7300
-F 0 "J2" H 4570 7517 50  0000 C CNN
-F 1 "POWER_B" H 4570 7426 50  0000 C CNN
-F 2 "Connector_Phoenix_MSTB:PhoenixContact_MSTBA_2,5_2-G-5,08_1x02_P5.08mm_Horizontal" H 4650 7300 50  0001 C CNN
-F 3 "~" H 4650 7300 50  0001 C CNN
-	1    4650 7300
+P 4900 6700
+F 0 "J2" H 4800 6400 50  0000 C CNN
+F 1 "POWER" H 4800 6500 50  0000 C CNN
+F 2 "Connector_Phoenix_MSTB:PhoenixContact_MSTBA_2,5_2-G-5,08_1x02_P5.08mm_Horizontal" H 4900 6700 50  0001 C CNN
+F 3 "~" H 4900 6700 50  0001 C CNN
+	1    4900 6700
 	-1   0    0    1
-$EndComp
-$Comp
-L Connector:Barrel_Jack J1
-U 1 1 5F4DF88A
-P 4800 6700
-F 0 "J1" H 4855 7025 50  0000 C CNN
-F 1 "POWER_A" H 4855 6934 50  0000 C CNN
-F 2 "Connector_BarrelJack:BarrelJack_CUI_PJ-063AH_Horizontal" H 4850 6660 50  0001 C CNN
-F 3 "~" H 4850 6660 50  0001 C CNN
-	1    4800 6700
-	1    0    0    -1
 $EndComp
 $Comp
@@
 $EndComp
 Wire Wire Line
-	5100 6600 5300 6600
-Wire Wire Line
-	5100 6800 5200 6800
-Wire Wire Line
-	5200 6800 5200 7300
+	5100 6700 5200 6700
 $Comp
 L power:GND #PWR0103
@@
 	1    0    0    -1
 $EndComp
-Wire Wire Line
-	4850 7300 5200 7300
-Connection ~ 5200 7300
-Wire Wire Line
-	5200 7300 5200 7450
-Wire Wire Line
-	4850 7200 5300 7200
-Wire Wire Line
-	5300 7200 5300 6600
-Connection ~ 5300 6600
-Wire Wire Line
-	5300 6600 5400 6600
 $Comp
 L power:PWR_FLAG #FLG0102
@@
 F 0 "Q1" H 6765 2342 45  0000 L CNN
 F 1 "FQP30N06L" H 6765 2258 45  0000 L CNN
-F 2 "TO220V" H 6600 2550 20  0001 C CNN
+F 2 "Package_TO_SOT_THT:TO-220-3_Horizontal_TabDown" H 6600 2550 20  0001 C CNN
 F 3 "" H 6600 2300 50  0001 C CNN
 F 4 "TRANS-10060" H 6765 2216 60  0001 L CNN "Field4"
@@
 	1    0    0    -1
 $EndComp
+Wire Wire Line
+	5100 6600 5400 6600
+Wire Wire Line
+	5200 6700 5200 7450
 $EndSCHEMATC

Commit message: Add Coax power back to display board. Save gerbers settings for rx1, tx1, tx2. Update dsp & rx1 schematic pdf.
Parts:
- added J1: POWER_A, Connector_BarrelJack:BarrelJack_CUI_PJ-063AH_Horizontal, symbol Connector:Barrel_Jack
- J2: value POWER -> POWER_B
Connections:
- wire segments 53 -> 58
Other:
- moved on the sheet: J2
Changed lines of the file:
@@
 L Connector:Screw_Terminal_01x02 J2
 U 1 1 5F4DF77C
-P 4900 6700
-F 0 "J2" H 4800 6400 50  0000 C CNN
-F 1 "POWER" H 4800 6500 50  0000 C CNN
-F 2 "Connector_Phoenix_MSTB:PhoenixContact_MSTBA_2,5_2-G-5,08_1x02_P5.08mm_Horizontal" H 4900 6700 50  0001 C CNN
-F 3 "~" H 4900 6700 50  0001 C CNN
-	1    4900 6700
+P 4650 7300
+F 0 "J2" H 4550 7000 50  0000 C CNN
+F 1 "POWER_B" H 4550 7100 50  0000 C CNN
+F 2 "Connector_Phoenix_MSTB:PhoenixContact_MSTBA_2,5_2-G-5,08_1x02_P5.08mm_Horizontal" H 4650 7300 50  0001 C CNN
+F 3 "~" H 4650 7300 50  0001 C CNN
+	1    4650 7300
 	-1   0    0    1
 $EndComp
@@
 $EndComp
 Wire Wire Line
-	5100 6700 5200 6700
+	5100 6800 5200 6800
 $Comp
 L power:GND #PWR0103
@@
 $EndComp
 Wire Wire Line
-	5100 6600 5400 6600
-Wire Wire Line
-	5200 6700 5200 7450
+	5100 6600 5300 6600
+Wire Wire Line
+	5200 6800 5200 7300
+$Comp
+L Connector:Barrel_Jack J1
+U 1 1 64053ABC
+P 4800 6700
+F 0 "J1" H 4855 7025 50  0000 C CNN
+F 1 "POWER_A" H 4855 6934 50  0000 C CNN
+F 2 "Connector_BarrelJack:BarrelJack_CUI_PJ-063AH_Horizontal" H 4850 6660 50  0001 C CNN
+F 3 "~" H 4850 6660 50  0001 C CNN
+	1    4800 6700
+	1    0    0    -1
+$EndComp
+Wire Wire Line
+	4850 7300 5200 7300
+Connection ~ 5200 7300
+Wire Wire Line
+	5200 7300 5200 7450
+Wire Wire Line
+	4850 7200 5300 7200
+Wire Wire Line
+	5300 7200 5300 6600
+Connection ~ 5300 6600
+Wire Wire Line
+	5300 6600 5400 6600
 $EndSCHEMATC

Commit message: Make io-analog a stackable family io-analog-core handles D to A io-analog-amplify handles voltage output io-analog-pwm handles pwm output for leds, drive display pro io-analog-led handles 5v pwm output for iot, drive display pro
Refactor display-pro to work with io-analog-pwm
Add correct coax power connector
Parts:
- removed J1: POWER_A, Connector_BarrelJack:BarrelJack_CUI_PJ-063AH_Horizontal, symbol Connector:Barrel_Jack
- removed R3, R4: R?, Resistor_THT:R_Axial_DIN0411_L9.9mm_D3.6mm_P15.24mm_Horizontal, symbol Device:R_US
- added J4: Power, POWER_JACK_PTH_BREAD, symbol CrazyGiraffe_DMXDemonstrator:POWER_JACKPTH_BREAD
- J3: renamed from J2; value POWER_B -> Power
- J5: value Clock -> C Out
- J6: value Data -> D Out
- renumbered J3 to J1, J4 to J2
Connections:
- net labels added: C, D
- net labels removed: CLOCK, DATA
- wire segments 58 -> 40
Other:
- note removed: "Cut trace to\nuse resistor"
- moved on the sheet: D1, J3, MH1, MH2, MH3, MH4, R1, R2

Commit message: Display Pro: - Switch to smaller screw terminal connectors - Add pull-down resistors - Add silkscreen values - Remove COAX power connector...again - Add test software
Core:
- Fix issue with A03 and A02 being reversed at Analog Extensions
- Fix issue with A1 and A0 at IO Extension header
- Label D0..D7 correctly
- Swap U4 and U5 in schematic to match board layout
- Change TO-92 footprint
- Add silkscreen values
- Add test software

PWM:
- Switch to smaller screw terminal connectors
- Add silkscreen values
- Remove COAX power connector

Voltage:
- Switch to smaller screw terminal connectors
- Add silkscreen values
- Remove COAX power connector

DMX:
- Fix issue with DMX A and B being reversed
- Group bypass-only resistors together
- Add ISO bypass solder bridges
- Add silkscreen values
- Remove RDM bias resistors
- Add test software

Rx-IO:
- Fix issue with A1 and A0 at IO Extension header
- Add silkscreen values

Tx-IO:
- Switch to 74LS07 for Led driver
- Add pulldown resistor for discovery
- Add silkscreen values

Discovery:
- Make use of new Tx-IO pulldown resistor
Parts:
- removed J4: Power, POWER_JACK_PTH_BREAD, symbol CrazyGiraffe_DMXDemonstrator:POWER_JACKPTH_BREAD
- added R3, R4: 10k, Resistor_THT:R_Axial_DIN0207_L6.3mm_D2.5mm_P10.16mm_Horizontal, symbol Device:R_US
- J3, J5, J6: footprint Connector_Phoenix_MSTB:PhoenixContact_MSTBA_2,5_2-G-5,08_1x02_P5.08mm_Horizontal -> Connector_Phoenix_MC:PhoenixContact_MC_1,5_2-G-3.81_1x02_P3.81mm_Horizontal
Connections:
- wire segments 40 -> 41
Changed lines of the file:
@@
 Sheet 1 1
 Title "DMX Demonstrator - Display-Pro (DMX-DSP)"
-Date "2023-07-02"
-Rev "1.4"
+Date "2023-09-17"
+Rev "1.5"
 Comp "Crazy Giraffe Software"
 Comment1 ""
@@
 F 0 "J5" H 8050 1900 50  0000 L CNN
 F 1 "C Out" H 8050 2000 50  0000 L CNN
-F 2 "Connector_Phoenix_MSTB:PhoenixContact_MSTBA_2,5_2-G-5,08_1x02_P5.08mm_Horizontal" H 7950 2000 50  0001 C CNN
+F 2 "Connector_Phoenix_MC:PhoenixContact_MC_1,5_2-G-3.81_1x02_P3.81mm_Horizontal" H 7950 2000 50  0001 C CNN
 F 3 "~" H 7950 2000 50  0001 C CNN
 	1    7950 2000
@@
 L power:GND #PWR0101
 U 1 1 5F306EF9
-P 5150 5150
-F 0 "#PWR0101" H 5150 4900 50  0001 C CNN
-F 1 "GND" H 5155 4977 50  0000 C CNN
-F 2 "" H 5150 5150 50  0001 C CNN
-F 3 "" H 5150 5150 50  0001 C CNN
-	1    5150 5150
+P 5150 5450
+F 0 "#PWR0101" H 5150 5200 50  0001 C CNN
+F 1 "GND" H 5155 5277 50  0000 C CNN
+F 2 "" H 5150 5450 50  0001 C CNN
+F 3 "" H 5150 5450 50  0001 C CNN
+	1    5150 5450
 	-1   0    0    -1
 $EndComp
@@
 F 0 "J3" H 2800 6400 50  0000 C CNN
 F 1 "Power" H 2800 6500 50  0000 C CNN
-F 2 "Connector_Phoenix_MSTB:PhoenixContact_MSTBA_2,5_2-G-5,08_1x02_P5.08mm_Horizontal" H 2900 6700 50  0001 C CNN
+F 2 "Connector_Phoenix_MC:PhoenixContact_MC_1,5_2-G-3.81_1x02_P3.81mm_Horizontal" H 2900 6700 50  0001 C CNN
 F 3 "~" H 2900 6700 50  0001 C CNN
 	1    2900 6700
@@
 	4400 6600 4800 6600
 Wire Wire Line
-	5150 5150 5150 4850
+	5150 5450 5150 4850
 $Comp
 L Connector_Generic:Conn_01x03 J2
@@
 	4850 4950 6000 4950
 Wire Wire Line
-	6750 4850 6750 5150
+	6750 4850 6750 5450
 $Comp
 L power:GND #PWR0107
 U 1 1 5F61744A
-P 6750 5150
-F 0 "#PWR0107" H 6750 4900 50  0001 C CNN
-F 1 "GND" H 6755 4977 50  0000 C CNN
-F 2 "" H 6750 5150 50  0001 C CNN
-F 3 "" H 6750 5150 50  0001 C CNN
-	1    6750 5150
+P 6750 5450
+F 0 "#PWR0107" H 6750 5200 50  0001 C CNN
+F 1 "GND" H 6755 5277 50  0000 C CNN
+F 2 "" H 6750 5450 50  0001 C CNN
+F 3 "" H 6750 5450 50  0001 C CNN
+	1    6750 5450
 	-1   0    0    -1
 $EndComp
@@
 F 0 "J6" H 8050 3250 50  0000 L CNN
 F 1 "D Out" H 8050 3350 50  0000 L CNN
-F 2 "Connector_Phoenix_MSTB:PhoenixContact_MSTBA_2,5_2-G-5,08_1x02_P5.08mm_Horizontal" H 7950 3350 50  0001 C CNN
+F 2 "Connector_Phoenix_MC:PhoenixContact_MC_1,5_2-G-3.81_1x02_P3.81mm_Horizontal" H 7950 3350 50  0001 C CNN
 F 3 "~" H 7950 3350 50  0001 C CNN
 	1    7950 3350
@@
 $EndComp
 Wire Wire Line
-	3100 6600 3550 6600
-Wire Wire Line
 	3450 6700 3450 7300
-Wire Wire Line
-	3150 7300 3450 7300
 Connection ~ 3450 7300
 Wire Wire Line
-	3450 7300 3450 7400
-Wire Wire Line
-	3150 7200 3550 7200
-Wire Wire Line
-	3550 7200 3550 6600
-Connection ~ 3550 6600
-Wire Wire Line
-	3550 6600 3750 6600
-Wire Wire Line
 	6850 2500 6850 2600
 Wire Wire Line
@@
 Wire Wire Line
 	6850 2000 7750 2000
-$Comp
-L CrazyGiraffe_DMXDemonstrator:POWER_JACKPTH_BREAD J4
-U 1 1 64A270C6
-P 2950 7300
-F 0 "J4" H 2906 7584 45  0000 C CNN
-F 1 "Power" H 2906 7500 45  0000 C CNN
-F 2 "POWER_JACK_PTH_BREAD" H 2950 7550 20  0001 C CNN
-F 3 "" H 2950 7300 50  0001 C CNN
-F 4 "PRT-10811" H 2906 7511 60  0001 C CNN "Field4"
-	1    2950 7300
-	1    0    0    -1
-$EndComp
-Wire Wire Line
-	3150 7400 3450 7400
-Connection ~ 3450 7400
-Wire Wire Line
-	3450 7400 3450 7450
+Wire Wire Line
+	3450 7300 3450 7450
+Wire Wire Line
+	3100 6600 3750 6600
+$Comp
+L Device:R_US R3
+U 1 1 65438E92
+P 5800 5200
+F 0 "R3" H 5732 5154 50  0000 R CNN
+F 1 "10k" H 5732 5245 50  0000 R CNN
+F 2 "Resistor_THT:R_Axial_DIN0207_L6.3mm_D2.5mm_P10.16mm_Horizontal" V 5840 5190 50  0001 C CNN
+F 3 "~" H 5800 5200 50  0001 C CNN
+	1    5800 5200
+	1    0    0    1
+$EndComp
+$Comp
+L Device:R_US R4
+U 1 1 65438ED8
+P 6000 5200
+F 0 "R4" H 6068 5246 50  0000 L CNN
+F 1 "10k" H 6068 5155 50  0000 L CNN
+F 2 "Resistor_THT:R_Axial_DIN0207_L6.3mm_D2.5mm_P10.16mm_Horizontal" V 6040 5190 50  0001 C CNN
+F 3 "~" H 6000 5200 50  0001 C CNN
+	1    6000 5200
+	1    0    0    -1
+$EndComp
+$Comp
+L power:GND #PWR0102
+U 1 1 6543AC2F
+P 5900 5450
+F 0 "#PWR0102" H 5900 5200 50  0001 C CNN
+F 1 "GND" H 5905 5277 50  0000 C CNN
+F 2 "" H 5900 5450 50  0001 C CNN
+F 3 "" H 5900 5450 50  0001 C CNN
+	1    5900 5450
+	-1   0    0    -1
+$EndComp
+Wire Wire Line
+	5800 5350 5800 5400
+Wire Wire Line
+	5800 5400 5900 5400
+Wire Wire Line
+	6000 5400 6000 5350
+Wire Wire Line
+	5900 5450 5900 5400
+Connection ~ 5900 5400
+Wire Wire Line
+	5900 5400 6000 5400
+Wire Wire Line
+	6000 5050 6000 4950
+Wire Wire Line
+	5800 5050 5800 4750
 $EndSCHEMATC
