File: hardware/led-driver/voltage/led-driver-voltage.kicad_pcb (KiCad board)
At the start: 2 copper layers, 60 x 60 mm, 19 parts, among them J1 Input, J2 Output, J3 Power, J5 C Out, J6 D Out, Q1 FQP30N06L, Q2 FQP30N06L

Commit message: Rebranded.
Other:
- board text added: "DMX-DCV, Rev 1.6 Sparky Bobo Designs"
- board text removed: "DMX-DCV, Rev 1.6 Crazy Giraffe Software"
