File: hardware/led-driver/voltage/led-driver-voltage.sch (KiCad schematic (older format))
At the start: 17 parts, among them J1 Input, J2 Output, J3 Power, J5 C Out, J6 D Out, Q1 FQP30N06L, Q2 FQP30N06L

Commit message: Library fixup. Rebrand.
Parts:
- Q1, Q2: symbol SparkFun-DiscreteSemi:MOSFET-NCH-FQP30N06L -> DMXDemonstrator:MOSFET-NCH-FQP30N06L-SparkFun-DiscreteSemi
Changed lines of the file:
@@
 $EndComp
 $Comp
-L SparkFun-DiscreteSemi:MOSFET-NCH-FQP30N06L Q2
+L DMXDemonstrator:MOSFET-NCH-FQP30N06L-SparkFun-DiscreteSemi Q2
 U 1 1 5F63E22E
 P 6750 3650
@@
 $EndComp
 $Comp
-L SparkFun-DiscreteSemi:MOSFET-NCH-FQP30N06L Q1
+L DMXDemonstrator:MOSFET-NCH-FQP30N06L-SparkFun-DiscreteSemi Q1
 U 1 1 5F640FDC
 P 6750 2300

Commit message: Add parts and BOMs for rest of boards. Cleanup .md files.
Parts:
- J1: PartId (none) -> H_1x3_RA,JP_1x3
- J2: PartId (none) -> H_1x3_RA
- J3, J5, J6: PartId (none) -> J-381x2,P-381x2
- Q1, Q2: Field4 TRANS-10060 -> (none); PartId (none) -> Q_NMOSFET,HW-M3-6,HW-M3-NUT
- R1, R2, R3, R4: PartId (none) -> R_10k
Changed lines of the file:
@@
 F 2 "Connector_Phoenix_MC:PhoenixContact_MC_1,5_2-G-3.81_1x02_P3.81mm_Horizontal" H 7950 2000 50  0001 C CNN
 F 3 "~" H 7950 2000 50  0001 C CNN
+F 4 "J-381x2,P-381x2" H 7950 2000 50  0001 C CNN "PartId"
 	1    7950 2000
 	1    0    0    1
@@
 F 2 "Connector_PinHeader_2.54mm:PinHeader_1x03_P2.54mm_Horizontal" H 4650 4850 50  0001 C CNN
 F 3 "~" H 4650 4850 50  0001 C CNN
+F 4 "H_1x3_RA,JP_1x3" H 4650 4850 50  0001 C CNN "PartId"
 	1    4650 4850
 	-1   0    0    -1
@@
 F 2 "Connector_Phoenix_MC:PhoenixContact_MC_1,5_2-G-3.81_1x02_P3.81mm_Horizontal" H 4650 6700 50  0001 C CNN
 F 3 "~" H 4650 6700 50  0001 C CNN
+F 4 "J-381x2,P-381x2" H 4650 6700 50  0001 C CNN "PartId"
 	1    4650 6700
 	-1   0    0    1
@@
 F 2 "Resistor_THT:R_Axial_DIN0207_L6.3mm_D2.5mm_P10.16mm_Horizontal" V 6290 2390 50  0001 C CNN
 F 3 "~" H 6250 2400 50  0001 C CNN
+F 4 "R_10k" V 6250 2400 50  0001 C CNN "PartId"
 	1    6250 2400
 	0    1    1    0
@@
 F 2 "Resistor_THT:R_Axial_DIN0207_L6.3mm_D2.5mm_P10.16mm_Horizontal" V 6340 3740 50  0001 C CNN
 F 3 "~" H 6300 3750 50  0001 C CNN
+F 4 "R_10k" V 6300 3750 50  0001 C CNN "PartId"
 	1    6300 3750
 	0    1    1    0
@@
 F 2 "Connector_PinHeader_2.54mm:PinHeader_1x03_P2.54mm_Horizontal" H 7250 4850 50  0001 C CNN
 F 3 "~" H 7250 4850 50  0001 C CNN
+F 4 "H_1x3_RA" H 7250 4850 50  0001 C CNN "PartId"
 	1    7250 4850
 	1    0    0    -1
@@
 F 2 "Connector_Phoenix_MC:PhoenixContact_MC_1,5_2-G-3.81_1x02_P3.81mm_Horizontal" H 7950 3350 50  0001 C CNN
 F 3 "~" H 7950 3350 50  0001 C CNN
+F 4 "J-381x2,P-381x2" H 7950 3350 50  0001 C CNN "PartId"
 	1    7950 3350
 	1    0    0    1
@@
 $EndComp
 $Comp
-L DMXDemonstrator:MOSFET-NCH-FQP30N06L-SparkFun-DiscreteSemi Q2
-U 1 1 5F63E22E
-P 6750 3650
-F 0 "Q2" H 6915 3692 45  0000 L CNN
-F 1 "FQP30N06L" H 6915 3608 45  0000 L CNN
-F 2 "Package_TO_SOT_THT:TO-220-3_Horizontal_TabDown" H 6750 3900 20  0001 C CNN
-F 3 "" H 6750 3650 50  0001 C CNN
-F 4 "TRANS-10060" H 6915 3566 60  0001 L CNN "Field4"
-	1    6750 3650
-	1    0    0    -1
-$EndComp
-$Comp
 L DMXDemonstrator:MOSFET-NCH-FQP30N06L-SparkFun-DiscreteSemi Q1
 U 1 1 5F640FDC
@@
 F 2 "Package_TO_SOT_THT:TO-220-3_Horizontal_TabDown" H 6750 2550 20  0001 C CNN
 F 3 "" H 6750 2300 50  0001 C CNN
-F 4 "TRANS-10060" H 6915 2216 60  0001 L CNN "Field4"
+F 4 "Q_NMOSFET,HW-M3-6,HW-M3-NUT" H 6915 2216 60  0001 L CNN "PartId"
 	1    6750 2300
 	1    0    0    -1
@@
 F 2 "Resistor_THT:R_Axial_DIN0207_L6.3mm_D2.5mm_P10.16mm_Horizontal" V 5840 5190 50  0001 C CNN
 F 3 "~" H 5800 5200 50  0001 C CNN
+F 4 "R_10k" H 5800 5200 50  0001 C CNN "PartId"
 	1    5800 5200
 	1    0    0    1
@@
 F 2 "Resistor_THT:R_Axial_DIN0207_L6.3mm_D2.5mm_P10.16mm_Horizontal" V 6040 5190 50  0001 C CNN
 F 3 "~" H 6000 5200 50  0001 C CNN
+F 4 "R_10k" H 6000 5200 50  0001 C CNN "PartId"
 	1    6000 5200
 	1    0    0    -1
@@
 NoConn ~ 7450 3700
 NoConn ~ 7450 2350
+$Comp
+L DMXDemonstrator:MOSFET-NCH-FQP30N06L-SparkFun-DiscreteSemi Q2
+U 1 1 5F63E22E
+P 6750 3650
+F 0 "Q2" H 6915 3692 45  0000 L CNN
+F 1 "FQP30N06L" H 6915 3608 45  0000 L CNN
+F 2 "Package_TO_SOT_THT:TO-220-3_Horizontal_TabDown" H 6750 3900 20  0001 C CNN
+F 3 "" H 6750 3650 50  0001 C CNN
+F 4 "Q_NMOSFET,HW-M3-6,HW-M3-NUT" H 6915 3566 60  0001 L CNN "PartId"
+	1    6750 3650
+	1    0    0    -1
+$EndComp
 $EndSCHEMATC
