File: hardware/receiver/receiver.sch (KiCad schematic (older format))
At the start: 15 parts, among them J1 Input, J3 LED_B

Commit message: Rev 1.1: - Fixed arduino shield footprint (it was backwards) - Added Fcu power plane - New Fcu layouts - Added rounded corners
Parts:
- added D7: ERROR, LED_THT:LED_D5.0mm, symbol Device:LED
- added D8: START_CODE, LED_THT:LED_D5.0mm, symbol Device:LED
- added R7, R8: 330, Resistor_THT:R_Axial_DIN0207_L6.3mm_D2.5mm_P10.16mm_Horizontal, symbol Device:R_US
- A1: footprint Module:Arduino_UNO_R3 -> footprints:ARDUINO_R3_NO_HOLES
- D3: value DIM0 -> DIM3
- D4: value DIM1 -> DIM2
- D5: value DIM2 -> DIM1
- D6: value DIM3 -> DIM0
- J3: value LED_B -> LED_OUT
Connections:
- net labels added: ~ERR, ~SC
- wire segments 59 -> 71
- no-connect marks 19 -> 17
Other:
- moved on the sheet: D1, D2, R1, R2
Changed lines of the file:
@@
 Sheet 1 1
 Title "DMX Demonstrator - Receiver (DMX-RX1)"
-Date "2020-09-25"
-Rev "1.0"
+Date "2020-11-07"
+Rev "1.1"
 Comp "Crazy Giraffe Software"
 Comment1 ""
@@
 L Device:LED D1
 U 1 1 5F304057
-P 4500 3600
-F 0 "D1" H 4491 3816 50  0000 C CNN
-F 1 "DATA" H 4491 3725 50  0000 C CNN
-F 2 "LED_THT:LED_D5.0mm" H 4500 3600 50  0001 C CNN
-F 3 "~" H 4500 3600 50  0001 C CNN
-	1    4500 3600
+P 4450 2700
+F 0 "D1" H 4441 2916 50  0000 C CNN
+F 1 "DATA" H 4441 2825 50  0000 C CNN
+F 2 "LED_THT:LED_D5.0mm" H 4450 2700 50  0001 C CNN
+F 3 "~" H 4450 2700 50  0001 C CNN
+	1    4450 2700
 	-1   0    0    -1
 $EndComp
@@
 L Device:R_US R1
 U 1 1 5F3040DD
-P 4150 3600
-F 0 "R1" V 3945 3600 50  0000 C CNN
-F 1 "330" V 4036 3600 50  0000 C CNN
-F 2 "Resistor_THT:R_Axial_DIN0207_L6.3mm_D2.5mm_P10.16mm_Horizontal" V 4190 3590 50  0001 C CNN
-F 3 "~" H 4150 3600 50  0001 C CNN
-	1    4150 3600
+P 4100 2700
+F 0 "R1" V 3895 2700 50  0000 C CNN
+F 1 "330" V 3986 2700 50  0000 C CNN
+F 2 "Resistor_THT:R_Axial_DIN0207_L6.3mm_D2.5mm_P10.16mm_Horizontal" V 4140 2690 50  0001 C CNN
+F 3 "~" H 4100 2700 50  0001 C CNN
+	1    4100 2700
 	0    -1   1    0
 $EndComp
 Wire Wire Line
-	4350 3600 4300 3600
+	4300 2700 4250 2700
 $Comp
 L Device:LED D2
 U 1 1 5F3048EA
-P 4500 3950
-F 0 "D2" H 4491 4166 50  0000 C CNN
-F 1 "CLOCK" H 4491 4075 50  0000 C CNN
-F 2 "LED_THT:LED_D5.0mm" H 4500 3950 50  0001 C CNN
-F 3 "~" H 4500 3950 50  0001 C CNN
-	1    4500 3950
+P 4450 3050
+F 0 "D2" H 4441 3266 50  0000 C CNN
+F 1 "CLOCK" H 4441 3175 50  0000 C CNN
+F 2 "LED_THT:LED_D5.0mm" H 4450 3050 50  0001 C CNN
+F 3 "~" H 4450 3050 50  0001 C CNN
+	1    4450 3050
 	-1   0    0    -1
 $EndComp
@@
 L Device:R_US R2
 U 1 1 5F3048F0
-P 4150 3950
-F 0 "R2" V 3945 3950 50  0000 C CNN
-F 1 "330" V 4036 3950 50  0000 C CNN
-F 2 "Resistor_THT:R_Axial_DIN0207_L6.3mm_D2.5mm_P10.16mm_Horizontal" V 4190 3940 50  0001 C CNN
-F 3 "~" H 4150 3950 50  0001 C CNN
-	1    4150 3950
+P 4100 3050
+F 0 "R2" V 3895 3050 50  0000 C CNN
+F 1 "330" V 3986 3050 50  0000 C CNN
+F 2 "Resistor_THT:R_Axial_DIN0207_L6.3mm_D2.5mm_P10.16mm_Horizontal" V 4140 3040 50  0001 C CNN
+F 3 "~" H 4100 3050 50  0001 C CNN
+	1    4100 3050
 	0    -1   1    0
 $EndComp
 Wire Wire Line
-	4350 3950 4300 3950
+	4300 3050 4250 3050
 $Comp
 L power:+5V #PWR0101
@@
 $EndComp
 Wire Wire Line
-	4000 3600 3900 3600
-Wire Wire Line
-	4000 3950 3900 3950
-Connection ~ 3900 3600
+	3950 2700 3900 2700
+Wire Wire Line
+	3950 3050 3900 3050
+Connection ~ 3900 2700
 NoConn ~ 5200 3050
 NoConn ~ 6200 2850
 NoConn ~ 6200 2950
-Wire Wire Line
-	4650 3600 4850 3600
-Wire Wire Line
-	4850 3850 4850 3600
 Text Label 6250 3350 0    50   ~ 0
 ~DIM3
@@
 Text Label 6250 3950 0    50   ~ 0
 ~DIM0
-Wire Wire Line
-	4850 3850 5200 3850
 NoConn ~ 5200 3250
 Wire Wire Line
@@
 P 7200 4100
 F 0 "D3" H 7191 4316 50  0000 C CNN
-F 1 "DIM0" H 7191 4225 50  0000 C CNN
+F 1 "DIM3" H 7191 4225 50  0000 C CNN
 F 2 "LED_THT:LED_D5.0mm" H 7200 4100 50  0001 C CNN
 F 3 "~" H 7200 4100 50  0001 C CNN
@@
 P 7200 4450
 F 0 "D4" H 7191 4666 50  0000 C CNN
-F 1 "DIM1" H 7191 4575 50  0000 C CNN
+F 1 "DIM2" H 7191 4575 50  0000 C CNN
 F 2 "LED_THT:LED_D5.0mm" H 7200 4450 50  0001 C CNN
 F 3 "~" H 7200 4450 50  0001 C CNN
@@
 P 7200 4800
 F 0 "D5" H 7191 5016 50  0000 C CNN
-F 1 "DIM2" H 7191 4925 50  0000 C CNN
+F 1 "DIM1" H 7191 4925 50  0000 C CNN
 F 2 "LED_THT:LED_D5.0mm" H 7200 4800 50  0001 C CNN
 F 3 "~" H 7200 4800 50  0001 C CNN
@@
 P 7200 5150
 F 0 "D6" H 7191 5366 50  0000 C CNN
-F 1 "DIM3" H 7191 5275 50  0000 C CNN
+F 1 "DIM0" H 7191 5275 50  0000 C CNN
 F 2 "LED_THT:LED_D5.0mm" H 7200 5150 50  0001 C CNN
 F 3 "~" H 7200 5150 50  0001 C CNN
@@
 P 8250 3550
 F 0 "J3" H 8330 3592 50  0000 L CNN
-F 1 "LED_B" H 8330 3501 50  0000 L CNN
+F 1 "LED_OUT" H 8330 3501 50  0000 L CNN
 F 2 "Connector_Phoenix_MSTB:PhoenixContact_MSTBA_2,5_5-G-5,08_1x05_P5.08mm_Horizontal" H 8250 3550 50  0001 C CNN
 F 3 "~" H 8250 3550 50  0001 C CNN
@@
 Text Label 6250 4150 0    50   ~ 0
 RXCLK
-Wire Wire Line
-	6200 3350 6650 3350
-Wire Wire Line
-	6200 3450 6750 3450
 NoConn ~ 5800 2450
 NoConn ~ 6200 3250
@@
 F 0 "A1" H 5500 4500 50  0000 C CNN
 F 1 "Arduino_UNO_R3" H 5250 4400 50  0000 C CNN
-F 2 "Module:Arduino_UNO_R3" H 5850 2400 50  0001 L CNN
+F 2 "footprints:ARDUINO_R3_NO_HOLES" H 5850 2400 50  0001 L CNN
 F 3 "https://www.arduino.cc/en/Main/arduinoBoardUno" H 5500 4500 50  0001 C CNN
 	1    5700 3450
@@
 Wire Wire Line
 	6950 4100 7050 4100
-Wire Wire Line
-	6650 3350 6650 5150
-Wire Wire Line
-	6200 3950 6950 3950
-Wire Wire Line
-	6950 3950 6950 4100
-Wire Wire Line
-	6200 3850 6850 3850
-Wire Wire Line
-	6850 3850 6850 4450
 $Comp
 L power:+5V #PWR0104
 U 1 1 5F407263
-P 3900 3450
-F 0 "#PWR0104" H 3900 3300 50  0001 C CNN
-F 1 "+5V" H 3915 3623 50  0000 C CNN
-F 2 "" H 3900 3450 50  0001 C CNN
-F 3 "" H 3900 3450 50  0001 C CNN
-	1    3900 3450
-	-1   0    0    -1
-$EndComp
-Wire Wire Line
-	3900 3600 3900 3950
-Wire Wire Line
-	3900 3450 3900 3600
-NoConn ~ 5200 3750
+P 3900 2450
+F 0 "#PWR0104" H 3900 2300 50  0001 C CNN
+F 1 "+5V" H 3915 2623 50  0000 C CNN
+F 2 "" H 3900 2450 50  0001 C CNN
+F 3 "" H 3900 2450 50  0001 C CNN
+	1    3900 2450
+	-1   0    0    -1
+$EndComp
+Wire Wire Line
+	3900 2700 3900 3050
 Text Label 4950 3850 0    50   ~ 0
 ~DATA
@@
 	4350 5050 4350 5250
 Wire Wire Line
-	4650 3950 5200 3950
-NoConn ~ 5200 3650
+	4600 3050 4800 3050
 NoConn ~ 5200 3550
 NoConn ~ 5200 3450
 NoConn ~ 6200 3550
-NoConn ~ 6200 3650
-NoConn ~ 6200 3750
 $Comp
 L power:PWR_FLAG #FLG0101
@@
 Wire Wire Line
 	6550 7350 6550 7450
-Connection ~ 6950 3950
-Connection ~ 6850 3850
-Connection ~ 6750 3450
 Wire Wire Line
 	7950 5250 7950 5150
 Connection ~ 7950 5150
 Wire Wire Line
-	8050 3650 6950 3650
-Wire Wire Line
-	6850 3550 8050 3550
-Wire Wire Line
-	8050 3450 6750 3450
-Wire Wire Line
-	6750 3450 6750 4800
-Wire Wire Line
-	6850 3550 6850 3850
-Wire Wire Line
-	6950 3650 6950 3950
-Wire Wire Line
-	6650 3350 8050 3350
-Connection ~ 6650 3350
-Wire Wire Line
 	7950 3750 7950 4100
 Connection ~ 7950 4100
@@
 Wire Wire Line
 	4150 4950 6450 4950
+Connection ~ 6650 3950
+Wire Wire Line
+	6650 3950 6650 5150
+Connection ~ 6750 3850
+Wire Wire Line
+	6750 3850 6750 4800
+Wire Wire Line
+	6750 3550 8050 3550
+Wire Wire Line
+	6650 3650 6650 3950
+Wire Wire Line
+	6750 3550 6750 3850
+Wire Wire Line
+	6850 4450 6850 3450
+Connection ~ 6850 3450
+Wire Wire Line
+	6850 3450 8050 3450
+Wire Wire Line
+	6650 3650 8050 3650
+Wire Wire Line
+	6200 3350 6950 3350
+Wire Wire Line
+	6200 3450 6850 3450
+Wire Wire Line
+	6200 3950 6650 3950
+Wire Wire Line
+	6200 3850 6750 3850
+NoConn ~ 6200 3650
+NoConn ~ 6200 3750
+Wire Wire Line
+	6950 4100 6950 3350
+Wire Wire Line
+	6950 3350 8050 3350
+Connection ~ 6950 3350
+$Comp
+L Device:LED D7
+U 1 1 5FA8D6CC
+P 4450 3400
+F 0 "D7" H 4441 3616 50  0000 C CNN
+F 1 "ERROR" H 4441 3525 50  0000 C CNN
+F 2 "LED_THT:LED_D5.0mm" H 4450 3400 50  0001 C CNN
+F 3 "~" H 4450 3400 50  0001 C CNN
+	1    4450 3400
+	-1   0    0    -1
+$EndComp
+$Comp
+L Device:R_US R7
+U 1 1 5FA8D6D2
+P 4100 3400
+F 0 "R7" V 3895 3400 50  0000 C CNN
+F 1 "330" V 3986 3400 50  0000 C CNN
+F 2 "Resistor_THT:R_Axial_DIN0207_L6.3mm_D2.5mm_P10.16mm_Horizontal" V 4140 3390 50  0001 C CNN
+F 3 "~" H 4100 3400 50  0001 C CNN
+	1    4100 3400
+	0    -1   1    0
+$EndComp
+Wire Wire Line
+	4300 3400 4250 3400
+$Comp
+L Device:LED D8
+U 1 1 5FA8D6D9
+P 4450 3750
+F 0 "D8" H 4441 3966 50  0000 C CNN
+F 1 "START_CODE" H 4441 3875 50  0000 C CNN
+F 2 "LED_THT:LED_D5.0mm" H 4450 3750 50  0001 C CNN
+F 3 "~" H 4450 3750 50  0001 C CNN
+	1    4450 3750
+	-1   0    0    -1
+$EndComp
+$Comp
+L Device:R_US R8
+U 1 1 5FA8D6DF
+P 4100 3750
+F 0 "R8" V 3895 3750 50  0000 C CNN
+F 1 "330" V 3986 3750 50  0000 C CNN
+F 2 "Resistor_THT:R_Axial_DIN0207_L6.3mm_D2.5mm_P10.16mm_Horizontal" V 4140 3740 50  0001 C CNN
+F 3 "~" H 4100 3750 50  0001 C CNN
+	1    4100 3750
+	0    -1   1    0
+$EndComp
+Wire Wire Line
+	4300 3750 4250 3750
+Wire Wire Line
+	3950 3400 3900 3400
+Wire Wire Line
+	3950 3750 3900 3750
+Connection ~ 3900 3400
+Wire Wire Line
+	3900 3400 3900 3750
+Wire Wire Line
+	5200 3950 4800 3950
+Wire Wire Line
+	4900 3850 5200 3850
+Wire Wire Line
+	4600 2700 4900 2700
+Wire Wire Line
+	5200 3650 4700 3650
+Wire Wire Line
+	4700 3650 4700 3400
+Wire Wire Line
+	4600 3400 4700 3400
+Text Label 4950 3650 0    50   ~ 0
+~ERR
+Text Label 4950 3750 0    50   ~ 0
+~SC
+Wire Wire Line
+	4800 3050 4800 3950
+Wire Wire Line
+	4900 2700 4900 3850
+Wire Wire Line
+	3900 3050 3900 3400
+Connection ~ 3900 3050
+Wire Wire Line
+	3900 2450 3900 2700
+Wire Wire Line
+	4600 3750 5200 3750
 $EndSCHEMATC

Commit message: Users/sparky/txrx12 (#11)
* TX1 1.2, RX1 1.2
Move Clock LED to avoid ICSP connector.
Align TX Fast/Slo clock LEDS and RX start code/error LEDs.

* Add RXCLK to D9 connection for Leonardo PCINT5.

Co-authored-by: SparkyBobo <sparky@crazygiraffesoftware.com>
Connections:
- wire segments 71 -> 73
- no-connect marks 17 -> 16
Other:
- moved on the sheet: D3, D4, D5, D6, R3, R4, R5, R6
Changed lines of the file:
@@
 Sheet 1 1
 Title "DMX Demonstrator - Receiver (DMX-RX1)"
-Date "2020-11-07"
-Rev "1.1"
+Date "2020-12-30"
+Rev "1.2"
 Comp "Crazy Giraffe Software"
 Comment1 ""
@@
 NoConn ~ 6200 2850
 NoConn ~ 6200 2950
-Text Label 6250 3350 0    50   ~ 0
+Text Label 6200 3350 0    50   ~ 0
 ~DIM3
-Text Label 6250 3450 0    50   ~ 0
+Text Label 6200 3450 0    50   ~ 0
 ~DIM2
-Text Label 6250 3850 0    50   ~ 0
+Text Label 6200 3850 0    50   ~ 0
 ~DIM1
-Text Label 6250 3950 0    50   ~ 0
+Text Label 6200 3950 0    50   ~ 0
 ~DIM0
 NoConn ~ 5200 3250
 Wire Wire Line
-	6200 4150 6450 4150
-Wire Wire Line
-	6450 4150 6450 4950
-Wire Wire Line
-	6200 4050 6550 4050
-Wire Wire Line
-	6550 4050 6550 5150
-Wire Wire Line
-	6650 5150 7050 5150
-Wire Wire Line
-	6750 4800 7050 4800
-Wire Wire Line
-	6850 4450 7050 4450
+	6200 4150 6550 4150
+Wire Wire Line
+	6550 4150 6550 4950
+Wire Wire Line
+	6200 4050 6650 4050
+Wire Wire Line
+	6650 4050 6650 5150
+Wire Wire Line
+	6750 5150 7150 5150
+Wire Wire Line
+	6850 4800 7150 4800
+Wire Wire Line
+	6950 4450 7150 4450
 $Comp
 L Device:LED D3
 U 1 1 5F3BEC78
-P 7200 4100
-F 0 "D3" H 7191 4316 50  0000 C CNN
-F 1 "DIM3" H 7191 4225 50  0000 C CNN
-F 2 "LED_THT:LED_D5.0mm" H 7200 4100 50  0001 C CNN
-F 3 "~" H 7200 4100 50  0001 C CNN
-	1    7200 4100
+P 7300 4100
+F 0 "D3" H 7291 4316 50  0000 C CNN
+F 1 "DIM3" H 7291 4225 50  0000 C CNN
+F 2 "LED_THT:LED_D5.0mm" H 7300 4100 50  0001 C CNN
+F 3 "~" H 7300 4100 50  0001 C CNN
+	1    7300 4100
 	-1   0    0    -1
 $EndComp
@@
 L Device:R_US R3
 U 1 1 5F3BECD4
-P 7600 4100
-F 0 "R3" V 7395 4100 50  0000 C CNN
-F 1 "330" V 7486 4100 50  0000 C CNN
-F 2 "Resistor_THT:R_Axial_DIN0207_L6.3mm_D2.5mm_P10.16mm_Horizontal" V 7640 4090 50  0001 C CNN
-F 3 "~" H 7600 4100 50  0001 C CNN
-	1    7600 4100
+P 7700 4100
+F 0 "R3" V 7495 4100 50  0000 C CNN
+F 1 "330" V 7586 4100 50  0000 C CNN
+F 2 "Resistor_THT:R_Axial_DIN0207_L6.3mm_D2.5mm_P10.16mm_Horizontal" V 7740 4090 50  0001 C CNN
+F 3 "~" H 7700 4100 50  0001 C CNN
+	1    7700 4100
 	0    1    1    0
 $EndComp
@@
 L Device:LED D4
 U 1 1 5F3BFD29
-P 7200 4450
-F 0 "D4" H 7191 4666 50  0000 C CNN
-F 1 "DIM2" H 7191 4575 50  0000 C CNN
-F 2 "LED_THT:LED_D5.0mm" H 7200 4450 50  0001 C CNN
-F 3 "~" H 7200 4450 50  0001 C CNN
-	1    7200 4450
+P 7300 4450
+F 0 "D4" H 7291 4666 50  0000 C CNN
+F 1 "DIM2" H 7291 4575 50  0000 C CNN
+F 2 "LED_THT:LED_D5.0mm" H 7300 4450 50  0001 C CNN
+F 3 "~" H 7300 4450 50  0001 C CNN
+	1    7300 4450
 	-1   0    0    -1
 $EndComp
@@
 L Device:R_US R4
 U 1 1 5F3BFD2F
-P 7600 4450
-F 0 "R4" V 7395 4450 50  0000 C CNN
-F 1 "330" V 7486 4450 50  0000 C CNN
-F 2 "Resistor_THT:R_Axial_DIN0207_L6.3mm_D2.5mm_P10.16mm_Horizontal" V 7640 4440 50  0001 C CNN
-F 3 "~" H 7600 4450 50  0001 C CNN
-	1    7600 4450
+P 7700 4450
+F 0 "R4" V 7495 4450 50  0000 C CNN
+F 1 "330" V 7586 4450 50  0000 C CNN
+F 2 "Resistor_THT:R_Axial_DIN0207_L6.3mm_D2.5mm_P10.16mm_Horizontal" V 7740 4440 50  0001 C CNN
+F 3 "~" H 7700 4450 50  0001 C CNN
+	1    7700 4450
 	0    1    1    0
 $EndComp
@@
 L Device:LED D5
 U 1 1 5F3C1D16
-P 7200 4800
-F 0 "D5" H 7191 5016 50  0000 C CNN
-F 1 "DIM1" H 7191 4925 50  0000 C CNN
-F 2 "LED_THT:LED_D5.0mm" H 7200 4800 50  0001 C CNN
-F 3 "~" H 7200 4800 50  0001 C CNN
-	1    7200 4800
+P 7300 4800
+F 0 "D5" H 7291 5016 50  0000 C CNN
+F 1 "DIM1" H 7291 4925 50  0000 C CNN
+F 2 "LED_THT:LED_D5.0mm" H 7300 4800 50  0001 C CNN
+F 3 "~" H 7300 4800 50  0001 C CNN
+	1    7300 4800
 	-1   0    0    -1
 $EndComp
@@
 L Device:R_US R5
 U 1 1 5F3C1D1C
-P 7600 4800
-F 0 "R5" V 7395 4800 50  0000 C CNN
-F 1 "330" V 7486 4800 50  0000 C CNN
-F 2 "Resistor_THT:R_Axial_DIN0207_L6.3mm_D2.5mm_P10.16mm_Horizontal" V 7640 4790 50  0001 C CNN
-F 3 "~" H 7600 4800 50  0001 C CNN
-	1    7600 4800
+P 7700 4800
+F 0 "R5" V 7495 4800 50  0000 C CNN
+F 1 "330" V 7586 4800 50  0000 C CNN
+F 2 "Resistor_THT:R_Axial_DIN0207_L6.3mm_D2.5mm_P10.16mm_Horizontal" V 7740 4790 50  0001 C CNN
+F 3 "~" H 7700 4800 50  0001 C CNN
+	1    7700 4800
 	0    1    1    0
 $EndComp
@@
 L Device:LED D6
 U 1 1 5F3C1D22
-P 7200 5150
-F 0 "D6" H 7191 5366 50  0000 C CNN
-F 1 "DIM0" H 7191 5275 50  0000 C CNN
-F 2 "LED_THT:LED_D5.0mm" H 7200 5150 50  0001 C CNN
-F 3 "~" H 7200 5150 50  0001 C CNN
-	1    7200 5150
+P 7300 5150
+F 0 "D6" H 7291 5366 50  0000 C CNN
+F 1 "DIM0" H 7291 5275 50  0000 C CNN
+F 2 "LED_THT:LED_D5.0mm" H 7300 5150 50  0001 C CNN
+F 3 "~" H 7300 5150 50  0001 C CNN
+	1    7300 5150
 	-1   0    0    -1
 $EndComp
@@
 L Device:R_US R6
 U 1 1 5F3C1D28
-P 7600 5150
-F 0 "R6" V 7395 5150 50  0000 C CNN
-F 1 "330" V 7486 5150 50  0000 C CNN
-F 2 "Resistor_THT:R_Axial_DIN0207_L6.3mm_D2.5mm_P10.16mm_Horizontal" V 7640 5140 50  0001 C CNN
-F 3 "~" H 7600 5150 50  0001 C CNN
-	1    7600 5150
+P 7700 5150
+F 0 "R6" V 7495 5150 50  0000 C CNN
+F 1 "330" V 7586 5150 50  0000 C CNN
+F 2 "Resistor_THT:R_Axial_DIN0207_L6.3mm_D2.5mm_P10.16mm_Horizontal" V 7740 5140 50  0001 C CNN
+F 3 "~" H 7700 5150 50  0001 C CNN
+	1    7700 5150
 	0    1    1    0
 $EndComp
 Wire Wire Line
-	7750 4800 7950 4800
-Wire Wire Line
-	7350 5150 7450 5150
-Wire Wire Line
-	7750 5150 7950 5150
-Wire Wire Line
-	7350 4100 7450 4100
-Wire Wire Line
-	7750 4100 7950 4100
-Wire Wire Line
-	7350 4450 7450 4450
-Wire Wire Line
-	7750 4450 7950 4450
-Wire Wire Line
-	7350 4800 7450 4800
-Connection ~ 7950 4800
-Wire Wire Line
-	7950 4800 7950 5150
-Connection ~ 7950 4450
-Wire Wire Line
-	7950 4450 7950 4800
-Wire Wire Line
-	7950 4100 7950 4450
+	7850 4800 8050 4800
+Wire Wire Line
+	7450 5150 7550 5150
+Wire Wire Line
+	7850 5150 8050 5150
+Wire Wire Line
+	7450 4100 7550 4100
+Wire Wire Line
+	7850 4100 8050 4100
+Wire Wire Line
+	7450 4450 7550 4450
+Wire Wire Line
+	7850 4450 8050 4450
+Wire Wire Line
+	7450 4800 7550 4800
+Connection ~ 8050 4800
+Wire Wire Line
+	8050 4800 8050 5150
+Connection ~ 8050 4450
+Wire Wire Line
+	8050 4450 8050 4800
+Wire Wire Line
+	8050 4100 8050 4450
 $Comp
 L Connector:Screw_Terminal_01x05 J3
 U 1 1 5F42826E
-P 8250 3550
-F 0 "J3" H 8330 3592 50  0000 L CNN
-F 1 "LED_OUT" H 8330 3501 50  0000 L CNN
-F 2 "Connector_Phoenix_MSTB:PhoenixContact_MSTBA_2,5_5-G-5,08_1x05_P5.08mm_Horizontal" H 8250 3550 50  0001 C CNN
-F 3 "~" H 8250 3550 50  0001 C CNN
-	1    8250 3550
+P 8350 3550
+F 0 "J3" H 8430 3592 50  0000 L CNN
+F 1 "LED_OUT" H 8430 3501 50  0000 L CNN
+F 2 "Connector_Phoenix_MSTB:PhoenixContact_MSTBA_2,5_5-G-5,08_1x05_P5.08mm_Horizontal" H 8350 3550 50  0001 C CNN
+F 3 "~" H 8350 3550 50  0001 C CNN
+	1    8350 3550
 	1    0    0    1
 $EndComp
@@
 L power:GND #PWR0113
 U 1 1 5F443F49
-P 7950 5250
-F 0 "#PWR0113" H 7950 5000 50  0001 C CNN
-F 1 "GND" H 7955 5077 50  0000 C CNN
-F 2 "" H 7950 5250 50  0001 C CNN
-F 3 "" H 7950 5250 50  0001 C CNN
-	1    7950 5250
+P 8050 5250
+F 0 "#PWR0113" H 8050 5000 50  0001 C CNN
+F 1 "GND" H 8055 5077 50  0000 C CNN
+F 2 "" H 8050 5250 50  0001 C CNN
+F 3 "" H 8050 5250 50  0001 C CNN
+	1    8050 5250
 	1    0    0    -1
 $EndComp
 Wire Wire Line
-	8050 3750 7950 3750
-Text Label 6250 4050 0    50   ~ 0
+	8150 3750 8050 3750
+Text Label 6200 4050 0    50   ~ 0
 RX
-Text Label 6250 4150 0    50   ~ 0
+Text Label 6200 4150 0    50   ~ 0
 RXCLK
 NoConn ~ 5800 2450
@@
 D0-D4\nReserved\nFor DMX\nShield
 Wire Wire Line
-	6950 4100 7050 4100
+	7050 4100 7150 4100
 $Comp
 L power:+5V #PWR0104
@@
 	6550 7350 6550 7450
 Wire Wire Line
-	7950 5250 7950 5150
-Connection ~ 7950 5150
-Wire Wire Line
-	7950 3750 7950 4100
-Connection ~ 7950 4100
-Wire Wire Line
-	4150 5150 6550 5150
-Wire Wire Line
-	4150 4950 6450 4950
-Connection ~ 6650 3950
-Wire Wire Line
-	6650 3950 6650 5150
-Connection ~ 6750 3850
-Wire Wire Line
-	6750 3850 6750 4800
-Wire Wire Line
-	6750 3550 8050 3550
-Wire Wire Line
-	6650 3650 6650 3950
-Wire Wire Line
-	6750 3550 6750 3850
-Wire Wire Line
-	6850 4450 6850 3450
-Connection ~ 6850 3450
-Wire Wire Line
-	6850 3450 8050 3450
-Wire Wire Line
-	6650 3650 8050 3650
-Wire Wire Line
-	6200 3350 6950 3350
-Wire Wire Line
-	6200 3450 6850 3450
-Wire Wire Line
-	6200 3950 6650 3950
-Wire Wire Line
-	6200 3850 6750 3850
+	8050 5250 8050 5150
+Connection ~ 8050 5150
+Wire Wire Line
+	8050 3750 8050 4100
+Connection ~ 8050 4100
+Wire Wire Line
+	4150 5150 6650 5150
+Wire Wire Line
+	4150 4950 6550 4950
+Connection ~ 6750 3950
+Wire Wire Line
+	6750 3950 6750 5150
+Connection ~ 6850 3850
+Wire Wire Line
+	6850 3850 6850 4800
+Wire Wire Line
+	6850 3550 8150 3550
+Wire Wire Line
+	6750 3650 6750 3950
+Wire Wire Line
+	6850 3550 6850 3850
+Wire Wire Line
+	6950 4450 6950 3450
+Connection ~ 6950 3450
+Wire Wire Line
+	6950 3450 8150 3450
+Wire Wire Line
+	6750 3650 8150 3650
 NoConn ~ 6200 3650
-NoConn ~ 6200 3750
-Wire Wire Line
-	6950 4100 6950 3350
-Wire Wire Line
-	6950 3350 8050 3350
-Connection ~ 6950 3350
+Wire Wire Line
+	7050 4100 7050 3350
+Wire Wire Line
+	7050 3350 8150 3350
 $Comp
 L Device:LED D7
@@
 Wire Wire Line
 	4600 3750 5200 3750
+Connection ~ 7050 3350
+Wire Wire Line
+	6550 4150 6550 3750
+Wire Wire Line
+	6550 3750 6200 3750
+Connection ~ 6550 4150
+Wire Wire Line
+	6200 3950 6750 3950
+Wire Wire Line
+	6200 3850 6850 3850
+Wire Wire Line
+	6200 3450 6950 3450
+Wire Wire Line
+	6200 3350 7050 3350
 $EndSCHEMATC
