File: hardware/receiver/receiver.sch (KiCad schematic (older format))
At the start: 19 parts, among them J1 Input, J3 LED_OUT

Commit message: Final tweaks to TX1 and RX1 based on construction. (#17)
* Improve surface areea of power plane.

* Add design badges
Remove PWM connect from RX1
Update TX1 board details

commit 6da493b019dfdde530e2737d5f7a25deacfc908e
Author: SparkyBobo <sparky@crazygiraffesoftware.com>
Date:   Sat Dec 23 15:05:08 2023 -0800

    Removing test code for io-modules
    Will re-add with a better directory structure at a later time.

commit b72ab0594753e08691ac3616bc0f5ada6908d406
Author: SparkyBobo <sparky@crazygiraffesoftware.com>
Date:   Tue Dec 19 16:54:35 2023 -0800

    Tweaks boards based on construction notes

commit 602837d9dbb6f727bbb7a236c7c3e837e53ecbe9
Author: SparkyBobo <sparky@crazygiraffesoftware.com>
Date:   Tue Dec 5 23:41:07 2023 -0800

    Update silk screen.

commit a51c91a46e9f89e3931cecfd64c2200cc67d3a55
Author: SparkyBobo <sparky@crazygiraffesoftware.com>
Date:   Mon Oct 30 00:06:53 2023 -0700

    Display Pro:
    - Switch to smaller screw terminal connectors
    - Add pull-down resistors
    - Add silkscreen values
    - Remove COAX power connector...again
    - Add test software

    Core:
    - Fix issue with A03 and A02 being reversed at Analog Extensions
    - Fix issue with A1 and A0 at IO Extension header
    - Label D0..D7 correctly
    - Swap U4 and U5 in schematic to match board layout
    - Change TO-92 footprint
    - Add silkscreen values
    - Add test software

    PWM:
    - Switch to smaller screw terminal connectors
    - Add silkscreen values
    - Remove COAX power connector

    Voltage:
    - Switch to smaller screw terminal connectors
    - Add silkscreen values
    - Remove COAX power connector

    DMX:
    - Fix issue with DMX A and B being reversed
    - Group bypass-only resistors together
    - Add ISO bypass solder bridges
    - Add silkscreen values
    - Remove RDM bias resistors
    - Add test software

    Rx-IO:
    - Fix issue with A1 and A0 at IO Extension head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
Parts:
- removed J3: LED_OUT, Connector_Phoenix_MSTB:PhoenixContact_MSTBA_2,5_5-G-5,08_1x05_P5.08mm_Horizontal, symbol Connector:Screw_Terminal_01x05
Connections:
- wire segments 73 -> 61
Other:
- note removed: "D0-D4\nReserved\nFor DMX\nShield"
- moved on the sheet: D3, D4, D5, D6, R3, R4, R5, R6
Changed lines of the file:
@@
 Sheet 1 1
 Title "DMX Demonstrator - Receiver (DMX-RX1)"
-Date "2020-12-30"
-Rev "1.2"
+Date "2023-03-02"
+Rev "1.3"
 Comp "Crazy Giraffe Software"
 Comment1 ""
@@
 	6650 4050 6650 5150
 Wire Wire Line
-	6750 5150 7150 5150
-Wire Wire Line
-	6850 4800 7150 4800
-Wire Wire Line
-	6950 4450 7150 4450
+	6950 4250 7150 4250
 $Comp
 L Device:LED D3
 U 1 1 5F3BEC78
-P 7300 4100
-F 0 "D3" H 7291 4316 50  0000 C CNN
-F 1 "DIM3" H 7291 4225 50  0000 C CNN
-F 2 "LED_THT:LED_D5.0mm" H 7300 4100 50  0001 C CNN
-F 3 "~" H 7300 4100 50  0001 C CNN
-	1    7300 4100
+P 7300 3050
+F 0 "D3" H 7291 3266 50  0000 C CNN
+F 1 "DIM3" H 7291 3175 50  0000 C CNN
+F 2 "LED_THT:LED_D5.0mm" H 7300 3050 50  0001 C CNN
+F 3 "~" H 7300 3050 50  0001 C CNN
+	1    7300 3050
 	-1   0    0    -1
 $EndComp
@@
 L Device:R_US R3
 U 1 1 5F3BECD4
-P 7700 4100
-F 0 "R3" V 7495 4100 50  0000 C CNN
-F 1 "330" V 7586 4100 50  0000 C CNN
-F 2 "Resistor_THT:R_Axial_DIN0207_L6.3mm_D2.5mm_P10.16mm_Horizontal" V 7740 4090 50  0001 C CNN
-F 3 "~" H 7700 4100 50  0001 C CNN
-	1    7700 4100
+P 7700 3050
+F 0 "R3" V 7495 3050 50  0000 C CNN
+F 1 "330" V 7586 3050 50  0000 C CNN
+F 2 "Resistor_THT:R_Axial_DIN0207_L6.3mm_D2.5mm_P10.16mm_Horizontal" V 7740 3040 50  0001 C CNN
+F 3 "~" H 7700 3050 50  0001 C CNN
+	1    7700 3050
 	0    1    1    0
 $EndComp
@@
 L Device:LED D4
 U 1 1 5F3BFD29
-P 7300 4450
-F 0 "D4" H 7291 4666 50  0000 C CNN
-F 1 "DIM2" H 7291 4575 50  0000 C CNN
-F 2 "LED_THT:LED_D5.0mm" H 7300 4450 50  0001 C CNN
-F 3 "~" H 7300 4450 50  0001 C CNN
-	1    7300 4450
+P 7300 3450
+F 0 "D4" H 7291 3666 50  0000 C CNN
+F 1 "DIM2" H 7291 3575 50  0000 C CNN
+F 2 "LED_THT:LED_D5.0mm" H 7300 3450 50  0001 C CNN
+F 3 "~" H 7300 3450 50  0001 C CNN
+	1    7300 3450
 	-1   0    0    -1
 $EndComp
@@
 L Device:R_US R4
 U 1 1 5F3BFD2F
-P 7700 4450
-F 0 "R4" V 7495 4450 50  0000 C CNN
-F 1 "330" V 7586 4450 50  0000 C CNN
-F 2 "Resistor_THT:R_Axial_DIN0207_L6.3mm_D2.5mm_P10.16mm_Horizontal" V 7740 4440 50  0001 C CNN
-F 3 "~" H 7700 4450 50  0001 C CNN
-	1    7700 4450
+P 7700 3450
+F 0 "R4" V 7495 3450 50  0000 C CNN
+F 1 "330" V 7586 3450 50  0000 C CNN
+F 2 "Resistor_THT:R_Axial_DIN0207_L6.3mm_D2.5mm_P10.16mm_Horizontal" V 7740 3440 50  0001 C CNN
+F 3 "~" H 7700 3450 50  0001 C CNN
+	1    7700 3450
 	0    1    1    0
 $EndComp
@@
 L Device:LED D5
 U 1 1 5F3C1D16
-P 7300 4800
-F 0 "D5" H 7291 5016 50  0000 C CNN
-F 1 "DIM1" H 7291 4925 50  0000 C CNN
-F 2 "LED_THT:LED_D5.0mm" H 7300 4800 50  0001 C CNN
-F 3 "~" H 7300 4800 50  0001 C CNN
-	1    7300 4800
+P 7300 3850
+F 0 "D5" H 7291 4066 50  0000 C CNN
+F 1 "DIM1" H 7291 3975 50  0000 C CNN
+F 2 "LED_THT:LED_D5.0mm" H 7300 3850 50  0001 C CNN
+F 3 "~" H 7300 3850 50  0001 C CNN
+	1    7300 3850
 	-1   0    0    -1
 $EndComp
@@
 L Device:R_US R5
 U 1 1 5F3C1D1C
-P 7700 4800
-F 0 "R5" V 7495 4800 50  0000 C CNN
-F 1 "330" V 7586 4800 50  0000 C CNN
-F 2 "Resistor_THT:R_Axial_DIN0207_L6.3mm_D2.5mm_P10.16mm_Horizontal" V 7740 4790 50  0001 C CNN
-F 3 "~" H 7700 4800 50  0001 C CNN
-	1    7700 4800
+P 7700 3850
+F 0 "R5" V 7495 3850 50  0000 C CNN
+F 1 "330" V 7586 3850 50  0000 C CNN
+F 2 "Resistor_THT:R_Axial_DIN0207_L6.3mm_D2.5mm_P10.16mm_Horizontal" V 7740 3840 50  0001 C CNN
+F 3 "~" H 7700 3850 50  0001 C CNN
+	1    7700 3850
 	0    1    1    0
 $EndComp
@@
 L Device:LED D6
 U 1 1 5F3C1D22
-P 7300 5150
-F 0 "D6" H 7291 5366 50  0000 C CNN
-F 1 "DIM0" H 7291 5275 50  0000 C CNN
-F 2 "LED_THT:LED_D5.0mm" H 7300 5150 50  0001 C CNN
-F 3 "~" H 7300 5150 50  0001 C CNN
-	1    7300 5150
+P 7300 4250
+F 0 "D6" H 7291 4466 50  0000 C CNN
+F 1 "DIM0" H 7291 4375 50  0000 C CNN
+F 2 "LED_THT:LED_D5.0mm" H 7300 4250 50  0001 C CNN
+F 3 "~" H 7300 4250 50  0001 C CNN
+	1    7300 4250
 	-1   0    0    -1
 $EndComp
@@
 L Device:R_US R6
 U 1 1 5F3C1D28
-P 7700 5150
-F 0 "R6" V 7495 5150 50  0000 C CNN
-F 1 "330" V 7586 5150 50  0000 C CNN
-F 2 "Resistor_THT:R_Axial_DIN0207_L6.3mm_D2.5mm_P10.16mm_Horizontal" V 7740 5140 50  0001 C CNN
-F 3 "~" H 7700 5150 50  0001 C CNN
-	1    7700 5150
+P 7700 4250
+F 0 "R6" V 7495 4250 50  0000 C CNN
+F 1 "330" V 7586 4250 50  0000 C CNN
+F 2 "Resistor_THT:R_Axial_DIN0207_L6.3mm_D2.5mm_P10.16mm_Horizontal" V 7740 4240 50  0001 C CNN
+F 3 "~" H 7700 4250 50  0001 C CNN
+	1    7700 4250
 	0    1    1    0
 $EndComp
 Wire Wire Line
-	7850 4800 8050 4800
-Wire Wire Line
-	7450 5150 7550 5150
-Wire Wire Line
-	7850 5150 8050 5150
-Wire Wire Line
-	7450 4100 7550 4100
-Wire Wire Line
-	7850 4100 8050 4100
-Wire Wire Line
-	7450 4450 7550 4450
-Wire Wire Line
-	7850 4450 8050 4450
-Wire Wire Line
-	7450 4800 7550 4800
-Connection ~ 8050 4800
-Wire Wire Line
-	8050 4800 8050 5150
-Connection ~ 8050 4450
-Wire Wire Line
-	8050 4450 8050 4800
-Wire Wire Line
-	8050 4100 8050 4450
-$Comp
-L Connector:Screw_Terminal_01x05 J3
-U 1 1 5F42826E
-P 8350 3550
-F 0 "J3" H 8430 3592 50  0000 L CNN
-F 1 "LED_OUT" H 8430 3501 50  0000 L CNN
-F 2 "Connector_Phoenix_MSTB:PhoenixContact_MSTBA_2,5_5-G-5,08_1x05_P5.08mm_Horizontal" H 8350 3550 50  0001 C CNN
-F 3 "~" H 8350 3550 50  0001 C CNN
-	1    8350 3550
-	1    0    0    1
-$EndComp
+	7850 3850 8050 3850
+Wire Wire Line
+	7450 4250 7550 4250
+Wire Wire Line
+	7850 4250 8050 4250
+Wire Wire Line
+	7450 3050 7550 3050
+Wire Wire Line
+	7850 3050 8050 3050
+Wire Wire Line
+	7450 3450 7550 3450
+Wire Wire Line
+	7850 3450 8050 3450
+Wire Wire Line
+	7450 3850 7550 3850
+Wire Wire Line
+	8050 3850 8050 4250
+Wire Wire Line
+	8050 3050 8050 3450
 $Comp
 L power:GND #PWR0113
 U 1 1 5F443F49
-P 8050 5250
-F 0 "#PWR0113" H 8050 5000 50  0001 C CNN
-F 1 "GND" H 8055 5077 50  0000 C CNN
-F 2 "" H 8050 5250 50  0001 C CNN
-F 3 "" H 8050 5250 50  0001 C CNN
-	1    8050 5250
+P 8050 4350
+F 0 "#PWR0113" H 8050 4100 50  0001 C CNN
+F 1 "GND" H 8055 4177 50  0000 C CNN
+F 2 "" H 8050 4350 50  0001 C CNN
+F 3 "" H 8050 4350 50  0001 C CNN
+	1    8050 4350
 	1    0    0    -1
 $EndComp
-Wire Wire Line
-	8150 3750 8050 3750
 Text Label 6200 4050 0    50   ~ 0
 RX
@@
 	-1   0    0    -1
 $EndComp
-Text Notes 6300 3200 0    50   ~ 0
-D0-D4\nReserved\nFor DMX\nShield
-Wire Wire Line
-	7050 4100 7150 4100
 $Comp
 L power:+5V #PWR0104
@@
 	6550 7350 6550 7450
 Wire Wire Line
-	8050 5250 8050 5150
-Connection ~ 8050 5150
-Wire Wire Line
-	8050 3750 8050 4100
-Connection ~ 8050 4100
+	8050 4350 8050 4250
+Connection ~ 8050 4250
 Wire Wire Line
 	4150 5150 6650 5150
 Wire Wire Line
 	4150 4950 6550 4950
-Connection ~ 6750 3950
-Wire Wire Line
-	6750 3950 6750 5150
-Connection ~ 6850 3850
-Wire Wire Line
-	6850 3850 6850 4800
-Wire Wire Line
-	6850 3550 8150 3550
-Wire Wire Line
-	6750 3650 6750 3950
-Wire Wire Line
-	6850 3550 6850 3850
-Wire Wire Line
-	6950 4450 6950 3450
-Connection ~ 6950 3450
-Wire Wire Line
-	6950 3450 8150 3450
-Wire Wire Line
-	6750 3650 8150 3650
 NoConn ~ 6200 3650
-Wire Wire Line
-	7050 4100 7050 3350
-Wire Wire Line
-	7050 3350 8150 3350
 $Comp
 L Device:LED D7
@@
 Wire Wire Line
 	4600 3750 5200 3750
-Connection ~ 7050 3350
 Wire Wire Line
 	6550 4150 6550 3750
@@
 Connection ~ 6550 4150
 Wire Wire Line
-	6200 3950 6750 3950
-Wire Wire Line
-	6200 3850 6850 3850
-Wire Wire Line
-	6200 3450 6950 3450
-Wire Wire Line
-	6200 3350 7050 3350
+	6200 3950 6950 3950
+Wire Wire Line
+	6200 3350 6950 3350
+Connection ~ 8050 3450
+Wire Wire Line
+	8050 3450 8050 3850
+Connection ~ 8050 3850
+Wire Wire Line
+	6200 3850 7150 3850
+Wire Wire Line
+	6200 3450 7150 3450
+Wire Wire Line
+	6950 3950 6950 4250
+Wire Wire Line
+	6950 3350 6950 3050
+Wire Wire Line
+	6950 3050 7150 3050
+Text Label 6200 3750 0    50   ~ 0
+RXCLK
 $EndSCHEMATC

Commit message: Create constant voltage (formerly display-pro) led driver Create constant current led driver Add PWM outputs for led drivers to the receiver
Parts:
- added J2: PWM-34, Connector_PinHeader_2.54mm:PinHeader_1x03_P2.54mm_Horizontal, symbol Connector_Generic:Conn_01x03
- added J3: PWM_12, Connector_PinHeader_2.54mm:PinHeader_1x03_P2.54mm_Horizontal, symbol Connector_Generic:Conn_01x03
Connections:
- wire segments 61 -> 75
Changed lines of the file:
@@
 EESchema Schematic File Version 4
-LIBS:receiver-cache
-EELAYER 26 0
+EELAYER 30 0
 EELAYER END
 $Descr A4 11693 8268
@@
 L power:GND #PWR0113
 U 1 1 5F443F49
-P 8050 4350
-F 0 "#PWR0113" H 8050 4100 50  0001 C CNN
-F 1 "GND" H 8055 4177 50  0000 C CNN
-F 2 "" H 8050 4350 50  0001 C CNN
-F 3 "" H 8050 4350 50  0001 C CNN
-	1    8050 4350
+P 8050 5250
+F 0 "#PWR0113" H 8050 5000 50  0001 C CNN
+F 1 "GND" H 8055 5077 50  0000 C CNN
+F 2 "" H 8050 5250 50  0001 C CNN
+F 3 "" H 8050 5250 50  0001 C CNN
+	1    8050 5250
 	1    0    0    -1
 $EndComp
@@
 Wire Wire Line
 	6550 7350 6550 7450
-Wire Wire Line
-	8050 4350 8050 4250
 Connection ~ 8050 4250
 Wire Wire Line
@@
 Connection ~ 8050 3850
 Wire Wire Line
-	6200 3850 7150 3850
-Wire Wire Line
-	6200 3450 7150 3450
+	6200 3850 6850 3850
+Wire Wire Line
+	6200 3450 6850 3450
 Wire Wire Line
 	6950 3950 6950 4250
@@
 Text Label 6200 3750 0    50   ~ 0
 RXCLK
+$Comp
+L Connector_Generic:Conn_01x03 J2
+U 1 1 65A47C21
+P 8550 2650
+F 0 "J2" H 8700 2600 50  0000 C CNN
+F 1 "PWM-34" H 8800 2700 50  0000 C CNN
+F 2 "Connector_PinHeader_2.54mm:PinHeader_1x03_P2.54mm_Horizontal" H 8550 2650 50  0001 C CNN
+F 3 "~" H 8550 2650 50  0001 C CNN
+	1    8550 2650
+	1    0    0    1
+$EndComp
+$Comp
+L Connector_Generic:Conn_01x03 J3
+U 1 1 65A481BA
+P 8550 5050
+F 0 "J3" H 8700 5000 50  0000 C CNN
+F 1 "PWM_12" H 8800 5100 50  0000 C CNN
+F 2 "Connector_PinHeader_2.54mm:PinHeader_1x03_P2.54mm_Horizontal" H 8550 5050 50  0001 C CNN
+F 3 "~" H 8550 5050 50  0001 C CNN
+	1    8550 5050
+	1    0    0    1
+$EndComp
+Wire Wire Line
+	8350 2650 8050 2650
+Wire Wire Line
+	8050 2650 8050 3050
+Connection ~ 8050 3050
+Wire Wire Line
+	8350 2750 6950 2750
+Wire Wire Line
+	6950 2750 6950 3050
+Connection ~ 6950 3050
+Wire Wire Line
+	8350 2550 6850 2550
+Wire Wire Line
+	6850 2550 6850 3450
+Connection ~ 6850 3450
+Wire Wire Line
+	6850 3450 7150 3450
+Wire Wire Line
+	6950 4250 6950 4950
+Wire Wire Line
+	6950 4950 8350 4950
+Connection ~ 6950 4250
+Wire Wire Line
+	8350 5150 6850 5150
+Wire Wire Line
+	6850 5150 6850 3850
+Connection ~ 6850 3850
+Wire Wire Line
+	6850 3850 7150 3850
+Wire Wire Line
+	8050 5250 8050 5050
+Wire Wire Line
+	8050 5050 8350 5050
+Wire Wire Line
+	8050 4250 8050 5050
+Connection ~ 8050 5050
 $EndSCHEMATC
