File: hardware/control-pro/clock-faceplate/clock-faceplate.kicad_pcb (KiCad board)
At the start: 2 copper layers, 100 x 90 mm, 11 parts

Commit message: Rebrand to Sparky Bobo Designs
Other:
- board text added: "DMX-CPCF, Rev 1.3 Sparky Bobo Designs"
- board text removed: "DMX-CPCF, Rev 1.3 Crazy Giraffe Software"
Changed lines of the file:
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@@
     (date 2023-12-04)
     (rev 1.3)
-    (company "Crazy Giraffe Software")
+    (company "Sparky Bobo Designs")
     (comment 2 "Designed by: SparkyBobo")
     (comment 3 https://creativecommons.org/licenses/by-sa/4.0/)
@@
     (effects (font (size 1.5 1.5) (thickness 0.3)))
   )
-  (gr_text "DMX-CPCF, Rev 1.3\nCrazy Giraffe Software" (at 160.414 136.102) (layer B.SilkS)
+  (gr_text "DMX-CPCF, Rev 1.3\nSparky Bobo Designs" (at 160.414 136.102) (layer B.SilkS)
     (effects (font (size 1 1) (thickness 0.15)) (justify mirror))
   )
