File: hardware/control-pro/clock-faceplate/clock-faceplate.sch (KiCad schematic (older format))
At the start: 17 parts

Commit message: Users/sparky/hwcleanup (#22)
* Rename control-pro
Update readmes
Delete old pngs

* Add PWM headers on DMX-RX1.

* Add BOM generator
Add BOM and parts .md's
Parts:
- MH1, MH2, MH3, MH4: PartId (none) -> HW-M3-8
Changed lines of the file:
@@
 EESchema Schematic File Version 4
-LIBS:clock-faceplate-cache
-EELAYER 26 0
+EELAYER 30 0
 EELAYER END
 $Descr A4 11693 8268
@@
 F 2 "MountingHole:MountingHole_3.2mm_M3" H 6200 6600 50  0001 C CNN
 F 3 "~" H 6200 6600 50  0001 C CNN
+F 4 "HW-M3-8" H 6200 6600 50  0001 C CNN "PartId"
 	1    6200 6600
 	1    0    0    -1
@@
 F 2 "MountingHole:MountingHole_3.2mm_M3" H 5400 6600 50  0001 C CNN
 F 3 "~" H 5400 6600 50  0001 C CNN
+F 4 "HW-M3-8" H 5400 6600 50  0001 C CNN "PartId"
 	1    5400 6600
 	1    0    0    -1
@@
 F 2 "MountingHole:MountingHole_3.2mm_M3" H 4600 6600 50  0001 C CNN
 F 3 "~" H 4600 6600 50  0001 C CNN
+F 4 "HW-M3-8" H 4600 6600 50  0001 C CNN "PartId"
 	1    4600 6600
 	1    0    0    -1
@@
 F 2 "MountingHole:MountingHole_3.2mm_M3" H 3800 6600 50  0001 C CNN
 F 3 "~" H 3800 6600 50  0001 C CNN
+F 4 "HW-M3-8" H 3800 6600 50  0001 C CNN "PartId"
 	1    3800 6600
 	1    0    0    -1
