File: hardware/led-driver/current/led-driver-current.kicad_pcb (KiCad board)
At the start: 2 copper layers, 60 x 60 mm, 29 parts, among them J1 Input, J10 CTRL_D, J2 Output, J4 Power, J5 C Out, J6 D Out, J7 LED C, J8 LED D, J9 CTRL_C, U1 AL8861, U2 AL8861

Commit message: Rebranded.
Parts:
- D3, D4: value 3v -> 5.1v
- L1, L2: footprint Inductor_SMD:L_6.3x6.3_H3 -> footprints:L_BOURNS_SRN6045TA
Routing:
- net GND: vias 26 -> 28
Other:
- board text added: "DMX-DCC, Rev 1.0 Sparky Bobo Designs"
- board text removed: "DMX-DCC, Rev 1.0 Crazy Giraffe Software"
