File: hardware/led-driver/current/led-driver-current.sch (KiCad schematic (older format))
At the start: 27 parts, among them J1 Input, J10 CTRL_D, J2 Output, J4 Power, J5 C Out, J6 D Out, J7 LED C, J8 LED D, J9 CTRL_C, U1 AL8861, U2 AL8861

Commit message: Rebranded.
Parts:
- L1, L2: footprint Inductor_SMD:L_6.3x6.3_H3 -> footprints:L_BOURNS_SRN6045TA
Changed lines of the file:
@@
 Sheet 1 1
 Title "DMX Demonstrator - Constant Current Driver (DMX-DCC)"
-Date "2024-02-02"
+Date "2024-02-09"
 Rev "1.0"
-Comp "Crazy Giraffe Software"
+Comp "Sparky Bobo Designs"
 Comment1 ""
 Comment2 "Designed by: SparkyBobo"
@@
 F 0 "L1" V 7640 2050 50  0000 C CNN
 F 1 "33uH" V 7549 2050 50  0000 C CNN
-F 2 "Inductor_SMD:L_6.3x6.3_H3" H 7450 2050 50  0001 C CNN
+F 2 "footprints:L_BOURNS_SRN6045TA" H 7450 2050 50  0001 C CNN
 F 3 "~" H 7450 2050 50  0001 C CNN
 	1    7450 2050
@@
 F 0 "L2" V 7640 4000 50  0000 C CNN
 F 1 "33uH" V 7549 4000 50  0000 C CNN
-F 2 "Inductor_SMD:L_6.3x6.3_H3" H 7450 4000 50  0001 C CNN
+F 2 "footprints:L_BOURNS_SRN6045TA" H 7450 4000 50  0001 C CNN
 F 3 "~" H 7450 4000 50  0001 C CNN
 	1    7450 4000

Commit message: Library fixup. Rebrand.
Parts:
- U1, U2: symbol CrazyGiraffe_DMXDemonstrator:AL8861 -> DMXDemonstrator:AL8861-CrazyGiraffe_DMXDemonstrator
Changed lines of the file:
@@
 $EndComp
 $Comp
-L CrazyGiraffe_DMXDemonstrator:AL8861 U1
+L DMXDemonstrator:AL8861-CrazyGiraffe_DMXDemonstrator U1
 U 1 1 659C45BE
 P 6450 1900
@@
 	4550 3800 5800 3800
 $Comp
-L CrazyGiraffe_DMXDemonstrator:AL8861 U2
+L DMXDemonstrator:AL8861-CrazyGiraffe_DMXDemonstrator U2
 U 1 1 659EAC1C
 P 6450 3850
