File: hardware/scrambler/scrambler.kicad_pcb (KiCad board)
At the start: 2 copper layers, 68.6 x 53.3 mm, 22 parts, among them J1 Input, J2 Output, J3 Display

Commit message: Rev 1.1 of scrambler Software for scrambler
Parts:
- added R7: 330, Resistor_THT:R_Axial_DIN0207_L6.3mm_D2.5mm_P10.16mm_Horizontal, F.Cu at (133.8, 69.3)
Connections:
- A1 pad 26: Net-(A1-Pad26) -> Net-(A1-Pad25)
Routing:
- net Net-(A1-Pad25): track 0.00 -> 33.2 mm
Other:
- board text added: "DMX-FS1, Rev 1.1 Crazy Giraffe Software"
- board text removed: "DMX-FS1, Rev 1.0 Crazy Giraffe Software"

Commit message: Fixup libraries. Rebrand.
Other:
- board text added: "DMX-FS1, Rev 1.1 Sparky Bobo Designs"
- board text removed: "DMX-FS1, Rev 1.1 Crazy Giraffe Software"
