File: hardware/control-pro/dimmer-control/dimmer-control.sch (KiCad schematic (older format))
At the start: 20 parts, among them J1 OUTPUT, J2 INPUT

Commit message: Users/sparky/hwcleanup (#22)
* Rename control-pro
Update readmes
Delete old pngs

* Add PWM headers on DMX-RX1.

* Add BOM generator
Add BOM and parts .md's
Parts:
- D11, D12, D13, D14: PartId (none) -> LED_COLORLEDKIT,LED_SPACER
- D8: PartId (none) -> LED_RED
- J1: PartId (none) -> H_CPRO_RA,JP_CPRO
- J2: PartId (none) -> H_CPRO_RA
- MH1, MH2, MH3, MH4: PartId (none) -> SO-M3-18,HW-M3-8
- R1, R2, R3, R4: PartId (none) -> RV_DIM_LRG,RV_DIM_LRG_KNOB
- R11, R12, R13, R14, R8: PartId (none) -> R_LED
Changed lines of the file:
@@
 EESchema Schematic File Version 4
-LIBS:dimmer-control-cache
-EELAYER 26 0
+EELAYER 30 0
 EELAYER END
 $Descr A4 11693 8268
@@
 F 2 "footprints:BOURNS_PTA4543" H 3400 4850 50  0001 C CNN
 F 3 "~" H 3400 4850 50  0001 C CNN
+F 4 "RV_DIM_LRG,RV_DIM_LRG_KNOB" H 3400 4850 50  0001 C CNN "PartId"
 	1    3400 4850
 	1    0    0    -1
@@
 F 2 "footprints:BOURNS_PTA4543" H 3400 4100 50  0001 C CNN
 F 3 "~" H 3400 4100 50  0001 C CNN
+F 4 "RV_DIM_LRG,RV_DIM_LRG_KNOB" H 3400 4100 50  0001 C CNN "PartId"
 	1    3400 4100
 	1    0    0    -1
@@
 F 2 "footprints:BOURNS_PTA4543" H 3400 3350 50  0001 C CNN
 F 3 "~" H 3400 3350 50  0001 C CNN
+F 4 "RV_DIM_LRG,RV_DIM_LRG_KNOB" H 3400 3350 50  0001 C CNN "PartId"
 	1    3400 3350
 	1    0    0    -1
@@
 F 2 "footprints:BOURNS_PTA4543" H 3400 2600 50  0001 C CNN
 F 3 "~" H 3400 2600 50  0001 C CNN
+F 4 "RV_DIM_LRG,RV_DIM_LRG_KNOB" H 3400 2600 50  0001 C CNN "PartId"
 	1    3400 2600
 	1    0    0    -1
@@
 F 2 "MountingHole:MountingHole_3.2mm_M3" H 5500 6650 50  0001 C CNN
 F 3 "~" H 5500 6650 50  0001 C CNN
+F 4 "SO-M3-18,HW-M3-8" H 5500 6650 50  0001 C CNN "PartId"
 	1    5500 6650
 	1    0    0    -1
@@
 F 2 "MountingHole:MountingHole_3.2mm_M3" H 5500 6900 50  0001 C CNN
 F 3 "~" H 5500 6900 50  0001 C CNN
+F 4 "SO-M3-18,HW-M3-8" H 5500 6900 50  0001 C CNN "PartId"
 	1    5500 6900
 	1    0    0    -1
@@
 F 2 "MountingHole:MountingHole_3.2mm_M3" H 5500 7150 50  0001 C CNN
 F 3 "~" H 5500 7150 50  0001 C CNN
+F 4 "SO-M3-18,HW-M3-8" H 5500 7150 50  0001 C CNN "PartId"
 	1    5500 7150
 	1    0    0    -1
@@
 F 2 "MountingHole:MountingHole_3.2mm_M3" H 5500 7400 50  0001 C CNN
 F 3 "~" H 5500 7400 50  0001 C CNN
+F 4 "SO-M3-18,HW-M3-8" H 5500 7400 50  0001 C CNN "PartId"
 	1    5500 7400
 	1    0    0    -1
@@
 F 2 "Connector_IDC:IDC-Header_2x08_P2.54mm_Horizontal" H 4650 3600 50  0001 C CNN
 F 3 "~" H 4650 3600 50  0001 C CNN
+F 4 "H_CPRO_RA,JP_CPRO" H 4650 3600 50  0001 C CNN "PartId"
 	1    4650 3600
 	1    0    0    -1
@@
 F 2 "Connector_IDC:IDC-Header_2x08_P2.54mm_Horizontal" H 7050 3600 50  0001 C CNN
 F 3 "~" H 7050 3600 50  0001 C CNN
+F 4 "H_CPRO_RA" H 7050 3600 50  0001 C CNN "PartId"
 	1    7050 3600
 	-1   0    0    -1
@@
 F 2 "Resistor_THT:R_Axial_DIN0207_L6.3mm_D2.5mm_P10.16mm_Horizontal" V 5140 2590 50  0001 C CNN
 F 3 "~" H 5100 2600 50  0001 C CNN
+F 4 "R_LED" V 5100 2600 50  0001 C CNN "PartId"
 	1    5100 2600
 	0    1    1    0
@@
 F 2 "LED_THT:LED_D5.0mm" H 4650 2600 50  0001 C CNN
 F 3 "~" H 4650 2600 50  0001 C CNN
+F 4 "LED_RED" H 4650 2600 50  0001 C CNN "PartId"
 	1    4650 2600
 	-1   0    0    -1
@@
 F 2 "Resistor_THT:R_Axial_DIN0207_L6.3mm_D2.5mm_P10.16mm_Horizontal" V 8590 3940 50  0001 C CNN
 F 3 "~" H 8550 3950 50  0001 C CNN
+F 4 "R_LED" V 8550 3950 50  0001 C CNN "PartId"
 	1    8550 3950
 	0    -1   1    0
@@
 F 2 "Resistor_THT:R_Axial_DIN0207_L6.3mm_D2.5mm_P10.16mm_Horizontal" V 8590 3590 50  0001 C CNN
 F 3 "~" H 8550 3600 50  0001 C CNN
+F 4 "R_LED" V 8550 3600 50  0001 C CNN "PartId"
 	1    8550 3600
 	0    -1   1    0
@@
 F 2 "Resistor_THT:R_Axial_DIN0207_L6.3mm_D2.5mm_P10.16mm_Horizontal" V 8590 3190 50  0001 C CNN
 F 3 "~" H 8550 3200 50  0001 C CNN
+F 4 "R_LED" V 8550 3200 50  0001 C CNN "PartId"
 	1    8550 3200
 	0    -1   1    0
@@
 F 2 "Resistor_THT:R_Axial_DIN0207_L6.3mm_D2.5mm_P10.16mm_Horizontal" V 8590 2840 50  0001 C CNN
 F 3 "~" H 8550 2850 50  0001 C CNN
+F 4 "R_LED" V 8550 2850 50  0001 C CNN "PartId"
 	1    8550 2850
 	0    -1   1    0
@@
 F 2 "LED_THT:LED_D5.0mm" H 8900 2850 50  0001 C CNN
 F 3 "~" H 8900 2850 50  0001 C CNN
+F 4 "LED_COLORLEDKIT,LED_SPACER" H 8900 2850 50  0001 C CNN "PartId"
 	1    8900 2850
 	1    0    0    -1
@@
 F 2 "LED_THT:LED_D5.0mm" H 8900 3200 50  0001 C CNN
 F 3 "~" H 8900 3200 50  0001 C CNN
+F 4 "LED_COLORLEDKIT,LED_SPACER" H 8900 3200 50  0001 C CNN "PartId"
 	1    8900 3200
 	1    0    0    -1
@@
 F 2 "LED_THT:LED_D5.0mm" H 8900 3600 50  0001 C CNN
 F 3 "~" H 8900 3600 50  0001 C CNN
+F 4 "LED_COLORLEDKIT,LED_SPACER" H 8900 3600 50  0001 C CNN "PartId"
 	1    8900 3600
 	1    0    0    -1
@@
 F 2 "LED_THT:LED_D5.0mm" H 8900 3950 50  0001 C CNN
 F 3 "~" H 8900 3950 50  0001 C CNN
+F 4 "LED_COLORLEDKIT,LED_SPACER" H 8900 3950 50  0001 C CNN "PartId"
 	1    8900 3950
 	1    0    0    -1
