File: hardware/receiver-io/receiver-io.sch (KiCad schematic (older format))
At the start: 3 parts

Commit message: Prototype version of DMX, Analog, and PWM IO Modules and both TX and RX IO interfaces.
Parts:
- J1, J2: renamed from J?; value Conn_02x07_Odd_Even -> IO EXTENSION; footprint (none) -> Connector_IDC:IDC-Header_2x07_P2.54mm_Horizontal
Connections:
- net labels added: A0, A1, DMX-DIR, DMX-RX, DMX-TX, SR-CLK, SR-OUT, ~SR_CLR, ~WR
- net labels removed: RX, RXCLK, ~CLOCK, ~DATA, ~DIM0, ~DIM1, ~DIM2, ~DIM3, ~ERR, ~SC
- wire segments 9 -> 52
- no-connect marks 16 -> 20
Other:
- note removed: "D0-D4\nReserved\nFor DMX\nShield"
- moved on the sheet: J1, J2

Commit message: Display Pro: - Switch to smaller screw terminal connectors - Add pull-down resistors - Add silkscreen values - Remove COAX power connector...again - Add test software
Core:
- Fix issue with A03 and A02 being reversed at Analog Extensions
- Fix issue with A1 and A0 at IO Extension header
- Label D0..D7 correctly
- Swap U4 and U5 in schematic to match board layout
- Change TO-92 footprint
- Add silkscreen values
- Add test software

PWM:
- Switch to smaller screw terminal connectors
- Add silkscreen values
- Remove COAX power connector

Voltage:
- Switch to smaller screw terminal connectors
- Add silkscreen values
- Remove COAX power connector

DMX:
- Fix issue with DMX A and B being reversed
- Group bypass-only resistors together
- Add ISO bypass solder bridges
- Add silkscreen values
- Remove RDM bias resistors
- Add test software

Rx-IO:
- Fix issue with A1 and A0 at IO Extension header
- Add silkscreen values

Tx-IO:
- Switch to 74LS07 for Led driver
- Add pulldown resistor for discovery
- Add silkscreen values

Discovery:
- Make use of new Tx-IO pulldown resistor
Changed lines of the file:
@@
 Sheet 1 1
 Title "DMX Demonstrator - Receiver IO Module (DMX-RX2)"
-Date "2023-02-20"
-Rev "1.1"
+Date "2023-10-28"
+Rev "1.2"
 Comp "Crazy Giraffe Software"
 Comment1 ""
@@
 Text Label 7550 3200 0    50   ~ 0
 ~SR_CLR
+Text Label 6850 4550 0    50   ~ 0
+A0
 Text Label 6850 4450 0    50   ~ 0
-A0
-Text Label 6850 4550 0    50   ~ 0
 A1
 Text Label 6850 4350 0    50   ~ 0
@@
 Text Label 7550 4350 0    50   ~ 0
 SR-OUT
+Text Label 6850 3200 0    50   ~ 0
+A0
 Text Label 6850 3100 0    50   ~ 0
-A0
-Text Label 6850 3200 0    50   ~ 0
 A1
 Text Label 6850 3000 0    50   ~ 0

Commit message: Remove non io-analog files. Rebrand.
Parts:
- A1: symbol MCU_Module:Arduino_UNO_R3 -> DMXDemonstrator:Arduino_UNO_R3-MCU_Module
Changed lines of the file:
@@
 EESchema Schematic File Version 4
-LIBS:receiver-io-cache
-EELAYER 26 0
+EELAYER 30 0
 EELAYER END
 $Descr A4 11693 8268
@@
 Date "2023-10-28"
 Rev "1.2"
-Comp "Crazy Giraffe Software"
+Comp "Sparky Bobo Designs"
 Comment1 ""
 Comment2 "Designed by: SparkyBobo"
@@
 NoConn ~ 4900 2750
 $Comp
-L MCU_Module:Arduino_UNO_R3 A1
+L DMXDemonstrator:Arduino_UNO_R3-MCU_Module A1
 U 1 1 5F3035A0
 P 4800 3750

Commit message: Users/sparky/hwcleanup (#22)
* Rename control-pro
Update readmes
Delete old pngs

* Add PWM headers on DMX-RX1.

* Add BOM generator
Add BOM and parts .md's
Parts:
- A1: PartId (none) -> H_ARDUINO
- J1, J2: PartId (none) -> H_IO_RA
Changed lines of the file:
@@
 F 2 "footprints:ARDUINO_R3_NO_HOLES" H 4950 2700 50  0001 L CNN
 F 3 "https://www.arduino.cc/en/Main/arduinoBoardUno" H 4600 4800 50  0001 C CNN
+F 4 "H_ARDUINO" H 4800 3750 50  0001 C CNN "PartId"
 	1    4800 3750
 	-1   0    0    -1
@@
 F 2 "Connector_IDC:IDC-Header_2x07_P2.54mm_Horizontal" H 7200 3200 50  0001 C CNN
 F 3 "~" H 7200 3200 50  0001 C CNN
+F 4 "H_IO_RA" H 7200 3200 50  0001 C CNN "PartId"
 	1    7200 3200
 	1    0    0    -1
@@
 F 2 "Connector_IDC:IDC-Header_2x07_P2.54mm_Horizontal" H 7200 4550 50  0001 C CNN
 F 3 "~" H 7200 4550 50  0001 C CNN
+F 4 "H_IO_RA" H 7200 4550 50  0001 C CNN "PartId"
 	1    7200 4550
 	1    0    0    -1
