File: hardware/transmitter/transmitter.sch (KiCad schematic (older format))
At the start: 23 parts, among them J1 Output

Commit message: Rev 1.1: - Fixed arduino shield footprint (it was backwards) - Added Fcu power plane - New Fcu layouts - Added rounded corners
Parts:
- A1: footprint Module:Arduino_UNO_R3 -> footprints:ARDUINO_R3_NO_HOLES
Changed lines of the file:
@@
 Sheet 1 1
 Title "DMX Demonstrator - Transmitter (DMX-TX1)"
-Date "2020-09-25"
-Rev "1.0"
+Date "2020-11-07"
+Rev "1.1"
 Comp "Crazy Giraffe Software"
 Comment1 ""
@@
 F 0 "A1" H 6000 4400 50  0000 C CNN
 F 1 "Arduino_UNO_R3" H 5750 4300 50  0000 C CNN
-F 2 "Module:Arduino_UNO_R3" H 6350 2300 50  0001 L CNN
+F 2 "footprints:ARDUINO_R3_NO_HOLES" H 6350 2300 50  0001 L CNN
 F 3 "https://www.arduino.cc/en/Main/arduinoBoardUno" H 6000 4400 50  0001 C CNN
 	1    6200 3350
@@
 F 4 "RES-09177" H 4782 4816 60  0001 R CNN "Field4"
 	1    4850 4900
-	1    0    0    -1
+	1    0    0    1
 $EndComp
 $Comp
@@
 F 4 "RES-11924" H 4832 2216 60  0001 R CNN "Field4"
 	1    4900 2300
-	1    0    0    -1
-$EndComp
-$Comp
+	1    0    0    1
+$EndComp
+$Comp

Commit message: Users/sparky/txrx12 (#11)
* TX1 1.2, RX1 1.2
Move Clock LED to avoid ICSP connector.
Align TX Fast/Slo clock LEDS and RX start code/error LEDs.

* Add RXCLK to D9 connection for Leonardo PCINT5.

Co-authored-by: SparkyBobo <sparky@crazygiraffesoftware.com>
Parts:
- D7: value CLK_SLO -> CLK_FST
- D8: value CLK_FST -> CLK_SLO
Changed lines of the file:
@@
 Sheet 1 1
 Title "DMX Demonstrator - Transmitter (DMX-TX1)"
-Date "2020-11-07"
-Rev "1.1"
+Date "2020-12-28"
+Rev "1.2"
 Comp "Crazy Giraffe Software"
 Comment1 ""
@@
 P 7700 4600
 F 0 "D8" H 7691 4816 50  0000 C CNN
-F 1 "CLK_FST" H 7691 4725 50  0000 C CNN
+F 1 "CLK_SLO" H 7691 4725 50  0000 C CNN
 F 2 "LED_THT:LED_D5.0mm" H 7700 4600 50  0001 C CNN
 F 3 "~" H 7700 4600 50  0001 C CNN
@@
 P 7700 4250
 F 0 "D7" H 7691 4466 50  0000 C CNN
-F 1 "CLK_SLO" H 7691 4375 50  0000 C CNN
+F 1 "CLK_FST" H 7691 4375 50  0000 C CNN
 F 2 "LED_THT:LED_D5.0mm" H 7700 4250 50  0001 C CNN
 F 3 "~" H 7700 4250 50  0001 C CNN
@@
 Clock Step
 Text Notes 8350 4600 0    50   ~ 0
+Clock Slow
+Text Notes 8350 4250 0    50   ~ 0
 Clock Fast
-Text Notes 8350 4250 0    50   ~ 0
-Clock Slow
 Wire Wire Line
 	5300 3350 5300 2300
@@
 ~CLOCK
 Text Label 6750 3550 0    50   ~ 0
+~CLK_FST
+Text Label 6750 3650 0    50   ~ 0
 ~CLK_SLO
-Text Label 6750 3650 0    50   ~ 0
-~CLK_FST
 Wire Wire Line
 	8050 4900 6900 4900

Commit message: Rebrand to Sparky Bobo Designs
Parts:
- A1: symbol MCU_Module:Arduino_UNO_R3 -> DMXDemonstrator:Arduino_UNO_R3-MCU_Module
- S1, S2, S3: symbol SparkFun-Switches:MOMENTARY-SWITCH-SPST-PTH-12MM -> DMXDemonstrator:MOMENTARY-SWITCH-SPST-PTH-12MM-SparkFun-Switches
- VR1: symbol SparkFun-Resistors:POTENTIOMETER_SLIDE-20MM-1_10W-20% -> DMXDemonstrator:POTENTIOMETER_SLIDE-20MM-1_10W-20%-SparkFun-Resistors
- VR2: symbol SparkFun-Resistors:POTENTIOMETER-PTH-9MM-1_20W-20% -> DMXDemonstrator:POTENTIOMETER-PTH-9MM-1_20W-20%-SparkFun-Resistors
Changed lines of the file:
@@
 EESchema Schematic File Version 4
-LIBS:transmitter-cache
-EELAYER 26 0
+EELAYER 30 0
 EELAYER END
 $Descr A4 11693 8268
@@
 Date "2023-12-04"
 Rev "1.3"
-Comp "Crazy Giraffe Software"
+Comp "Sparky Bobo Designs"
 Comment1 ""
 Comment2 "Designed by: SparkyBobo"
@@
 $EndDescr
 $Comp
-L MCU_Module:Arduino_UNO_R3 A1
+L DMXDemonstrator:Arduino_UNO_R3-MCU_Module A1
 U 1 1 5F3035A0
 P 6200 3350
@@
 Connection ~ 4250 3850
 $Comp
-L SparkFun-Resistors:POTENTIOMETER-PTH-9MM-1_20W-20% VR2
+L DMXDemonstrator:POTENTIOMETER-PTH-9MM-1_20W-20%-SparkFun-Resistors VR2
 U 1 1 5F517499
 P 4850 4900
@@
 $EndComp
 $Comp
-L SparkFun-Resistors:POTENTIOMETER_SLIDE-20MM-1_10W-20% VR1
+L DMXDemonstrator:POTENTIOMETER_SLIDE-20MM-1_10W-20%-SparkFun-Resistors VR1
 U 1 1 5F51752E
 P 4900 2300
@@
 $EndComp
 $Comp
-L SparkFun-Switches:MOMENTARY-SWITCH-SPST-PTH-12MM S1
+L DMXDemonstrator:MOMENTARY-SWITCH-SPST-PTH-12MM-SparkFun-Switches S1
 U 1 1 5F53A7F8
 P 4550 3050
@@
 $EndComp
 $Comp
-L SparkFun-Switches:MOMENTARY-SWITCH-SPST-PTH-12MM S2
+L DMXDemonstrator:MOMENTARY-SWITCH-SPST-PTH-12MM-SparkFun-Switches S2
 U 1 1 5F53A858
 P 4550 3550
@@
 $EndComp
 $Comp
-L SparkFun-Switches:MOMENTARY-SWITCH-SPST-PTH-12MM S3
+L DMXDemonstrator:MOMENTARY-SWITCH-SPST-PTH-12MM-SparkFun-Switches S3
 U 1 1 5F53A8A0
 P 4550 3850

Commit message: Users/sparky/hwcleanup (#22)
* Rename control-pro
Update readmes
Delete old pngs

* Add PWM headers on DMX-RX1.

* Add BOM generator
Add BOM and parts .md's
Parts:
- A1: PartId (none) -> A_ARDUINO,H_ARDUINO
- D1, D8: PartId (none) -> LED_GRN
- D2, D7: PartId (none) -> LED_RED
- D3, D4, D5, D6: PartId (none) -> LED_COLORLEDKIT
- J1: PartId (none) -> H_1x3_RA
- R1, R2, R3, R4, R5, R6, R7, R8: PartId (none) -> R_LED
- S1, S2, S3: Field4 SWCH-09185 -> (none); PartId (none) -> S_MOM
- VR1: Field4 RES-11924 -> (none); PartId (none) -> RV_DIM_SM,RV_DIM_SM_KNOB
- VR2: Field4 RES-09177 -> (none); PartId (none) -> RV_CLK
Changed lines of the file:
@@
 F 1 "Arduino_UNO_R3" H 5750 4300 50  0000 C CNN
 F 2 "footprints:ARDUINO_R3_NO_HOLES" H 6350 2300 50  0001 L CNN
-F 3 "https://www.arduino.cc/en/Main/arduinoBoardUno" H 6000 4400 50  0001 C CNN
+F 3 "" H 6000 4400 50  0001 C CNN
+F 4 "A_ARDUINO,H_ARDUINO" H 6200 3350 50  0001 C CNN "PartId"
 	1    6200 3350
 	-1   0    0    -1
@@
 F 2 "Connector_PinHeader_2.54mm:PinHeader_1x03_P2.54mm_Horizontal" H 8250 5000 50  0001 C CNN
 F 3 "~" H 8250 5000 50  0001 C CNN
+F 4 "H_1x3_RA" H 8250 5000 50  0001 C CNN "PartId"
 	1    8250 5000
 	1    0    0    -1
@@
 F 2 "LED_THT:LED_D5.0mm" H 7700 2050 50  0001 C CNN
 F 3 "~" H 7700 2050 50  0001 C CNN
+F 4 "LED_GRN" H 7700 2050 50  0001 C CNN "PartId"
 	1    7700 2050
 	1    0    0    -1
@@
 F 2 "Resistor_THT:R_Axial_DIN0207_L6.3mm_D2.5mm_P10.16mm_Horizontal" V 8090 2040 50  0001 C CNN
 F 3 "~" H 8050 2050 50  0001 C CNN
+F 4 "R_LED" V 8050 2050 50  0001 C CNN "PartId"
 	1    8050 2050
 	0    1    1    0
@@
 F 2 "LED_THT:LED_D5.0mm" H 7700 2400 50  0001 C CNN
 F 3 "~" H 7700 2400 50  0001 C CNN
+F 4 "LED_RED" H 7700 2400 50  0001 C CNN "PartId"
 	1    7700 2400
 	1    0    0    -1
@@
 F 2 "Resistor_THT:R_Axial_DIN0207_L6.3mm_D2.5mm_P10.16mm_Horizontal" V 8090 2390 50  0001 C CNN
 F 3 "~" H 8050 2400 50  0001 C CNN
+F 4 "R_LED" V 8050 2400 50  0001 C CNN "PartId"
 	1    8050 2400
 	0    1    1    0
@@
 F 2 "LED_THT:LED_D5.0mm" H 7700 4600 50  0001 C CNN
 F 3 "~" H 7700 4600 50  0001 C CNN
+F 4 "LED_GRN" H 7700 4600 50  0001 C CNN "PartId"
 	1    7700 4600
 	1    0    0    -1
@@
 F 2 "Resistor_THT:R_Axial_DIN0207_L6.3mm_D2.5mm_P10.16mm_Horizontal" V 8090 4590 50  0001 C CNN
 F 3 "~" H 8050 4600 50  0001 C CNN
+F 4 "R_LED" V 8050 4600 50  0001 C CNN "PartId"
 	1    8050 4600
 	0    1    1    0
@@
 F 2 "LED_THT:LED_D5.0mm" H 7700 4250 50  0001 C CNN
 F 3 "~" H 7700 4250 50  0001 C CNN
+F 4 "LED_RED" H 7700 4250 50  0001 C CNN "PartId"
 	1    7700 4250
 	1    0    0    -1
@@
 F 2 "Resistor_THT:R_Axial_DIN0207_L6.3mm_D2.5mm_P10.16mm_Horizontal" V 8090 4240 50  0001 C CNN
 F 3 "~" H 8050 4250 50  0001 C CNN
+F 4 "R_LED" V 8050 4250 50  0001 C CNN "PartId"
 	1    8050 4250
 	0    1    1    0
@@
 F 2 "LED_THT:LED_D5.0mm" H 7700 3850 50  0001 C CNN
 F 3 "~" H 7700 3850 50  0001 C CNN
+F 4 "LED_COLORLEDKIT" H 7700 3850 50  0001 C CNN "PartId"
 	1    7700 3850
 	1    0    0    -1
@@
 F 2 "Resistor_THT:R_Axial_DIN0207_L6.3mm_D2.5mm_P10.16mm_Horizontal" V 8090 3840 50  0001 C CNN
 F 3 "~" H 8050 3850 50  0001 C CNN
+F 4 "R_LED" V 8050 3850 50  0001 C CNN "PartId"
 	1    8050 3850
 	0    1    1    0
@@
 F 2 "LED_THT:LED_D5.0mm" H 7700 3500 50  0001 C CNN
 F 3 "~" H 7700 3500 50  0001 C CNN
+F 4 "LED_COLORLEDKIT" H 7700 3500 50  0001 C CNN "PartId"
 	1    7700 3500
 	1    0    0    -1
@@
 F 2 "Resistor_THT:R_Axial_DIN0207_L6.3mm_D2.5mm_P10.16mm_Horizontal" V 8090 3490 50  0001 C CNN
 F 3 "~" H 8050 3500 50  0001 C CNN
+F 4 "R_LED" V 8050 3500 50  0001 C CNN "PartId"
 	1    8050 3500
 	0    1    1    0
@@
 F 2 "LED_THT:LED_D5.0mm" H 7700 3100 50  0001 C CNN
 F 3 "~" H 7700 3100 50  0001 C CNN
+F 4 "LED_COLORLEDKIT" H 7700 3100 50  0001 C CNN "PartId"
 	1    7700 3100
 	1    0    0    -1
@@
 F 2 "Resistor_THT:R_Axial_DIN0207_L6.3mm_D2.5mm_P10.16mm_Horizontal" V 8090 3090 50  0001 C CNN
 F 3 "~" H 8050 3100 50  0001 C CNN
+F 4 "R_LED" V 8050 3100 50  0001 C CNN "PartId"
 	1    8050 3100
 	0    1    1    0
@@
 F 2 "LED_THT:LED_D5.0mm" H 7700 2750 50  0001 C CNN
 F 3 "~" H 7700 2750 50  0001 C CNN
+F 4 "LED_COLORLEDKIT" H 7700 2750 50  0001 C CNN "PartId"
 	1    7700 2750
 	1    0    0    -1
@@
 F 2 "Resistor_THT:R_Axial_DIN0207_L6.3mm_D2.5mm_P10.16mm_Horizontal" V 8090 2740 50  0001 C CNN
 F 3 "~" H 8050 2750 50  0001 C CNN
+F 4 "R_LED" V 8050 2750 50  0001 C CNN "PartId"
 	1    8050 2750
 	0    1    1    0
@@
 F 2 "Resistors:POT-PTH-ALPS" V 4700 4900 20  0001 C CNN
 F 3 "" H 4850 4900 60  0001 C CNN
-F 4 "RES-09177" H 4782 4816 60  0001 R CNN "Field4"
+F 4 "RV_CLK" H 4782 4816 60  0001 R CNN "PartId"
 	1    4850 4900
 	1    0    0    1
@@
 F 2 "Resistors:SLIDER-SMALL" V 4750 2300 20  0001 C CNN
 F 3 "" H 4900 2300 60  0001 C CNN
-F 4 "RES-11924" H 4832 2216 60  0001 R CNN "Field4"
+F 4 "RV_DIM_SM,RV_DIM_SM_KNOB" H 4832 2216 60  0001 R CNN "PartId"
 	1    4900 2300
 	1    0    0    1
@@
 F 2 "Switches:TACTILE_SWITCH_PTH_12MM" H 4550 3250 20  0001 C CNN
 F 3 "" H 4550 3050 50  0001 C CNN
-F 4 "SWCH-09185" H 4550 3181 60  0001 C CNN "Field4"
+F 4 "S_MOM" H 4550 3181 60  0001 C CNN "PartId"
 	1    4550 3050
 	1    0    0    -1
@@
 F 2 "Switches:TACTILE_SWITCH_PTH_12MM" H 4550 3750 20  0001 C CNN
 F 3 "" H 4550 3550 50  0001 C CNN
-F 4 "SWCH-09185" H 4550 3681 60  0001 C CNN "Field4"
+F 4 "S_MOM" H 4550 3681 60  0001 C CNN "PartId"
 	1    4550 3550
 	1    0    0    -1
@@
 F 2 "Switches:TACTILE_SWITCH_PTH_12MM" H 4550 4050 20  0001 C CNN
 F 3 "" H 4550 3850 50  0001 C CNN
-F 4 "SWCH-09185" H 4550 3981 60  0001 C CNN "Field4"
+F 4 "S_MOM" H 4550 3981 60  0001 C CNN "PartId"
 	1    4550 3850
 	1    0    0    -1
