File: hardware/io-analog/core/io-analog-core.sch (KiCad schematic (older format))
At the start: 24 parts, among them J1 IO Extension, J3 Analog Extension, U1 74LS164, U2 74LS139, U3 TLC7524CN, U4 TLC7524CN, U5 TLC7524CN, U6 TLC7524CN, U7 TLV2772, U8 TLV2772

Commit message: Finalize io-analog boards.
Connections:
- wire segments 197 -> 200
Changed lines of the file:
@@
 Wire Wire Line
 	1500 7450 1950 7450
+Text Notes 10500 3700 0    50   ~ 0
+Analog Output\n0v-2.5v
+$Comp
+L power:PWR_FLAG #FLG?
+U 1 1 64BE351C
+P 4200 7500
+AR Path="/647E1209/64BE351C" Ref="#FLG?"  Part="1"
+AR Path="/64BE351C" Ref="#FLG0101"  Part="1"
+F 0 "#FLG0101" H 4200 7575 50  0001 C CNN
+F 1 "PWR_FLAG" H 4200 7673 50  0000 C CNN
+F 2 "" H 4200 7500 50  0001 C CNN
+F 3 "~" H 4200 7500 50  0001 C CNN
+	1    4200 7500
+	-1   0    0    1
+$EndComp
+Wire Wire Line
+	4200 7500 4200 7450
+$Comp
+L power:PWR_FLAG #FLG?
+U 1 1 64BF9D93
+P 5950 6500
+AR Path="/647E1209/64BF9D93" Ref="#FLG?"  Part="1"
+AR Path="/64BF9D93" Ref="#FLG0103"  Part="1"
+F 0 "#FLG0103" H 5950 6575 50  0001 C CNN
+F 1 "PWR_FLAG" H 5950 6673 50  0000 C CNN
+F 2 "" H 5950 6500 50  0001 C CNN
+F 3 "~" H 5950 6500 50  0001 C CNN
+	1    5950 6500
+	1    0    0    -1
+$EndComp
+Wire Wire Line
+	5950 6550 5950 6500
+Wire Wire Line
+	5600 6550 5950 6550
 Wire Bus Line
-	2750 4200 2750 4750
+	7200 1300 7200 4600
 Wire Bus Line
-	4600 1200 7100 1200
+	5200 1300 5200 4600
 Wire Bus Line
-	4800 1400 6900 1400
-Wire Bus Line
-	2250 3000 2250 4750
-Wire Bus Line
-	2350 4850 4600 4850
+	4500 1300 4500 3200
 Wire Bus Line
 	4350 4200 4350 4750
@@
 	5000 1500 5000 4850
 Wire Bus Line
-	4500 1300 4500 3200
+	2350 4850 4600 4850
 Wire Bus Line
-	5200 1300 5200 4600
+	2250 3000 2250 4750
 Wire Bus Line
-	7200 1300 7200 4600
-Text Notes 10500 3700 0    50   ~ 0
-Analog Output\n0v-2.5v
+	2750 4200 2750 4750
+Wire Bus Line
+	4600 1200 7100 1200
+Wire Bus Line
+	4800 1400 6900 1400
 $EndSCHEMATC

Commit message: Added Bill Of Materials (BOM)
Parts:
- C1, C2, C3, C4, C5, C6, C8: AF_Detail_Page (none) -> https://www.adafruit.com/product/753; AF_PN (none) -> 753; Description (none) -> Decoupling Capacitor; MO_Detail_Page (none) -> https://www.mouser.com/ProductDetail/KEMET/C320C104K5R5TA73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; MO_PN (none) -> 80-C320C104K5R7301; NW_Detail_Page (none) -> https://www.newark.com/kemet/c315c104m5u5ta/capacitor-mlcc-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; NW_PN (none) -> 13K6284; SP_Detail_Page (none) -> https://www.sparkfun.com/products/8375; SP_PN (none) -> COM-08375
- C7: AF_Detail_Page (none) -> https://www.adafruit.com/product/2195; AF_PN (none) -> 2195; DK_Detail_Page (none) -> en/products/detail/panasonic-electronic-components/ECA-1HM1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; Description (none) -> Filter Capacitor; Digi-Key_PN (none) -> P10425CT-ND; MO_Detail_Page (none) -> https://www.mouser.com/ProductDetail/Panasonic/ECA-1HM100I; MO_PN (none) -> 667-ECA-1HM100I; NW_PN (none) -> ECA-1HM100I; NW_Page_Detail (none) -> https://www.newark.com/panasonic/eca-1hm100i/aluminum-elect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; SP_Detail_Page (none) -> https://www.sparkfun.com/products/523; SP_PN (none) -> COM-00523
- J1: DK_Detail_Page (none) -> en/products/detail/würth-elektronik/61201421721/4846921?s=N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; Digi-Key_PN (none) -> 732-5407-ND; MO_Detail_Page (none) -> https://www.mouser.com/ProductDetail/Wurth-Elektronik/61201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; MO_PN (none) -> 710-61201421721; NW_Detail_Page (none) -> https://www.newark.com/wurth-elektronik/612014235221/conn-r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; NW_PN (none) -> 75AJ1395
- J3: Description (none) -> Header - 8 Pin; MO_Detail_Page (none) -> https://www.mouser.com/ProductDetail/Gravitech/8Fx1-254mm?q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; MO_PN (none) -> 992-8FX1-254MM; SP_Detail_Page (none) -> https://www.sparkfun.com/products/11895; SP_PN (none) -> PRT-11895
- R9: DK_Detail_Page (none) -> en/products/detail/yageo/CFR-25JB-52-1K6/141; Digi-Key_PN (none) -> 1.6KQBK-ND; MO_Detail_Page (none) -> https://www.mouser.com/ProductDetail/YAGEO/CFR-25JB-52-1K6?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; MO_PN (none) -> 603-CFR-25JB-52-1K6; NW_Detail_Page (none) -> https://www.newark.com/multicomp-pro/mcmf0w4ff1601a50/metal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; NW_PN (none) -> 59K8662
- U1: DK_Detail_Page (none) -> en/products/detail/texas-instruments/SN74LS164N/277293; Description (none) -> 8-Bit Parallel-Out Serial Shift Register; Digi-Key_PN (none) -> 296-1647-5-ND; MO_Detail_Page (none) -> https://www.mouser.com/ProductDetail/Texas-Instruments/SN74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; MO_PN (none) -> 595-SN74LS164N
- U2: DK_Detail_Page (none) -> en/products/detail/texas-instruments/SN74LS139AN/277286; Description (none) -> Dual 2-line to 4-line decoders; Digi-Key_PN (none) -> 296-1640-5-ND; MO_Detail_Page (none) -> https://www.mouser.com/ProductDetail/Texas-Instruments/SN74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; MO_PN (none) -> 595-SN74LS139AN
- U3, U4, U5, U6: DK_Detail_Page (none) -> en/products/detail/texas-instruments/TLC7524CN/277513; Description (none) -> 8-bit Multiplying Digital to Analog Converter; Digi-Key_PN (none) -> 296-1868-5-ND; MO_Detail_Page (none) -> https://www.mouser.com/ProductDetail/Texas-Instruments/TLC7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; MO_PN (none) -> 595-TLC7524CN
- U7, U8: DK_Detail_Page (none) -> en/products/detail/texas-instruments/TLV2772CP/374329; Description (none) -> Rail-to-Rail Operational Amplifier; Digi-Key_PN (none) -> 296-7592-5-ND; MO_Detail_Page (none) -> https://www.mouser.com/ProductDetail/Texas-Instruments/TLV2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; MO_PN (none) -> TLV2772CP
- VR1: footprint Package_TO_SOT_THT:TO-92L_HandSolder -> TO-92-3_Formed_Leads; DK_Detail_Page (none) -> products/detail/texas-instruments/TL1431CLP/380747; Description (none) -> Precision Voltage Reference; Digi-Key_PN (none) -> 296-10130-5-ND; MO_Detail_Page (none) -> https://www.mouser.com/ProductDetail/Texas-Instruments/TL14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; MO_PN (none) -> 595-TL1431CLPR

Commit message: Display Pro: - Switch to smaller screw terminal connectors - Add pull-down resistors - Add silkscreen values - Remove COAX power connector...again - Add test software
Core:
- Fix issue with A03 and A02 being reversed at Analog Extensions
- Fix issue with A1 and A0 at IO Extension header
- Label D0..D7 correctly
- Swap U4 and U5 in schematic to match board layout
- Change TO-92 footprint
- Add silkscreen values
- Add test software

PWM:
- Switch to smaller screw terminal connectors
- Add silkscreen values
- Remove COAX power connector

Voltage:
- Switch to smaller screw terminal connectors
- Add silkscreen values
- Remove COAX power connector

DMX:
- Fix issue with DMX A and B being reversed
- Group bypass-only resistors together
- Add ISO bypass solder bridges
- Add silkscreen values
- Remove RDM bias resistors
- Add test software

Rx-IO:
- Fix issue with A1 and A0 at IO Extension header
- Add silkscreen values

Tx-IO:
- Switch to 74LS07 for Led driver
- Add pulldown resistor for discovery
- Add silkscreen values

Discovery:
- Make use of new Tx-IO pulldown resistor
Parts:
- VR1: footprint TO-92-3_Formed_Leads -> Package_TO_SOT_THT:TO-92_Inline_Wide
- renumbered U5 to U4, U4 to U5

Commit message: Remove non io-analog files. Rebrand.
Parts:
- U1: symbol CrazyGiraffe_DMXDemonstrator:74LS164 -> DMXDemonstrator:74LS164
- U3, U4, U5, U6: symbol CrazyGiraffe_DMXDemonstrator:TLC7524CN -> DMXDemonstrator:TLC7524CN
- U7, U8: symbol CrazyGiraffe_DMXDemonstrator:TLV2772CP -> DMXDemonstrator:TLV2772CP
- VR1: symbol CrazyGiraffe_DMXDemonstrator:TL1431 -> DMXDemonstrator:TL1431
Changed lines of the file:
@@
 EESchema Schematic File Version 4
-LIBS:io-analog-core-cache
-EELAYER 26 0
+EELAYER 30 0
 EELAYER END
 $Descr A4 11693 8268
@@
 Date "2023-09-17"
 Rev "1.3"
-Comp "Crazy Giraffe Software"
+Comp "Sparky Bobo Designs"
 Comment1 ""
 Comment2 "Designed by: SparkyBobo"
@@
 	4200 6850 4200 6550
 $Comp
-L CrazyGiraffe_DMXDemonstrator:74LS164 U?
+L DMXDemonstrator:74LS164 U?
 U 1 1 647F5755
 P 3900 3000
@@
 	5600 7050 5400 7050
 $Comp
-L CrazyGiraffe_DMXDemonstrator:TL1431 VR?
+L DMXDemonstrator:TL1431 VR?
 U 1 1 647F5A12
 P 5200 7050
@@
 	4200 7450 4650 7450
 $Comp
-L CrazyGiraffe_DMXDemonstrator:TLC7524CN U3
+L DMXDemonstrator:TLC7524CN U3
 U 1 1 648A85B8
 P 5850 2400
@@
 $EndComp
 $Comp
-L CrazyGiraffe_DMXDemonstrator:TLC7524CN U5
+L DMXDemonstrator:TLC7524CN U5
 U 1 1 6495FADC
 P 5850 4400
@@
 $EndComp
 $Comp
-L CrazyGiraffe_DMXDemonstrator:TLC7524CN U4
+L DMXDemonstrator:TLC7524CN U4
 U 1 1 64968030
 P 7850 2400
@@
 $EndComp
 $Comp
-L CrazyGiraffe_DMXDemonstrator:TLC7524CN U6
+L DMXDemonstrator:TLC7524CN U6
 U 1 1 64968095
 P 7850 4400
@@
 AO0
 $Comp
-L CrazyGiraffe_DMXDemonstrator:TLV2772CP U7
+L DMXDemonstrator:TLV2772CP U7
 U 1 1 6511AB4A
 P 9350 2400
@@
 $EndComp
 $Comp
-L CrazyGiraffe_DMXDemonstrator:TLV2772CP U7
+L DMXDemonstrator:TLV2772CP U7
 U 2 1 6511ABB9
 P 9350 4500
@@
 $EndComp
 $Comp
-L CrazyGiraffe_DMXDemonstrator:TLV2772CP U8
+L DMXDemonstrator:TLV2772CP U8
 U 3 1 6511AC32
 P 1400 7000
@@
 $EndComp
 $Comp
-L CrazyGiraffe_DMXDemonstrator:TLV2772CP U8
+L DMXDemonstrator:TLV2772CP U8
 U 1 1 6511AD0D
 P 9350 3800
@@
 $EndComp
 $Comp
-L CrazyGiraffe_DMXDemonstrator:TLV2772CP U8
+L DMXDemonstrator:TLV2772CP U8
 U 2 1 6511AD82
 P 9350 3100
@@
 $EndComp
 $Comp
-L CrazyGiraffe_DMXDemonstrator:TLV2772CP U7
+L DMXDemonstrator:TLV2772CP U7
 U 3 1 6511ADEF
 P 1150 7000
@@
 Wire Wire Line
 	9850 3100 9700 3100
+Connection ~ 9700 3100
 Wire Bus Line
 	2750 4200 2750 4750
@@
 Wire Bus Line
 	7200 1300 7200 4600
-Connection ~ 9700 3100
 $EndSCHEMATC

Commit message: Add parts and BOMs for rest of boards. Cleanup .md files.
Parts:
- C1, C2, C3, C4, C5, C6: AF_Detail_Page https://www.adafruit.com/product/753 -> (none); AF_PN 753 -> (none); Description Decoupling Capacitor -> (none); MO_Detail_Page https://www.mouser.com/ProductDetail/KEMET/C320C104K5R5TA73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 -> (none); MO_PN 80-C320C104K5R7301 -> (none); NW_Detail_Page https://www.newark.com/kemet/c315c104m5u5ta/capacitor-mlcc-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 -> (none); NW_PN 13K6284 -> (none); PartId (none) -> C_DECOUPLE; SP_Detail_Page https://www.sparkfun.com/products/8375 -> (none); SP_PN COM-08375 -> (none)
- C7: AF_Detail_Page https://www.adafruit.com/product/2195 -> (none); AF_PN 2195 -> (none); DK_Detail_Page en/products/detail/panasonic-electronic-components/ECA-1HM1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 -> (none); Digi-Key_PN P10425CT-ND -> (none); MO_Detail_Page https://www.mouser.com/ProductDetail/Panasonic/ECA-1HM100I -> (none); MO_PN 667-ECA-1HM100I -> (none); NW_PN ECA-1HM100I -> (none); NW_Page_Detail https://www.newark.com/panasonic/eca-1hm100i/aluminum-elect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 -> (none); PartId (none) -> C_FILTER; SP_Detail_Page https://www.sparkfun.com/products/523 -> (none); SP_PN COM-00523 -> (none)
- C8: AF_Detail_Page https://www.adafruit.com/product/753 -> (none); AF_PN 753 -> (none); MO_Detail_Page https://www.mouser.com/ProductDetail/KEMET/C320C104K5R5TA73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 -> (none); MO_PN 80-C320C104K5R7301 -> (none); NW_Detail_Page https://www.newark.com/kemet/c315c104m5u5ta/capacitor-mlcc-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 -> (none); NW_PN 13K6284 -> (none); PartId (none) -> C_DECOUPLE; SP_Detail_Page https://www.sparkfun.com/products/8375 -> (none); SP_PN COM-08375 -> (none)
- J1: DK_Detail_Page en/products/detail/würth-elektronik/61201421721/4846921?s=N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 -> (none); Digi-Key_PN 732-5407-ND -> (none); MO_Detail_Page https://www.mouser.com/ProductDetail/Wurth-Elektronik/61201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 -> (none); MO_PN 710-61201421721 -> (none); NW_Detail_Page https://www.newark.com/wurth-elektronik/612014235221/conn-r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 -> (none); NW_PN 75AJ1395 -> (none); PartId (none) -> H_IO_RA,JP_IO
- J3: MO_Detail_Page https://www.mouser.com/ProductDetail/Gravitech/8Fx1-254mm?q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 -> (none); MO_PN 992-8FX1-254MM -> (none); PartId (none) -> H_ANALOG_SHORT; SP_Detail_Page https://www.sparkfun.com/products/11895 -> (none); SP_PN PRT-11895 -> (none)
- R9: DK_Detail_Page en/products/detail/yageo/CFR-25JB-52-1K6/141 -> (none); Digi-Key_PN 1.6KQBK-ND -> (none); MO_Detail_Page https://www.mouser.com/ProductDetail/YAGEO/CFR-25JB-52-1K6?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 -> (none); MO_PN 603-CFR-25JB-52-1K6 -> (none); NW_Detail_Page https://www.newark.com/multicomp-pro/mcmf0w4ff1601a50/metal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 -> (none); NW_PN 59K8662 -> (none); PartId (none) -> R_1k6
- U1: DK_Detail_Page en/products/detail/texas-instruments/SN74LS164N/277293 -> (none); Digi-Key_PN 296-1647-5-ND -> (none); MO_Detail_Page https://www.mouser.com/ProductDetail/Texas-Instruments/SN74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 -> (none); MO_PN 595-SN74LS164N -> (none); PartId (none) -> U_74LS164
- U2: DK_Detail_Page en/products/detail/texas-instruments/SN74LS139AN/277286 -> (none); Digi-Key_PN 296-1640-5-ND -> (none); MO_Detail_Page https://www.mouser.com/ProductDetail/Texas-Instruments/SN74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 -> (none); MO_PN 595-SN74LS139AN -> (none); PartId (none) -> U_74LS139
- U3, U4, U5, U6: DK_Detail_Page en/products/detail/texas-instruments/TLC7524CN/277513 -> (none); Digi-Key_PN 296-1868-5-ND -> (none); MO_Detail_Page https://www.mouser.com/ProductDetail/Texas-Instruments/TLC7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 -> (none); MO_PN 595-TLC7524CN -> (none); PartId (none) -> U_TLC7524CN
- U7, U8: DK_Detail_Page en/products/detail/texas-instruments/TLV2772CP/374329 -> (none); Description Rail-to-Rail Operational Amplifier -> (none); Digi-Key_PN 296-7592-5-ND -> (none); MO_Detail_Page https://www.mouser.com/ProductDetail/Texas-Instruments/TLV2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 -> (none); MO_PN TLV2772CP -> (none); PartId (none) -> U_TLV2772
- VR1: DK_Detail_Page products/detail/texas-instruments/TL1431CLP/380747 -> (none); Digi-Key_PN 296-10130-5-ND -> (none); MO_Detail_Page https://www.mouser.com/ProductDetail/Texas-Instruments/TL14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 -> (none); MO_PN 595-TL1431CLPR -> (none); PartId (none) -> U_TL1431
