File: hardware/transmitter-io/transmitter-io.sch (KiCad schematic (older format))
At the start: 23 parts, among them J1 Output

Commit message: Move TX2 to tx-io
Parts:
- removed D3: DIM3, LED_THT:LED_D5.0mm, symbol Device:LED
- removed D4: DIM2, LED_THT:LED_D5.0mm, symbol Device:LED
- removed D5: DIM1, LED_THT:LED_D5.0mm, symbol Device:LED
- removed D6: DIM0, LED_THT:LED_D5.0mm, symbol Device:LED
- removed D7: CLK_FST, LED_THT:LED_D5.0mm, symbol Device:LED
- removed D8: CLK_SLO, LED_THT:LED_D5.0mm, symbol Device:LED
- removed R4, R5, R6, R7, R8: 330, Resistor_THT:R_Axial_DIN0207_L6.3mm_D2.5mm_P10.16mm_Horizontal, symbol Device:R_US
- removed S1: DIM_SELECT, Switches:TACTILE_SWITCH_PTH_12MM, symbol SparkFun-Switches:MOMENTARY-SWITCH-SPST-PTH-12MM
- removed S2: CLOCK_MODE, Switches:TACTILE_SWITCH_PTH_12MM, symbol SparkFun-Switches:MOMENTARY-SWITCH-SPST-PTH-12MM
- removed S3: CLOCK_STEP, Switches:TACTILE_SWITCH_PTH_12MM, symbol SparkFun-Switches:MOMENTARY-SWITCH-SPST-PTH-12MM
- removed VR1: 10k, Resistors:SLIDER-SMALL, symbol SparkFun-Resistors:POTENTIOMETER_SLIDE-20MM-1_10W-20%
- removed VR2: 10k, Resistors:POT-PTH-ALPS, symbol SparkFun-Resistors:POTENTIOMETER-PTH-9MM-1_20W-20%
- added C1: 0.1uF, Capacitor_THT:C_Disc_D3.0mm_W1.6mm_P2.50mm, symbol Device:C_Small
- added C2: 10uF, Capacitor_THT:CP_Radial_D4.0mm_P1.50mm, symbol Device:CP1
- added J2: INPUT, Connector_IDC:IDC-Header_2x08_P2.54mm_Vertical, symbol Connector_Generic:Conn_02x08_Odd_Even
- added U1: 74LS365, Package_DIP:DIP-16_W7.62mm, symbol 74xx:74LS365
Connections:
- net labels added: A3, CLOCK, DATA, HWD_DT, ~HWD_DT
- net labels removed: ~DIM0, ~DIM1, ~DIM2, ~DIM3
- wire segments 82 -> 77
- no-connect marks 12 -> 15
Other:
- note removed: "Clock Fast"
- note removed: "Clock Mode\nStop/Slow/Fast"
- note removed: "Clock Slow"
- note removed: "Clock Speed"
- note removed: "Clock Step"
- note removed: "Dimmer Level\n"
- note removed: "Dimmer Select\nDim0-Dim3"
- note removed: "Select Dim 0"
- note removed: "Select Dim 1\n"
- note removed: "Select Dim 2"
- note removed: "Select Dim 3"
- moved on the sheet: D1, D2, J1, R1, R2

Commit message: Prototype version of DMX, Analog, and PWM IO Modules and both TX and RX IO interfaces.
Parts:
- removed C2: 10uF, Capacitor_THT:CP_Radial_D4.0mm_P1.50mm, symbol Device:CP1
- added J3: IO EXTENSION, Connector_IDC:IDC-Header_2x07_P2.54mm_Horizontal, symbol Connector_Generic:Conn_02x07_Odd_Even
Connections:
- wire segments 77 -> 89
- no-connect marks 15 -> 20
Other:
- moved on the sheet: C1
Changed lines of the file:
@@
 EESchema Schematic File Version 4
-LIBS:transmitter-cache
+LIBS:transmitter-io-cache
 EELAYER 26 0
 EELAYER END
@@
 encoding utf-8
 Sheet 1 1
-Title "DMX Demonstrator - Transmitter for Control-Pro (DMX-TX2)"
-Date "2023-02-11"
+Title "DMX Demonstrator - Transmitter IO Module (DMX-TX2)"
+Date "2023-03-02"
 Rev "1.2"
 Comp "Crazy Giraffe Software"
@@
 $EndComp
 NoConn ~ 6850 2950
-NoConn ~ 7850 2750
-NoConn ~ 7850 2850
 $Comp
 L power:PWR_FLAG #FLG0101
@@
 	3250 4350 3250 4250
 Wire Wire Line
-	6150 3450 6150 4850
-Wire Wire Line
-	6150 4850 4500 4850
-Wire Wire Line
-	5450 3450 6150 3450
+	6100 3450 6100 4550
+Wire Wire Line
+	6100 4550 4500 4550
+Wire Wire Line
+	5450 3450 6100 3450
 Text Label 4700 3550 0    50   ~ 0
 ~CLOCK
@@
 	4300 3550 4950 3550
 Wire Wire Line
-	4500 4050 4500 4850
+	4500 4050 4500 4550
 Wire Wire Line
 	4400 3750 4300 3750
@@
 NoConn ~ 3300 3950
 $Comp
-L power:GND #PWR0114
-U 1 1 63F80A2D
-P 5700 7250
-F 0 "#PWR0114" H 5700 7000 50  0001 C CNN
-F 1 "GND" H 5705 7077 50  0000 C CNN
-F 2 "" H 5700 7250 50  0001 C CNN
-F 3 "" H 5700 7250 50  0001 C CNN
-	1    5700 7250
-	1    0    0    -1
-$EndComp
-$Comp
-L power:+5V #PWR?
-U 1 1 63F80AC6
-P 5700 6950
-AR Path="/6841E790/63F80AC6" Ref="#PWR?"  Part="1"
-AR Path="/63F80AC6" Ref="#PWR0115"  Part="1"
-AR Path="/5F613CCA/63F80AC6" Ref="#PWR?"  Part="1"
-F 0 "#PWR0115" H 5700 6800 50  0001 C CNN
-F 1 "+5V" H 5715 7123 50  0000 C CNN
-F 2 "" H 5700 6950 50  0001 C CNN
-F 3 "" H 5700 6950 50  0001 C CNN
-	1    5700 6950
-	1    0    0    -1
-$EndComp
-$Comp
 L Device:C_Small C1
 U 1 1 63F80B8A
-P 5300 7100
-F 0 "C1" H 5209 7054 50  0000 R CNN
-F 1 "0.1uF" H 5209 7145 50  0000 R CNN
-F 2 "Capacitor_THT:C_Disc_D3.0mm_W1.6mm_P2.50mm" H 5300 7100 50  0001 C CNN
-F 3 "~" H 5300 7100 50  0001 C CNN
-	1    5300 7100
+P 5750 7050
+F 0 "C1" H 5659 7004 50  0000 R CNN
+F 1 "0.1uF" H 5659 7095 50  0000 R CNN
+F 2 "Capacitor_THT:C_Disc_D3.0mm_W1.6mm_P2.50mm" H 5750 7050 50  0001 C CNN
+F 3 "~" H 5750 7050 50  0001 C CNN
+	1    5750 7050
 	1    0    0    1
 $EndComp
@@
 L power:GND #PWR0116
 U 1 1 63F80B90
-P 5300 7250
-F 0 "#PWR0116" H 5300 7000 50  0001 C CNN
-F 1 "GND" H 5305 7077 50  0000 C CNN
-F 2 "" H 5300 7250 50  0001 C CNN
-F 3 "" H 5300 7250 50  0001 C CNN
-	1    5300 7250
+P 5750 7250
+F 0 "#PWR0116" H 5750 7000 50  0001 C CNN
+F 1 "GND" H 5755 7077 50  0000 C CNN
+F 2 "" H 5750 7250 50  0001 C CNN
+F 3 "" H 5750 7250 50  0001 C CNN
+	1    5750 7250
 	1    0    0    -1
 $EndComp
@@
 L power:+5V #PWR?
 U 1 1 63F80B96
-P 5300 6950
+P 5750 6850
 AR Path="/6841E790/63F80B96" Ref="#PWR?"  Part="1"
 AR Path="/63F80B96" Ref="#PWR0117"  Part="1"
 AR Path="/5F613CCA/63F80B96" Ref="#PWR?"  Part="1"
-F 0 "#PWR0117" H 5300 6800 50  0001 C CNN
-F 1 "+5V" H 5315 7123 50  0000 C CNN
-F 2 "" H 5300 6950 50  0001 C CNN
-F 3 "" H 5300 6950 50  0001 C CNN
-	1    5300 6950
-	1    0    0    -1
-$EndComp
-$Comp
-L Device:CP1 C2
-U 1 1 63F82DD4
-P 5700 7100
-F 0 "C2" H 5500 7150 50  0000 L CNN
-F 1 "10uF" H 5450 7050 50  0000 L CNN
-F 2 "Capacitor_THT:CP_Radial_D4.0mm_P1.50mm" H 5700 7100 50  0001 C CNN
-F 3 "~" H 5700 7100 50  0001 C CNN
-	1    5700 7100
-	1    0    0    -1
-$EndComp
-Wire Wire Line
-	5300 7000 5300 6950
-Wire Wire Line
-	5300 7250 5300 7200
+F 0 "#PWR0117" H 5750 6700 50  0001 C CNN
+F 1 "+5V" H 5765 7023 50  0000 C CNN
+F 2 "" H 5750 6850 50  0001 C CNN
+F 3 "" H 5750 6850 50  0001 C CNN
+	1    5750 6850
+	1    0    0    -1
+$EndComp
+Wire Wire Line
+	5750 6950 5750 6850
+Wire Wire Line
+	5750 7250 5750 7150
+$Comp
+L Connector_Generic:Conn_02x07_Odd_Even J3
+U 1 1 63F5E071
+P 9250 2650
+F 0 "J3" H 9300 3167 50  0000 C CNN
+F 1 "IO EXTENSION" H 9300 3076 50  0000 C CNN
+F 2 "Connector_IDC:IDC-Header_2x07_P2.54mm_Horizontal" H 9250 2650 50  0001 C CNN
+F 3 "~" H 9250 2650 50  0001 C CNN
+	1    9250 2650
+	1    0    0    -1
+$EndComp
+Wire Wire Line
+	7850 2750 9050 2750
+Wire Wire Line
+	7850 2850 9050 2850
+$Comp
+L power:GND #PWR0118
+U 1 1 63F62AE3
+P 8900 3050
+F 0 "#PWR0118" H 8900 2800 50  0001 C CNN
+F 1 "GND" H 8905 2877 50  0000 C CNN
+F 2 "" H 8900 3050 50  0001 C CNN
+F 3 "" H 8900 3050 50  0001 C CNN
+	1    8900 3050
+	1    0    0    -1
+$EndComp
+$Comp
+L power:GND #PWR0119
+U 1 1 63F62B06
+P 9700 3050
+F 0 "#PWR0119" H 9700 2800 50  0001 C CNN
+F 1 "GND" H 9705 2877 50  0000 C CNN
+F 2 "" H 9700 3050 50  0001 C CNN
+F 3 "" H 9700 3050 50  0001 C CNN
+	1    9700 3050
+	1    0    0    -1
+$EndComp
+Wire Wire Line
+	9050 2950 8900 2950
+Wire Wire Line
+	8900 2950 8900 3050
+Wire Wire Line
+	9550 2950 9700 2950
+Wire Wire Line
+	9700 2950 9700 3050
+$Comp
+L power:+5V #PWR0120
+U 1 1 63F67888
+P 9700 2150
+F 0 "#PWR0120" H 9700 2000 50  0001 C CNN
+F 1 "+5V" H 9715 2323 50  0000 C CNN
+F 2 "" H 9700 2150 50  0001 C CNN
+F 3 "" H 9700 2150 50  0001 C CNN
+	1    9700 2150
+	1    0    0    -1
+$EndComp
+$Comp
+L power:+5V #PWR0121
+U 1 1 63F678AD
+P 8900 2150
+F 0 "#PWR0121" H 8900 2000 50  0001 C CNN
+F 1 "+5V" H 8915 2323 50  0000 C CNN
+F 2 "" H 8900 2150 50  0001 C CNN
+F 3 "" H 8900 2150 50  0001 C CNN
+	1    8900 2150
+	1    0    0    -1
+$EndComp
+Wire Wire Line
+	9700 2350 9700 2150
+Wire Wire Line
+	9050 2350 8900 2350
+Wire Wire Line
+	8900 2350 8900 2150
+Connection ~ 9700 2350
+Wire Wire Line
+	9550 2350 9700 2350
+NoConn ~ 9550 2450
+NoConn ~ 9550 2550
+NoConn ~ 9550 2650
+NoConn ~ 9050 2450
+NoConn ~ 9050 2550
+NoConn ~ 9050 2650
+Wire Wire Line
+	9550 2750 9700 2750
+Wire Wire Line
+	9700 2750 9700 2350
+NoConn ~ 9550 2850
+Wire Bus Line
+	3000 4900 8450 4900
+Wire Bus Line
+	6000 3200 6000 3750
 Wire Bus Line
 	6000 4050 6000 4800
 Wire Bus Line
-	6000 3200 6000 3750
-Wire Bus Line
-	3000 4900 8450 4900
+	8550 3050 8550 4800
 Wire Bus Line
 	4600 3850 4600 4650
 Wire Bus Line
-	8550 3050 8550 4800
-Wire Bus Line
 	2900 3650 2900 4800

Commit message: Ouptut local gerbers (ignored) Add detected LED to tx2
Parts:
- added D3: DETECTED, LED_THT:LED_D5.0mm, symbol Device:LED
- added R3: 330, Resistor_THT:R_Axial_DIN0207_L6.3mm_D2.5mm_P10.16mm_Horizontal, symbol Device:R_US
- renumbered R3 to R4
Connections:
- net labels added: ~CLOCK_OUT, ~DATA_OUT, ~HWD_DT_OUT
- net labels removed: CLOCK, DATA, HWD_DT
- wire segments 89 -> 96
- no-connect marks 20 -> 18
Other:
- note added: "Detected"
- moved on the sheet: D1, D2, R1, R2

Commit message: Use 74LS07 Led driver Add R5 for discovery.
Parts:
- removed U1: 74LS365, Package_DIP:DIP-16_W7.62mm, symbol 74xx:74LS365
- added R5: 330, Resistor_THT:R_Axial_DIN0207_L6.3mm_D2.5mm_P10.16mm_Horizontal, symbol Device:R_US
- added U1: 74LS07, Package_DIP:DIP-14_W7.62mm, symbol CrazyGiraffe_DMXDemonstrator:74LS07
Connections:
- wire segments 96 -> 97
- no-connect marks 18 -> 16
Other:
- moved on the sheet: R4
Changed lines of the file:
@@
 Sheet 1 1
 Title "DMX Demonstrator - Transmitter IO Module (DMX-TX2)"
-Date "2023-03-02"
-Rev "1.2"
+Date "2023-09-16"
+Rev "1.3"
 Comp "Crazy Giraffe Software"
 Comment1 ""
@@
 L Device:R_US R?
 U 1 1 5F6228C3
-P 8250 4250
+P 8400 4250
 AR Path="/5F613CCA/5F6228C3" Ref="R?"  Part="1"
 AR Path="/5F6228C3" Ref="R4"  Part="1"
-F 0 "R4" H 8100 4300 50  0000 L CNN
-F 1 "330" H 8050 4200 50  0000 L CNN
-F 2 "Resistor_THT:R_Axial_DIN0207_L6.3mm_D2.5mm_P10.16mm_Horizontal" V 8290 4240 50  0001 C CNN
-F 3 "~" H 8250 4250 50  0001 C CNN
-	1    8250 4250
-	-1   0    0    -1
+F 0 "R4" H 8250 4300 50  0000 L CNN
+F 1 "330" H 8200 4200 50  0000 L CNN
+F 2 "Resistor_THT:R_Axial_DIN0207_L6.3mm_D2.5mm_P10.16mm_Horizontal" V 8440 4240 50  0001 C CNN
+F 3 "~" H 8400 4250 50  0001 C CNN
+	1    8400 4250
+	1    0    0    -1
 $EndComp
 $Comp
 L power:GND #PWR?
 U 1 1 5F6228CA
-P 8250 4600
+P 8400 4600
 AR Path="/5F613CCA/5F6228CA" Ref="#PWR?"  Part="1"
 AR Path="/5F6228CA" Ref="#PWR0110"  Part="1"
-F 0 "#PWR0110" H 8250 4350 50  0001 C CNN
-F 1 "GND" H 8255 4427 50  0000 C CNN
-F 2 "" H 8250 4600 50  0001 C CNN
-F 3 "" H 8250 4600 50  0001 C CNN
-	1    8250 4600
+F 0 "#PWR0110" H 8400 4350 50  0001 C CNN
+F 1 "GND" H 8405 4427 50  0000 C CNN
+F 2 "" H 8400 4600 50  0001 C CNN
+F 3 "" H 8400 4600 50  0001 C CNN
+	1    8400 4600
 	1    0    0    -1
 $EndComp
@@
 	8450 3650 8550 3750
 Wire Wire Line
-	7850 3850 8250 3850
+	7850 3850 8400 3850
 Wire Wire Line
 	7850 3750 8450 3750
@@
 	7850 3950 8750 3950
 Wire Wire Line
-	8250 3850 8250 4100
-Wire Wire Line
-	8250 4400 8250 4600
+	8400 3850 8400 4100
+Wire Wire Line
+	8400 4400 8400 4600
 Wire Wire Line
 	9100 4250 8750 4250
@@
 	8450 3050 8550 3150
 NoConn ~ 7850 3150
-NoConn ~ 7850 3250
-NoConn ~ 7850 3350
 NoConn ~ 7850 3450
 Wire Wire Line
@@
 Wire Wire Line
 	5450 3850 5900 3850
-$Comp
-L 74xx:74LS365 U1
-U 1 1 63EBDEC4
-P 3700 3950
-F 0 "U1" H 3900 4600 50  0000 C CNN
-F 1 "74LS365" H 3950 4500 50  0000 C CNN
-F 2 "Package_DIP:DIP-16_W7.62mm" H 3700 3950 50  0001 C CNN
-F 3 "http://www.ti.com/lit/gpn/sn74LS365" H 3700 3950 50  0001 C CNN
-	1    3700 3950
-	1    0    0    -1
-$EndComp
 $Comp
 L power:+5V #PWR?
@@
 Wire Wire Line
 	2700 3650 3200 3650
-$Comp
-L power:GND #PWR?
-U 1 1 63ED20FA
-P 3150 4650
-AR Path="/5F613CCA/63ED20FA" Ref="#PWR?"  Part="1"
-AR Path="/63ED20FA" Ref="#PWR0113"  Part="1"
-F 0 "#PWR0113" H 3150 4400 50  0001 C CNN
-F 1 "GND" H 3155 4477 50  0000 C CNN
-F 2 "" H 3150 4650 50  0001 C CNN
-F 3 "" H 3150 4650 50  0001 C CNN
-	1    3150 4650
-	1    0    0    -1
-$EndComp
-Wire Wire Line
-	3150 4650 3150 4350
-Wire Wire Line
-	3150 4250 3200 4250
-Wire Wire Line
-	3200 4350 3150 4350
-Connection ~ 3150 4350
-Wire Wire Line
-	3150 4350 3150 4250
 Wire Wire Line
 	6100 3450 6100 4550
@@
 Wire Wire Line
 	4400 3850 4400 2150
+Wire Wire Line
+	4400 2150 4750 2150
+$Comp
+L Device:R_US R?
+U 1 1 6506CFB2
+P 8400 2450
+AR Path="/5F613CCA/6506CFB2" Ref="R?"  Part="1"
+AR Path="/6506CFB2" Ref="R5"  Part="1"
+F 0 "R5" H 8250 2500 50  0000 L CNN
+F 1 "330" H 8200 2400 50  0000 L CNN
+F 2 "Resistor_THT:R_Axial_DIN0207_L6.3mm_D2.5mm_P10.16mm_Horizontal" V 8440 2440 50  0001 C CNN
+F 3 "~" H 8400 2450 50  0001 C CNN
+	1    8400 2450
+	1    0    0    -1
+$EndComp
+Wire Wire Line
+	8400 2600 8400 3250
+Wire Wire Line
+	7850 3350 8400 3350
+Wire Wire Line
+	7850 3250 8400 3250
+Connection ~ 8400 3250
+Wire Wire Line
+	8400 3250 8400 3350
+$Comp
+L power:+5V #PWR0114
+U 1 1 65080226
+P 8400 2150
+F 0 "#PWR0114" H 8400 2000 50  0001 C CNN
+F 1 "+5V" H 8415 2323 50  0000 C CNN
+F 2 "" H 8400 2150 50  0001 C CNN
+F 3 "" H 8400 2150 50  0001 C CNN
+	1    8400 2150
+	1    0    0    -1
+$EndComp
+Wire Wire Line
+	8400 2150 8400 2300
+Wire Bus Line
+	2600 3650 2600 4800
+Wire Bus Line
+	6400 3200 6400 4650
+Wire Bus Line
+	4600 3850 4600 4650
+Wire Bus Line
+	8550 3050 8550 4800
+Wire Bus Line
+	6000 4050 6000 4800
+Wire Bus Line
+	6000 3200 6000 3750
 Wire Bus Line
 	2700 4900 8450 4900
-Wire Bus Line
-	6000 3200 6000 3750
-Wire Bus Line
-	6000 4050 6000 4800
-Wire Bus Line
-	8550 3050 8550 4800
-Wire Bus Line
-	4600 3850 4600 4650
-Wire Bus Line
-	6400 3200 6400 4650
-Wire Bus Line
-	2600 3650 2600 4800
-Wire Wire Line
-	4400 2150 4750 2150
+$Comp
+L CrazyGiraffe_DMXDemonstrator:74LS07 U1
+U 1 1 6508D26C
+P 3700 3950
+F 0 "U1" H 3900 4600 50  0000 C CNN
+F 1 "74LS07" H 3950 4500 50  0000 C CNN
+F 2 "Package_DIP:DIP-14_W7.62mm" H 3700 3950 50  0001 C CNN
+F 3 "https://www.ti.com/lit/ds/symlink/sn74ls07.pdf" H 3700 3950 50  0001 C CNN
+	1    3700 3950
+	1    0    0    -1
+$EndComp
 $EndSCHEMATC

Commit message: Rebrand to Sparky Bobo Designs
Parts:
- A1: symbol MCU_Module:Arduino_UNO_R3 -> DMXDemonstrator:Arduino_UNO_R3-MCU_Module
- U1: symbol CrazyGiraffe_DMXDemonstrator:74LS07 -> DMXDemonstrator:74LS07
Changed lines of the file:
@@
 EESchema Schematic File Version 4
-LIBS:transmitter-io-cache
-EELAYER 26 0
+EELAYER 30 0
 EELAYER END
 $Descr A4 11693 8268
@@
 Date "2023-09-16"
 Rev "1.3"
-Comp "Crazy Giraffe Software"
+Comp "Sparky Bobo Designs"
 Comment1 ""
 Comment2 "Designed by: SparkyBobo"
@@
 $EndDescr
 $Comp
-L MCU_Module:Arduino_UNO_R3 A1
+L DMXDemonstrator:Arduino_UNO_R3-MCU_Module A1
 U 1 1 5F3035A0
 P 7350 3350
@@
 Wire Wire Line
 	8400 2150 8400 2300
-Wire Bus Line
-	2600 3650 2600 4800
-Wire Bus Line
-	6400 3200 6400 4650
-Wire Bus Line
-	4600 3850 4600 4650
-Wire Bus Line
-	8550 3050 8550 4800
-Wire Bus Line
-	6000 4050 6000 4800
-Wire Bus Line
-	6000 3200 6000 3750
-Wire Bus Line
-	2700 4900 8450 4900
-$Comp
-L CrazyGiraffe_DMXDemonstrator:74LS07 U1
+$Comp
+L DMXDemonstrator:74LS07 U1
 U 1 1 6508D26C
 P 3700 3950
@@
 	1    0    0    -1
 $EndComp
+Wire Bus Line
+	6000 4050 6000 4800
+Wire Bus Line
+	6000 3200 6000 3750
+Wire Bus Line
+	2700 4900 8450 4900
+Wire Bus Line
+	4600 3850 4600 4650
+Wire Bus Line
+	8550 3050 8550 4800
+Wire Bus Line
+	6400 3200 6400 4650
+Wire Bus Line
+	2600 3650 2600 4800
 $EndSCHEMATC

Commit message: Users/sparky/hwcleanup (#22)
* Rename control-pro
Update readmes
Delete old pngs

* Add PWM headers on DMX-RX1.

* Add BOM generator
Add BOM and parts .md's
Parts:
- A1: PartId (none) -> A_ARDUINO,H_ARDUINO
- C1: PartId (none) -> C_DECOUPLE
- D1: PartId (none) -> LED_GRN
- D2, D3: PartId (none) -> LED_RED
- J1: PartId (none) -> H_1x3_RA
- J2: footprint Connector_IDC:IDC-Header_2x08_P2.54mm_Vertical -> Connector_IDC:IDC-Header_2x08_P2.54mm_Horizontal; PartId (none) -> H_CPRO
- J3: PartId (none) -> H_IO_RA
- R1, R2, R3, R4, R5: PartId (none) -> R_LED
- U1: PartId (none) -> U_74LS07
Changed lines of the file:
@@
 F 2 "footprints:ARDUINO_R3_NO_HOLES" H 7500 2300 50  0001 L CNN
 F 3 "https://www.arduino.cc/en/Main/arduinoBoardUno" H 7150 4400 50  0001 C CNN
+F 4 "A_ARDUINO,H_ARDUINO" H 7350 3350 50  0001 C CNN "PartId"
 	1    7350 3350
 	-1   0    0    -1
@@
 F 2 "Connector_PinHeader_2.54mm:PinHeader_1x03_P2.54mm_Horizontal" H 9300 4150 50  0001 C CNN
 F 3 "~" H 9300 4150 50  0001 C CNN
+F 4 "H_1x3_RA" H 9300 4150 50  0001 C CNN "PartId"
 	1    9300 4150
 	1    0    0    -1
@@
 F 2 "LED_THT:LED_D5.0mm" H 4900 2150 50  0001 C CNN
 F 3 "~" H 4900 2150 50  0001 C CNN
+F 4 "LED_GRN" H 4900 2150 50  0001 C CNN "PartId"
 	1    4900 2150
 	1    0    0    -1
@@
 F 2 "Resistor_THT:R_Axial_DIN0207_L6.3mm_D2.5mm_P10.16mm_Horizontal" V 5290 2140 50  0001 C CNN
 F 3 "~" H 5250 2150 50  0001 C CNN
+F 4 "R_LED" V 5250 2150 50  0001 C CNN "PartId"
 	1    5250 2150
 	0    1    1    0
@@
 F 2 "LED_THT:LED_D5.0mm" H 4900 2500 50  0001 C CNN
 F 3 "~" H 4900 2500 50  0001 C CNN
+F 4 "LED_RED" H 4900 2500 50  0001 C CNN "PartId"
 	1    4900 2500
 	1    0    0    -1
@@
 F 2 "Resistor_THT:R_Axial_DIN0207_L6.3mm_D2.5mm_P10.16mm_Horizontal" V 5290 2490 50  0001 C CNN
 F 3 "~" H 5250 2500 50  0001 C CNN
+F 4 "R_LED" V 5250 2500 50  0001 C CNN "PartId"
 	1    5250 2500
 	0    1    1    0
@@
 F 0 "J2" H 5200 4267 50  0000 C CNN
 F 1 "INPUT" H 5200 4176 50  0000 C CNN
-F 2 "Connector_IDC:IDC-Header_2x08_P2.54mm_Vertical" H 5150 3750 50  0001 C CNN
+F 2 "Connector_IDC:IDC-Header_2x08_P2.54mm_Horizontal" H 5150 3750 50  0001 C CNN
 F 3 "~" H 5150 3750 50  0001 C CNN
+F 4 "H_CPRO" H 5150 3750 50  0001 C CNN "PartId"
 	1    5150 3750
 	1    0    0    -1
@@
 F 2 "Resistor_THT:R_Axial_DIN0207_L6.3mm_D2.5mm_P10.16mm_Horizontal" V 8440 4240 50  0001 C CNN
 F 3 "~" H 8400 4250 50  0001 C CNN
+F 4 "R_LED" H 8400 4250 50  0001 C CNN "PartId"
 	1    8400 4250
 	1    0    0    -1
@@
 F 2 "Capacitor_THT:C_Disc_D3.0mm_W1.6mm_P2.50mm" H 5750 7050 50  0001 C CNN
 F 3 "~" H 5750 7050 50  0001 C CNN
+F 4 "C_DECOUPLE" H 5750 7050 50  0001 C CNN "PartId"
 	1    5750 7050
 	1    0    0    1
@@
 F 2 "Connector_IDC:IDC-Header_2x07_P2.54mm_Horizontal" H 9250 2650 50  0001 C CNN
 F 3 "~" H 9250 2650 50  0001 C CNN
+F 4 "H_IO_RA" H 9250 2650 50  0001 C CNN "PartId"
 	1    9250 2650
 	1    0    0    -1
@@
 F 2 "LED_THT:LED_D5.0mm" H 4900 2850 50  0001 C CNN
 F 3 "~" H 4900 2850 50  0001 C CNN
+F 4 "LED_RED" H 4900 2850 50  0001 C CNN "PartId"
 	1    4900 2850
 	1    0    0    -1
@@
 F 2 "Resistor_THT:R_Axial_DIN0207_L6.3mm_D2.5mm_P10.16mm_Horizontal" V 5290 2840 50  0001 C CNN
 F 3 "~" H 5250 2850 50  0001 C CNN
+F 4 "R_LED" V 5250 2850 50  0001 C CNN "PartId"
 	1    5250 2850
 	0    1    1    0
@@
 F 2 "Resistor_THT:R_Axial_DIN0207_L6.3mm_D2.5mm_P10.16mm_Horizontal" V 8440 2440 50  0001 C CNN
 F 3 "~" H 8400 2450 50  0001 C CNN
+F 4 "R_LED" H 8400 2450 50  0001 C CNN "PartId"
 	1    8400 2450
 	1    0    0    -1
@@
 F 2 "Package_DIP:DIP-14_W7.62mm" H 3700 3950 50  0001 C CNN
 F 3 "https://www.ti.com/lit/ds/symlink/sn74ls07.pdf" H 3700 3950 50  0001 C CNN
+F 4 "U_74LS07" H 3700 3950 50  0001 C CNN "PartId"
 	1    3700 3950
 	1    0    0    -1
