File: hardware/io-dmx/io-dmx-512.sch (KiCad schematic (older format))
At the start: 26 parts, among them J1 IO EXTENSION, J2 NC3FAH/NC5FAH, J3 NC3MAH/NC5MAH, U1 NMA0505SC, U2 6N137, U3 6N137, U4 6N137, U5 MAX3485CPA+

Commit message: Prototype version of DMX, Analog, and PWM IO Modules and both TX and RX IO interfaces.
Parts:
- removed R1: 330, Resistor_THT:R_Axial_DIN0207_L6.3mm_D2.5mm_P10.16mm_Horizontal, symbol Device:R_US
Connections:
- net labels added: DMX-DIR, DMX-RX, DMX-TX
- wire segments 113 -> 110
- no-connect marks 14 -> 15
Changed lines of the file:
@@
 EESchema Schematic File Version 4
-LIBS:dimmer-dmx-cache
+LIBS:io-dmx-512-cache
 EELAYER 26 0
 EELAYER END
@@
 encoding utf-8
 Sheet 1 1
-Title "DMX Demonstrator - DMX-512 IO Module (DMX-DD1)"
+Title "DMX Demonstrator - DMX-512 IO Module (DMX-IO1)"
 Date "2023-02-19"
 Rev "1.1"
@@
 	4150 3750 5150 3750
 $Comp
-L Device:R_US R1
-U 1 1 63F76368
-P 4500 3850
-F 0 "R1" V 4400 3850 50  0000 C CNN
-F 1 "330" V 4300 3850 50  0000 C CNN
-F 2 "Resistor_THT:R_Axial_DIN0207_L6.3mm_D2.5mm_P10.16mm_Horizontal" V 4540 3840 50  0001 C CNN
-F 3 "~" H 4500 3850 50  0001 C CNN
-	1    4500 3850
-	0    1    -1   0
-$EndComp
-Wire Wire Line
-	4150 3850 4350 3850
-Wire Wire Line
-	4650 3850 4750 3850
-Wire Wire Line
-	4750 3850 4750 4050
-$Comp
-L power:GND #PWR0131
-U 1 1 63F877A0
-P 4750 4050
-F 0 "#PWR0131" H 4750 3800 50  0001 C CNN
-F 1 "GND" H 4755 3877 50  0000 C CNN
-F 2 "" H 4750 4050 50  0001 C CNN
-F 3 "" H 4750 4050 50  0001 C CNN
-	1    4750 4050
-	1    0    0    -1
-$EndComp
-$Comp
 L Mechanical:MountingHole MH1
 U 1 1 63F9E49B
@@
 	4600 3350 4250 3350
 Connection ~ 4250 3350
+Text Label 3350 3750 0    50   ~ 0
+DMX-RX
+Text Label 3350 3850 0    50   ~ 0
+DMX-TX
+Text Label 4200 3750 0    50   ~ 0
+DMX-DIR
+NoConn ~ 4150 3850
 $EndSCHEMATC

Commit message: Finalize io-dmx board
Parts:
- C2, C3, C4, C5: footprint Capacitors:CAP-PTH-2.54 -> Capacitor_THT:C_Rect_L4.6mm_W2.0mm_P2.50mm_MKS02_FKP02
Changed lines of the file:
@@
 F 0 "C2" H 2915 6996 50  0000 L CNN
 F 1 ".01uF" H 2915 6905 50  0000 L CNN
-F 2 "Capacitors:CAP-PTH-2.54" H 2838 6800 50  0001 C CNN
+F 2 "Capacitor_THT:C_Rect_L4.6mm_W2.0mm_P2.50mm_MKS02_FKP02" H 2838 6800 50  0001 C CNN
 F 3 "~" H 2800 6950 50  0001 C CNN
 	1    2800 6950
@@
 F 0 "C3" H 5765 7046 50  0000 L CNN
 F 1 ".01uF" H 5765 6955 50  0000 L CNN
-F 2 "Capacitors:CAP-PTH-2.54" H 5688 6850 50  0001 C CNN
+F 2 "Capacitor_THT:C_Rect_L4.6mm_W2.0mm_P2.50mm_MKS02_FKP02" H 5688 6850 50  0001 C CNN
 F 3 "~" H 5650 7000 50  0001 C CNN
 	1    5650 7000
@@
 F 0 "C4" H 6215 7046 50  0000 L CNN
 F 1 ".01uF" H 6215 6955 50  0000 L CNN
-F 2 "Capacitors:CAP-PTH-2.54" H 6138 6850 50  0001 C CNN
+F 2 "Capacitor_THT:C_Rect_L4.6mm_W2.0mm_P2.50mm_MKS02_FKP02" H 6138 6850 50  0001 C CNN
 F 3 "~" H 6100 7000 50  0001 C CNN
 	1    6100 7000
@@
 F 0 "C5" H 6665 7046 50  0000 L CNN
 F 1 ".01uF" H 6665 6955 50  0000 L CNN
-F 2 "Capacitors:CAP-PTH-2.54" H 6588 6850 50  0001 C CNN
+F 2 "Capacitor_THT:C_Rect_L4.6mm_W2.0mm_P2.50mm_MKS02_FKP02" H 6588 6850 50  0001 C CNN
 F 3 "~" H 6550 7000 50  0001 C CNN
 	1    6550 7000

Commit message: Added Bill Of Materials (BOM)
Parts:
- removed R10, R8: 680, Resistor_THT:R_Axial_DIN0207_L6.3mm_D2.5mm_P10.16mm_Horizontal, symbol Device:R_US
- C2, C3, C4, C5: value .01uF -> 0.1uF; AF_Detail_Page (none) -> https://www.adafruit.com/product/753; AF_PN (none) -> 753; Description (none) -> Decoupling Capacitor; MO_Detail_Page (none) -> https://www.mouser.com/ProductDetail/KEMET/C320C104K5R5TA73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; MO_PN (none) -> 80-C320C104K5R7301; NW_Detail_Page (none) -> https://www.newark.com/kemet/c315c104m5u5ta/capacitor-mlcc-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; NW_PN (none) -> 13K6284; SP_Detail_Page (none) -> https://www.sparkfun.com/products/8375; SP_PN (none) -> COM-08375
- J1: MO_Detail_Page (none) -> https://www.mouser.com/ProductDetail/Wurth-Elektronik/61201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; MO_PN (none) -> 710-61201421721; NW_Detail_Page (none) -> https://www.newark.com/wurth-elektronik/612014235221/conn-r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; NW_PN (none) -> 75AJ1395
- J2: Description (none) -> DMX Connector; MO_Detail_Page (none) -> https://www.mouser.com/ProductDetail/Neutrik/NC5FAH/?qs=JfN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; MO_PN (none) -> 568-NC5FAH; NW_Detail_Page (none) -> https://www.newark.com/neutrik/nc5fah/connector-xlr-recepta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; NW_PN (none) -> 94C1524
- J3: Description (none) -> DMX Connector; MO (none) -> 568-NC5MAH; MO_Detail_page (none) -> https://www.mouser.com/ProductDetail/Neutrik/NC5MAH/?qs=43p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; NW_Detail_Page (none) -> https://www.newark.com/neutrik/nc5mah/connector-xlr-audio-p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; NW_PM (none) -> 25C4313
- R1: renamed from R9; Description (none) -> DMX Termination; MO_Detail_Page (none) -> https://www.mouser.com/ProductDetail/Yageo/CFR-25JT-52-120R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; MO_PN (none) -> 603-CFR-25JT-52-120R; NW_Detail_Page (none) -> https://www.newark.com/multicomp-pro/mcf-0-25w-120r/carbon-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; NW_PN (none) -> 38K0333
- R2, R3, R4, R5, R6, R7: AF_Detail_Page (none) -> https://www.adafruit.com/product/2781; AF_PN (none) -> 2781; MO_Detail_Page (none) -> https://www.mouser.com/ProductDetail/Yageo/CFR-25JT-52-470R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; MO_PN (none) -> 603-CFR-25JT-52-470R; NW_Detail_Page (none) -> https://www.newark.com/multicomp-pro/mcf-0-25w-470r/carbon-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; NW_PN (none) -> 38K0375
- U1: Description (none) -> Isolated 1W Dual Output DC-DC Converter; MO_Detail_Page (none) -> https://www.mouser.com/ProductDetail/Murata-Power-Solutions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; MO_PN (none) -> 580-NMA0505SC; NW_Detail_Page (none) -> https://www.newark.com/murata-power-solutions/nma0505sc/dc-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; NW_PN (none) -> 61K3058
- U2, U3, U4: MO_Detail_Page (none) -> https://www.mouser.com/ProductDetail/Vishay-Semiconductors/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; MO_PN (none) -> 782-6N137; NW_Detail_Page (none) -> https://www.newark.com/vishay/6n137/optocoupler-transistor-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; NW_PN (none) -> 52M1895
- U5: DK_Page_Detail (none) -> products/detail/MAX3485CPA%2B/MAX3485CPA%2B-ND/1702227; Description (none) -> RS-485/RS-422 Transceiver; Digi-Key_PN (none) -> MAX3485CPA+-ND; MO_Detail_Page (none) -> https://www.mouser.com/ProductDetail/Maxim-Integrated/MAX34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; MO_PN (none) -> 700-MAX3485CPA; NW_Detail_Page (none) -> https://www.newark.com/maxim-integrated-products/max3485cpa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; NW_PN (none) -> 81Y9431
Connections:
- wire segments 110 -> 107
Other:
- note removed: "Connect J4 to J5\nto bypass isolator"
- note removed: "Connect pin 2 to 4\nto bypass isolator"
- note removed: "Connect\npin 3 to 6\nto bypass\nisolator"

Commit message: Display Pro: - Switch to smaller screw terminal connectors - Add pull-down resistors - Add silkscreen values - Remove COAX power connector...again - Add test software
Core:
- Fix issue with A03 and A02 being reversed at Analog Extensions
- Fix issue with A1 and A0 at IO Extension header
- Label D0..D7 correctly
- Swap U4 and U5 in schematic to match board layout
- Change TO-92 footprint
- Add silkscreen values
- Add test software

PWM:
- Switch to smaller screw terminal connectors
- Add silkscreen values
- Remove COAX power connector

Voltage:
- Switch to smaller screw terminal connectors
- Add silkscreen values
- Remove COAX power connector

DMX:
- Fix issue with DMX A and B being reversed
- Group bypass-only resistors together
- Add ISO bypass solder bridges
- Add silkscreen values
- Remove RDM bias resistors
- Add test software

Rx-IO:
- Fix issue with A1 and A0 at IO Extension header
- Add silkscreen values

Tx-IO:
- Switch to 74LS07 for Led driver
- Add pulldown resistor for discovery
- Add silkscreen values

Discovery:
- Make use of new Tx-IO pulldown resistor
Parts:
- added JP1, JP2, JP3: Bypass Iso, Jumper:SolderJumper-2_P1.3mm_Open_Pad1.0x1.5mm, symbol Jumper:SolderJumper_2_Open
Connections:
- wire segments 107 -> 121
Other:
- note added: "Jump to\nBypass Iso"
Changed lines of the file:
@@
 Sheet 1 1
 Title "DMX Demonstrator - DMX-512 IO Module (DMX-IO1)"
-Date "2023-08-11"
-Rev "1.3"
+Date "2023-10-28"
+Rev "1.4"
 Comp "Crazy Giraffe Software"
 Comment1 ""
@@
 Connection ~ 6000 1950
 Wire Wire Line
-	5400 1950 5300 1950
-Wire Wire Line
-	5300 1950 5300 2300
-Connection ~ 5300 2300
+	5400 1950 5000 1950
+Wire Wire Line
+	5000 1950 5000 2300
+Connection ~ 5000 2300
 $Comp
 L dk_Optoisolators-Logic-Output:6N137 U4
@@
 	7800 3800 7900 3800
 Wire Wire Line
-	8000 3900 8100 3900
-Wire Wire Line
 	8100 3900 8100 3800
 Connection ~ 8100 3900
@@
 Wire Wire Line
 	8700 3900 8550 3900
-Wire Wire Line
-	8000 3500 8000 3900
-Wire Wire Line
-	7800 3500 8000 3500
-Wire Wire Line
-	7900 3800 7900 3400
 Wire Wire Line
 	7900 3400 8100 3400
@@
 	3100 6750 3700 6750
 Wire Wire Line
-	6900 2400 6900 3500
+	6900 2400 6900 2900
 Wire Wire Line
 	6400 2400 6550 2400
 Wire Wire Line
-	5300 2300 5600 2300
+	5000 2300 5600 2300
 Wire Wire Line
 	5450 3750 5600 3750
@@
 	3300 3750 3300 2300
 Wire Wire Line
-	3300 2300 5300 2300
-Wire Wire Line
-	3300 5100 5150 5100
+	3300 2300 5000 2300
+Wire Wire Line
+	3300 5100 5000 5100
 Wire Wire Line
 	3300 5100 3300 3850
 Wire Wire Line
-	4150 3750 5150 3750
+	4150 3750 5000 3750
 $Comp
 L Mechanical:MountingHole MH1
@@
 	1    0    0    -1
 $EndComp
+$Comp
+L Jumper:SolderJumper_2_Open JP1
+U 1 1 651B256A
+P 5250 2900
+F 0 "JP1" H 5250 3105 50  0000 C CNN
+F 1 "Bypass Iso" H 5250 3014 50  0000 C CNN
+F 2 "Jumper:SolderJumper-2_P1.3mm_Open_Pad1.0x1.5mm" H 5250 2900 50  0001 C CNN
+F 3 "~" H 5250 2900 50  0001 C CNN
+	1    5250 2900
+	1    0    0    -1
+$EndComp
+Wire Wire Line
+	5400 2900 6900 2900
+Connection ~ 6900 2900
+Wire Wire Line
+	6900 2900 6900 3500
+Wire Wire Line
+	5100 2900 5000 2900
+Wire Wire Line
+	5000 2900 5000 2300
+$Comp
+L Jumper:SolderJumper_2_Open JP2
+U 1 1 651B907A
+P 5300 4250
+F 0 "JP2" H 5300 4455 50  0000 C CNN
+F 1 "Bypass Iso" H 5300 4364 50  0000 C CNN
+F 2 "Jumper:SolderJumper-2_P1.3mm_Open_Pad1.0x1.5mm" H 5300 4250 50  0001 C CNN
+F 3 "~" H 5300 4250 50  0001 C CNN
+	1    5300 4250
+	1    0    0    -1
+$EndComp
+Wire Wire Line
+	5450 4250 6700 4250
+Wire Wire Line
+	6700 4250 6700 3650
+Wire Wire Line
+	5000 3750 5000 4250
+Wire Wire Line
+	5000 4250 5150 4250
+Connection ~ 5000 3750
+Wire Wire Line
+	5000 3750 5150 3750
+$Comp
+L Jumper:SolderJumper_2_Open JP3
+U 1 1 651C0494
+P 5300 5600
+F 0 "JP3" H 5300 5805 50  0000 C CNN
+F 1 "Bypass Iso" H 5300 5714 50  0000 C CNN
+F 2 "Jumper:SolderJumper-2_P1.3mm_Open_Pad1.0x1.5mm" H 5300 5600 50  0001 C CNN
+F 3 "~" H 5300 5600 50  0001 C CNN
+	1    5300 5600
+	1    0    0    -1
+$EndComp
+Wire Wire Line
+	5450 5600 6900 5600
+Wire Wire Line
+	6900 5600 6900 5000
+Connection ~ 6900 5000
+Wire Wire Line
+	5150 5600 5000 5600
+Wire Wire Line
+	5000 5600 5000 5100
+Connection ~ 5000 5100
+Wire Wire Line
+	5000 5100 5150 5100
+Text Notes 4000 7500 0    50   ~ 0
+Jump to\nBypass Iso
+Text Notes 4050 6400 0    50   ~ 0
+Jump to\nBypass Iso
+Wire Notes Line
+	4500 6300 4750 6300
+Wire Notes Line
+	4750 6300 4750 6750
+Wire Notes Line
+	4750 7150 4750 7400
+Wire Notes Line
+	4750 7400 4450 7400
+Wire Notes Line
+	3950 7400 3650 7400
+Wire Notes Line
+	3650 7400 3650 7150
+Wire Notes Line
+	3650 6750 3650 6300
+Wire Notes Line
+	3650 6300 4000 6300
+Wire Wire Line
+	7800 3500 7900 3500
+Wire Wire Line
+	7900 3500 7900 3400
+Wire Wire Line
+	7900 3800 7900 3900
+Wire Wire Line
+	7900 3900 8100 3900
 $EndSCHEMATC

Commit message: Consolidate parts library. Rebrand.
Parts:
- J2, J3: symbol parts.library:XLR-3-5 -> DMXDemonstrator:XLR-3-5
- U2, U3, U4: symbol dk_Optoisolators-Logic-Output:6N137 -> DMXDemonstrator:6N137-dk_Optoisolators-Logic-Output
Changed lines of the file:
@@
 EESchema Schematic File Version 4
-LIBS:io-dmx-512-cache
-EELAYER 26 0
+EELAYER 30 0
 EELAYER END
 $Descr A4 11693 8268
@@
 Date "2023-12-19"
 Rev "1.5"
-Comp "Crazy Giraffe Software"
+Comp "Sparky Bobo Designs"
 Comment1 ""
 Comment2 "Designed by: SparkyBobo"
@@
 Connection ~ 5000 2300
 $Comp
-L dk_Optoisolators-Logic-Output:6N137 U4
+L DMXDemonstrator:6N137-dk_Optoisolators-Logic-Output U4
 U 1 1 5F60D784
 P 6000 5000
@@
 	8100 3900 8550 3900
 $Comp
-L parts.library:XLR-3-5 J3
+L DMXDemonstrator:XLR-3-5 J3
 U 1 1 5FA9D811
 P 9000 3800
@@
 $EndComp
 $Comp
-L parts.library:XLR-3-5 J2
+L DMXDemonstrator:XLR-3-5 J2
 U 1 1 5FA9D8B9
 P 9000 3000
@@
 $EndComp
 $Comp
-L dk_Optoisolators-Logic-Output:6N137 U3
+L DMXDemonstrator:6N137-dk_Optoisolators-Logic-Output U3
 U 1 1 64D4B0B9
 P 6000 3650
@@
 $EndComp
 $Comp
-L dk_Optoisolators-Logic-Output:6N137 U2
+L DMXDemonstrator:6N137-dk_Optoisolators-Logic-Output U2
 U 1 1 64D4B117
 P 6000 2300
